File: hardware/EVAL MSPM0lG3507 BQ7962/EVAL MSPM0lG3507 BQ7962.kicad_pcb (KiCad board)
At the start: 2 copper layers, 72.5 x 101.3 mm, 168 parts, among them J1 Conn_01x09_Socket, J10 Screw_Terminal_01x02, J11 Screw_Terminal_01x02, J12 Screw_Terminal_01x02, J13 Screw_Terminal_01x02, J14 Screw_Terminal_01x02, J15 Conn_01x02_Pin, J16 USB_B_Micro, J2 Conn_02x05_Odd_Even, J3 Conn_01x04_Pin, J4 Screw_Terminal_01x02, J6 Conn_01x02_Pin, J7 Screw_Terminal_01x02, J8 Screw_Terminal_01x02, J9 Screw_Terminal_01x02, Q1 2N7002, Q2 2N7002, Q6 2N7002, SW1 SW_Push, U1 ISO7721D, U10 MCP2542FDxMF, U11 FCX495, U12 FT230XS, U13 PBQ76952PFBT, U14 FCX495, U2 MCU-MSM0G3507SPM, U4 ISO7721D, U5 ISO7721D, U6 TPD4E05U06DQA, U7 TPD4E05U06DQA, U8 TPD4E05U06DQA, U9 LMR51603XDBVR

Commit message: complete layout
Parts:
- removed D2: LED, LED_SMD:LED_0201_0603Metric_Pad0.64x0.40mm_HandSolder
- removed J15: Conn_01x02_Pin, Connector_PinHeader_2.54mm:PinHeader_1x02_P2.54mm_Vertical
- removed J2: Conn_02x05_Odd_Even, Connector_PinHeader_1.27mm:PinHeader_2x05_P1.27mm_Vertical_SMD
- removed R12: 700, Resistor_SMD:R_1206_3216Metric_Pad1.30x1.75mm_HandSolder
- removed TP10, TP11, TP13, TP17, TP21, TP22, TP23, TP25, TP27, TP28, TP8: TestPoint, TestPoint:TestPoint_Loop_D2.50mm_Drill1.0mm_LowProfile
- added C12: 220n, Capacitor_SMD:C_1206_3216Metric_Pad1.33x1.80mm_HandSolder, F.Cu at (126.8, 84.4)
- added C13: 220n, Capacitor_SMD:C_1206_3216Metric_Pad1.33x1.80mm_HandSolder, F.Cu at (157.3, 79.8)
- added C17: 100n, Capacitor_SMD:C_1206_3216Metric_Pad1.33x1.80mm_HandSolder, F.Cu at (150.7, 75.9)
- added J17: Conn_02x02_Odd_Even, Connector_PinHeader_2.54mm:PinHeader_2x02_P2.54mm_Vertical, F.Cu at (137.0, 69.4)
- added J5: Conn_01x09_Socket, Connector_PinHeader_2.54mm:PinHeader_1x09_P2.54mm_Vertical, F.Cu at (112.3, 59.4)
- added NT1: NetTie_2, NetTie:NetTie-2_SMD_Pad0.5mm, F.Cu at (116.9, 28.5)
- added SW2: SW_Push, Button_Switch_SMD:SW_SPST_PTS645, F.Cu at (159.6, 71.9)
- R1: value 200 -> 4.99k
- moved C4 146.7 mm to (169.1, 59.7)
- moved TP16 146.7 mm to (172.2, 91.2)
- moved C6 146.6 mm to (169.1, 62.2)
- moved C36 145.4 mm to (168.4, 42.8), turned to 180 degrees
- moved D3 141.9 mm to (165.3, 54.6), turned to -45 degrees
- moved R7 139.2 mm to (162.5, 79.8)
- moved R3 136.7 mm to (160.1, 90.1)
- moved C2 134.2 mm to (155.9, 59.9), turned to 90 degrees
- moved R2 133.7 mm to (157.3, 76.9), turned to 180 degrees
- moved C37 132.9 mm to (162.3, 42.8), turned to 180 degrees
- moved C1 132.4 mm to (153.4, 59.9), turned to 90 degrees
- moved R1 128.5 mm to (152.0, 68.9), turned to -90 degrees
- moved C48 126.8 mm to (161.8, 46.7), turned to 180 degrees
- moved C38 126.6 mm to (156.2, 42.8), turned to 180 degrees
- moved SW1 125.6 mm to (167.1, 84.7)
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Connections:
- net /BQ76952 16C/16P renamed +BATT
- C1 pad 2: GND -> -BATT
- C10 pad 2: Net-(Q2-S) -> Net-(D11-K)
- C11 pad 2: GND -> -BATT
- C14 pad 2: GND -> -BATT
- C15 pad 2: GND -> -BATT
- C2 pad 2: GND -> -BATT
- C22 pad 1: Net-(D11-A) -> Net-(JP4-A)
- C22 pad 2: Net-(Q2-S) -> Net-(D11-K)
- C3 pad 2: GND -> -BATT
- C35 pad 1: Net-(D11-A) -> Net-(JP4-A)
- C35 pad 2: Net-(Q2-S) -> Net-(D11-K)
- C4 pad 2: GND -> -BATT
- C47 pad 2: GND -> -BATT
- C5 pad 2: GND -> -BATT
- C56 pad 2: GND -> -BATT
- C57 pad 2: GND -> -BATT
- C6 pad 2: GND -> -BATT
- C7 pad 2: GND -> -BATT
- D1 pad 1: Net-(D1-K) -> -BATT
- D1 pad 2: VDD -> Net-(D1-A)
- D3 pad 2: GND -> -BATT
- D6 pad 1: Net-(D6-K) -> -BATT
- J1 pad 1: GND -> -BATT
- J3 pad 1: /GLV CAN TRX/CAN_VSS -> /GLV CAN TRX/CAN_L
- J3 pad 2: /GLV CAN TRX/CAN_L -> /GLV CAN TRX/CAN_H
- J3 pad 3: /GLV CAN TRX/CAN_H -> /GLV CAN TRX/CAN_VSS
- J4 pad 1: GND -> -BATT
- J6 pad 1: Net-(J6-Pin_1) -> PA15_I2C1_SCL
- J6 pad 2: Net-(J6-Pin_2) -> PA16_I2C1_SDA
- J7 pad 2: /BQ76952 16C/2P -> Net-(J7-Pin_2)
- JP4 pad 1: Net-(D11-A) -> Net-(JP4-A)
- L4 pad 2: Net-(D11-A) -> Net-(JP4-A)
- Q2 pad 2: Net-(Q2-S) -> Net-(D11-K)
- Q6 pad 1: PB26 -> PA21_A1_7_VREF-
- Q6 pad 3: /BQ0_3.3v -> onboard 3.3v src
- R1 pad 1: Net-(D2-K) -> onboard 3.3v src
- R11 pad 1: GND -> -BATT
- R15 pad 2: Net-(D11-A) -> Net-(JP4-A)
- R16 pad 1: PA19_SWDIO -> PA15_I2C1_SCL
- R17 pad 1: Net-(J6-Pin_1) -> Net-(J17-Pin_3)
- R18 pad 2: PA20_SWCLK -> PA16_I2C1_SDA
- R2 pad 1: GND -> -BATT
- R2 pad 2: PB26 -> PA21_A1_7_VREF-
- R26 pad 1: GND -> -BATT
- R3 pad 1: Net-(D6-K) -> PA14
- R3 pad 2: GND -> Net-(D6-A)
- R31 pad 1: Net-(D11-K) -> Net-(JP4-A)
- R31 pad 2: Net-(Q2-S) -> Net-(D11-A)
- R39 pad 1: Net-(Q2-S) -> Net-(D11-K)
- R4 pad 2: Net-(J6-Pin_2) -> Net-(J17-Pin_1)
- R5 pad 1: GND -> -BATT
- R6 pad 1: GND -> Net-(D1-A)
- R6 pad 2: Net-(D1-K) -> VDD
- R8 pad 1: GND -> -BATT
- SW1 pad 2: GND -> -BATT
- TH1 pad 1: /BQ76952 16C/TS1 -> /BQ76952 16C/DCHG
- TH1 pad 2: GND -> -BATT
- TH2 pad 1: /BQ76952 16C/TS2 -> /BQ76952 16C/DFETOFF
- TH2 pad 2: GND -> -BATT
- TH3 pad 1: /BQ76952 16C/TS3 -> /BQ76952 16C/CFETOFF
- TH3 pad 2: GND -> -BATT
- TH4 pad 1: /BQ76952 16C/HDQ -> /BQ76952 16C/DDSG
- TH4 pad 2: GND -> -BATT
- TH5 pad 1: /BQ76952 16C/DFETOFF -> /BQ76952 16C/HDQ
- TH5 pad 2: GND -> -BATT
- TH6 pad 1: /BQ76952 16C/DCHG -> /BQ76952 16C/ALERT
- TH6 pad 2: GND -> -BATT
- TH7 pad 1: /BQ76952 16C/DDSG -> /BQ76952 16C/TS1
- TH7 pad 2: GND -> -BATT
- TH8 pad 1: /BQ76952 16C/ALERT -> /BQ76952 16C/TS2
- TH8 pad 2: GND -> -BATT
- TH9 pad 1: /BQ76952 16C/CFETOFF -> /BQ76952 16C/TS3
- TH9 pad 2: GND -> -BATT
- TP14 pad 1: GND -> -BATT
- TP15 pad 1: GND -> -BATT
- TP16 pad 1: GND -> -BATT
- TP6 pad 1: Net-(D11-A) -> Net-(JP4-A)
- TP9 pad 1: GND -> -BATT
- U1 pad 5: GND -> -BATT
- U13 pad 17: GND -> -BATT
- U13 pad 35: /BQ0_3.3v -> onboard 3.3v src
- U2 pad 14: Net-(U2-PB17_A1_4) -> unconnected-(U2-PB17_A1_4-Pad14)
- U2 pad 16: Net-(U2-PB19_A1_6) -> unconnected-(U2-PB19_A1_6-Pad16)
- U2 pad 17: unconnected-(U2-PA21_A1_7_VREF--Pad17) -> PA21_A1_7_VREF-
- U2 pad 22: Net-(U2-PB23) -> unconnected-(U2-PB23-Pad22)
- U2 pad 26: Net-(U2-PA25_A0_2) -> unconnected-(U2-PA25_A0_2-Pad26)
- U2 pad 27: Net-(U2-PB25_A0_4) -> unconnected-(U2-PB25_A0_4-Pad27)
- U2 pad 29: Net-(D6-A) -> unconnected-(U2-PB27-Pad29)
- U2 pad 36: Net-(U2-PA29) -> unconnected-(U2-PA29-Pad36)
- U2 pad 41: GND -> -BATT
- U4 pad 5: GND -> -BATT
- U5 pad 5: GND -> -BATT
- U6 pad 1: PA11_UART0-RX_XDS -> PA10_UART0-TX_XDS
- U6 pad 2: PA10_UART0-TX_XDS -> RST_N
- U6 pad 3: GND -> -BATT
- U6 pad 4: RST_N -> PA19_SWDIO
- U6 pad 5: PA19_SWDIO -> PA20_SWCLK
- U6 pad 8: GND -> -BATT
- U7 pad 1: /XDS_3v_supply -> unconnected-(U7-D1+-Pad1)
- U7 pad 3: GND -> -BATT
- U7 pad 4: PA20_SWCLK -> /XDS_3v_supply
- U7 pad 5: /XDS_3v_supply -> PA11_UART0-RX_XDS
- U7 pad 8: GND -> -BATT
- U8 pad 1: /UART_USB/VBUS_5v -> unconnected-(U8-D1+-Pad1)
- U9 pad 2: Net-(Q2-S) -> Net-(D11-K)
Routing:
- net VDD: track 0.00 -> 107.4 mm, vias 0 -> 2
- net RST_N: track 0.00 -> 102.6 mm, vias 0 -> 1
- net PA20_SWCLK: track 0.00 -> 77.5 mm, vias 0 -> 1
- net PA19_SWDIO: track 0.00 -> 75.6 mm, vias 0 -> 1
- net onboard 3.3v src: track 0.00 -> 75.1 mm
- net PA10_UART0-TX_XDS: track 0.00 -> 65.9 mm, vias 0 -> 2
- net PA11_UART0-RX_XDS: track 0.00 -> 62.8 mm, vias 0 -> 2
- net /XDS_3v_supply: track 0.00 -> 47.6 mm
- net Net-(U13-VC16): track 0.00 -> 45.5 mm
- net PA15_I2C1_SCL: track 0.00 -> 41.6 mm
- net Net-(U13-VC15): track 0.00 -> 41.3 mm
- net /BQ76952 16C/BAT: track 0.00 -> 38.5 mm
- net Net-(U13-VC14): track 0.00 -> 38.4 mm
- net Net-(Q1-S): track 0.00 -> 38.4 mm
- net Net-(D11-K): track 0.00 -> 36.3 mm
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- added copper zone on B.Cu, net -BATT
- added copper zone on F.Cu, net -BATT
- added copper zone on B.Cu, net /BQ76952 16C/1N
- added copper zone on F.Cu, net /BQ76952 16C/1N
- added copper zone on B.Cu, net /GLV CAN TRX/CAN_VSS
- added copper zone on F.Cu, net /GLV CAN TRX/CAN_VSS
- added copper zone on B.Cu, net /UART_USB/GND
- added copper zone on F.Cu, net /UART_USB/GND
- added copper zone on B.Cu, net Net-(J7-Pin_2)
- added copper zone on F.Cu, net Net-(J7-Pin_2)
- added copper zone on F.Cu, net Net-(U2-VCORE)
- removed copper zone on B.Cu, net /BQ76952 16C/2P
- removed copper zone on B.Cu, net GND
- removed copper zone on F.Cu, net GND
Other:
- board text added: "12V-50V"
- board text added: "3v3"
- board text added: "BQ RST"
- board text added: "CAN_H"
- board text added: "CAN_L"
- board text added: "GND"
- board text added: "GND 5v 3v3 TXD RXD RESET_OUT TMS_SWDIO TCK_SWDCLK BLSi"
- board text added: "MCU RST"
- board text added: "SCL"
- board text added: "SDA"
- board text added: "XDS110 connector"
