File: hardware/EVAL MSPM0lG3507 BQ7962/EVAL MSPM0lG3507 BQ7962.kicad_sch (KiCad schematic)
At the start: 74 parts, among them J1 Conn_01x09_Socket, J10 Screw_Terminal_01x02, J11 Screw_Terminal_01x02, J12 Screw_Terminal_01x02, J13 Screw_Terminal_01x02, J14 Screw_Terminal_01x02, J15 Conn_01x02_Pin, J2 Conn_02x05_Odd_Even, J3 Conn_01x04_Pin, J4 Screw_Terminal_01x02, J6 Conn_01x02_Pin, J7 Screw_Terminal_01x02, J8 Screw_Terminal_01x02, J9 Screw_Terminal_01x02, Q6 2N7002, SW1 SW_Push, U2 MCU-MSM0G3507SPM, U6 TPD4E05U06DQA, U7 TPD4E05U06DQA

Commit message: complete layout
Parts:
- removed D2: LED, LED_SMD:LED_0201_0603Metric_Pad0.64x0.40mm_HandSolder, symbol Device:LED
- removed J15: Conn_01x02_Pin, Connector_PinHeader_2.54mm:PinHeader_1x02_P2.54mm_Vertical, symbol Connector:Conn_01x02_Pin
- removed R12: 700, Resistor_SMD:R_1206_3216Metric_Pad1.30x1.75mm_HandSolder, symbol Device:R_US
- removed TP10, TP11, TP13, TP17, TP21, TP22, TP23, TP25, TP27, TP28: TestPoint, TestPoint:TestPoint_Loop_D2.50mm_Drill1.0mm_LowProfile, symbol Connector:TestPoint
- added C12, C13: 220n, Capacitor_SMD:C_1206_3216Metric_Pad1.33x1.80mm_HandSolder, symbol Device:C_Small
- added C17: 100n, Capacitor_SMD:C_1206_3216Metric_Pad1.33x1.80mm_HandSolder, symbol Device:C_Small
- added J17: Conn_02x02_Odd_Even, Connector_PinHeader_2.54mm:PinHeader_2x02_P2.54mm_Vertical, symbol Connector_Generic:Conn_02x02_Odd_Even
- added J5: Conn_01x09_Socket, Connector_PinHeader_2.54mm:PinHeader_1x09_P2.54mm_Vertical, symbol Connector:Conn_01x09_Socket
- added NT1: NetTie_2, NetTie:NetTie-2_SMD_Pad0.5mm, symbol Device:NetTie_2
- added SW2: SW_Push, Button_Switch_SMD:SW_SPST_PTS645, symbol Switch:SW_Push
- J2: now not fitted; now left out of the parts list
- J6: now in the parts list
- R1: value 200 -> 4.99k; mouser https://www.mouser.com/ProductDetail/Panasonic/ERJ-P08J201V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 -> https://www.mouser.com/ProductDetail/SEI-Stackpole/RNCP1206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; specs 200Ohms, 660mW, 200PPM, 500V, 5%, -55C, +155C -> 4.99kOhm, 200V, 500mW, 1%, 100PPM, -55C, +155C; unit x10 (none) -> 0.017
Connections:
- net BQ0_3.3v is gone; now on net onboard 3.3v src: Q6.3 (D)
- net BQ76952 16C/16P is gone; now on net +BATT: J14.2 (Pin_2)
- net +3.3V: now also R6.2, C12.1, C13.1; no longer D1.2 (A)
- net -BATT: now also C11.2, C14.2, C15.2, C3.2, C5.2, D1.1 (K), D6.1 (K), J1.1 (Pin_1), J2.3 (Pin_3), J2.5 (Pin_5), J2.7 (Pin_7), J2.9 (Pin_9), J4.1 (Pin_1), R11.1, R2.1, R5.1, R8.1, SW1.2, TH1.2, TH2.2, TH3.2, TH4.2, TH5.2, TH6.2, TH7.2, TH8.2, TH9.2, TP14.1, TP15.1, TP16.1, TP9.1, U2.41 (VSS), U6.3 (GND), U6.8 (GND), U7.3 (GND), U7.8 (GND), C12.2, C13.2, C17.1
- net BQ76952 16C/2P: now also NT1.2; no longer J7.2 (Pin_2)
- net BQ76952 16C/ALERT: now also TH6.1, J5.4 (Pin_4); no longer TH8.1
- net BQ76952 16C/CFETOFF: now also TH3.1, J5.6 (Pin_6); no longer TH9.1
- net BQ76952 16C/DCHG: now also TH1.1, J5.8 (Pin_8); no longer TH6.1
- net BQ76952 16C/DDSG: now also TH4.1, J5.9 (Pin_9); no longer TH7.1
- net BQ76952 16C/DFETOFF: now also TH2.1, J5.7 (Pin_7); no longer TH5.1
- net BQ76952 16C/HDQ: now also TH5.1, J5.5 (Pin_5); no longer TH4.1
- net BQ76952 16C/TS1: now also TH7.1, J5.3 (Pin_3); no longer TH1.1
- net BQ76952 16C/TS2: now also TH8.1, J5.2 (Pin_2); no longer TH2.1
- net BQ76952 16C/TS3: now also TH9.1, J5.1 (Pin_1); no longer TH3.1
- net GLV CAN TRX/CAN_H: now also J3.2 (Pin_2); no longer J3.3 (Pin_3)
- net GLV CAN TRX/CAN_L: now also J3.1 (Pin_1); no longer J3.2 (Pin_2)
- net GLV CAN TRX/CAN_VSS: now also J3.3 (Pin_3); no longer J3.1 (Pin_1)
- net PA10_UART0-TX_XDS: now also U6.1 (D1+); no longer U6.2 (D1-)
- net PA11_UART0-RX_XDS: now also U7.5 (D2-); no longer U6.1 (D1+)
- net PA14: now also R3.1
- net PA15_I2C1_SCL: now also J6.1 (Pin_1), R16.1, J17.2 (Pin_2)
- net PA16_I2C1_SDA: now also J6.2 (Pin_2), R18.2, J17.4 (Pin_4)
- net PA19_SWDIO: now also U6.4 (D2+); no longer R16.1, U6.5 (D2-)
- net PA20_SWCLK: now also U6.5 (D2-); no longer R18.2, U7.4 (D2+)
- net PB26: no longer Q6.1 (G), R2.2
- net RST_N: now also U6.2 (D1-); no longer U6.4 (D2+)
- net XDS_3v_supply: now also U7.4 (D2+); no longer U7.1 (D1+), U7.5 (D2-)
- net onboard 3.3v src: now also R1.1
- net at R4.2: now also J17.1 (Pin_1); no longer J6.2 (Pin_2)
- net at R17.1: now also J17.3 (Pin_3); no longer J6.1 (Pin_1)
- net PA21_A1_7_VREF-: now reaches U2.17 (PA21_A1_7_VREF-)
- net PA21_A1_7_VREF-: now also Q6.1 (G), R2.2, C17.2, SW2.2
- net at U2.29 (PB27): no longer D6.2 (A)
- net at R1.2: now also SW2.1
- removed net GND: C11.2, C14.2, C15.2, C3.2, C5.2, J1.1 (Pin_1), J2.3 (Pin_3), J2.5 (Pin_5), J2.7 (Pin_7), J2.9 (Pin_9), J4.1 (Pin_1), R11.1, R2.1, R3.2, R5.1, R6.1, R8.1, SW1.2, TH1.2, TH2.2, TH3.2, TH4.2, TH5.2, TH6.2, TH7.2, TH8.2, TH9.2, TP14.1, TP15.1, TP16.1, TP9.1, U2.41 (VSS), U6.3 (GND), U6.8 (GND), U7.3 (GND), U7.8 (GND)
- new net: D1.2 (A), R6.1
- new net: J7.2 (Pin_2), NT1.1
- new net: D6.2 (A), R3.2
- no-connect marks 50 -> 57
Other:
- note added: "7/13/2025"
- note added: "Files at github.com/Gregification/BeeMS"
- note removed: "Files found at github.com/Gregification/BeeMS"
- moved on the sheet: D1, D6, J7, Q6, R11, R14, R16, R18, R2, R3, R50, R6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
