File: hardware/EVAL MSPM0lG3507 BQ7962/UART_USB.kicad_sch (KiCad schematic)
At the start: 1 part, among them U12 FT230XS

Commit message: mouser doom scrolling labor
Parts:
- added C8, C9: 220n, Capacitor_SMD:C_1206_3216Metric_Pad1.33x1.80mm_HandSolder, symbol Device:C_Small
- added J16: USB_B_Micro, symbol Connector:USB_B_Micro
- added Q2: ~, zzLocalLibraries-Footprints:SOT8001, symbol zzLocalLibrary:NX138BKHH
- added R49: 4.99k, Resistor_SMD:R_1206_3216Metric_Pad1.30x1.75mm_HandSolder, symbol Device:R_US
- added TP19: TestPoint, TestPoint:TestPoint_Loop_D2.50mm_Drill1.0mm_LowProfile, symbol Connector:TestPoint
- added U1, U4: ISO7721D, Package_SO:SOIC-8_3.9x4.9mm_P1.27mm, symbol Isolator:ISO7721D
- U12: mouser (none) -> https://www.mouser.com/ProductDetail/FTDI/FT230XS-U?qs=Gp1Y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; specs (none) -> USB x UART bridge, 1 chan
Connections:
- net at U12.1 (TXD): now also U1.2 (OUTA)
- net at U12.10 (3V3OUT): now also U12.3 (VCCIO), C9.1, R49.2, U1.1 (VCC1), U4.1 (VCC1)
- net VBUS_5v: now reaches U12.12 (VCC)
- net VBUS_5v: now also C8.1, J16.1 (VBUS), Q2.1 (G)
- net at U12.13 (GND): now also U12.5 (GND), C8.2, C9.2, Q2.2 (S), U1.4 (GND1), U4.4 (GND1)
- net at U12.2 (~{RTS}): now also U4.3 (INB)
- net at U12.4 (RXD): now also U1.3 (INB)
- net at U12.6 (~{CTS}): now also U4.2 (OUTA)
- net at U12.8 (USBDP): now also J16.3 (D+)
- net at U12.9 (USBDM): now also J16.2 (D-), R49.1
- new net: J16.6 (Shield), TP19.1
- new net CTS: U4.7 (INA)
- new net GND: J16.5 (GND), Q2.3 (D)
- new net RTS: U4.6 (OUTB)
- new net RXD: U1.6 (OUTB)
- new net TXD: U1.7 (INA)
- new net VDD: U1.8 (VCC2), U4.8 (VCC2)
- new net VSS: U4.5 (GND2)
- no-connect marks 0 -> 6
Other:
- note added: ""CBUS signal options" programmed using manufacturer software(see DS). things like high when TX, etc"
- note added: "ground if u r host. floating if u r peripheral"
- note added: "reverse polarity protection"
- moved on the sheet: U12

Commit message: ti once again making the most convenient IC's around
new TVS solution. use the
TPD4E05U06DQA
Parts:
- added Q3: ~, zzLocalLibraries-Footprints:SOT8001, symbol zzLocalLibrary:NX138BKHH
- added TP20, TP29, TP30, TP31: TestPoint, TestPoint:TestPoint_Loop_D2.50mm_Drill1.0mm_LowProfile, symbol Connector:TestPoint
- Q2: unit x10 (none) -> 0.052
- R49: mouser https://www.mouser.com/ProductDetail/YAGEO/RC1206FR-7W1K5L?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 -> https://www.mouser.com/ProductDetail/SEI-Stackpole/RNCP1206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; specs 1.5kOhm, 500mW, 200V, 1%, 100PPM, -55C, +155C -> 4.99kOhm, 200V, 500mW, 1%, 100PPM, -55C, +155C; unit x10 0.036 -> 0.017
Connections:
- net VDD: now also Q3.1 (G)
- net VSS: now also Q3.3 (D); no longer U4.5 (GND2)
- net at U1.2 (OUTA), U12.1 (TXD): now also TP20.1
- net at U1.3 (INB), U12.4 (RXD): now also TP29.1
- net at U1.5 (GND2): now also U4.5 (GND2), Q3.2 (S)
- net at U12.6 (~{CTS}), U4.2 (OUTA): now also TP30.1
- net at U12.2 (~{RTS}), U4.3 (INB): now also TP31.1
Other:
- note removed: "reverse polarity protection"

Commit message: corrected mosfet choice and started jumper board with xds110
Parts:
- removed Q2, Q3: ~, zzLocalLibraries-Footprints:SOT8001, symbol zzLocalLibrary:NX138BKHH
- added Q1: 2N7002, Package_TO_SOT_SMD:SOT-23, symbol Transistor_FET:2N7002
- added U8: TPD4E05U06DQA, Package_SON:USON-10_2.5x1.0mm_P0.5mm, symbol Power_Protection:TPD4E05U06DQA
Connections:
- net GND: now also Q1.2 (S), U8.3 (GND), U8.8 (GND)
- net VBUS_5v: now also Q1.1 (G), U8.1 (D1+)
- net VSS: now also U1.5 (GND2), U4.5 (GND2)
- net at C8.2, C9.2, U1.4 (GND1)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: now also Q1.3 (D)
- net D-: now reaches J16.2 (D-), R49.1, U12.9 (USBDM)
- net D-: now also U8.5 (D2-)
- net D+: now reaches J16.3 (D+), U12.8 (USBDP)
- net D+: now also U8.4 (D2+)
- no-connect marks 6 -> 11
Other:
- moved on the sheet: C8, C9, J16, R49, TP19, TP20, TP29, TP30, TP31, U1, U12, U4

Commit message: indicated layout so someone else can do it
Parts:
- J16: footprint (none) -> Connector_USB:USB_Micro-B_Amphenol_10118194-0001LF_Horizontal; mouser (none) -> https://www.mouser.com/ProductDetail/Amphenol-FCI/10118194-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; specs (none) -> 1GOhm isolation allegedly; unit x10 (none) -> 0.363
Connections:
- net GND: now also Q1.3 (D); no longer Q1.2 (S)
- net VBUS_5v: no longer U8.1 (D1+)
- net at C8.2, C9.2, U1.4 (GND1)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: now also Q1.2 (S); no longer Q1.3 (D)
Other:
- moved on the sheet: C8, C9, J16, Q1, R49, TP19, TP20, TP29, TP30, TP31, U1, U12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

Commit message: complete layout
Connections:
- net GND: now also C8.2, C9.2, Q1.2 (S), U1.4 (GND1), U12.13 (GND), U12.5 (GND), U4.4 (GND1); no longer J16.5 (GND), Q1.3 (D)
- new net: J16.5 (GND), Q1.3 (D)
- no-connect marks 11 -> 12
Changed lines of the file:
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@@
+	)
+	(no_connect
+		(at 46.99 52.07)
 	)
 	(no_connect
@@
 	)
 	(label "GND"
-		(at 50.8 123.19 0)
+		(at 101.6 123.19 0)
 		(effects
 			(font
