File: hardware/HC ohm tester/HC ohm tester.kicad_pcb (KiCad board)
At the start: 2 copper layers, 35 parts, among them J1 Conn_01x02_Pin, J2 Conn_01x02_Pin, J3 Conn_01x02_Pin, J4 DCPS+, J5 Conn_01x08_Pin, Q1 NTMFS0D8N03C, Q2 NTMFS0D8N03C, Q3 NTMFS0D8N03C, Q4 2N7002K, Q5 NTMFS0D8N03C, U1 MCP3550-50-EMS, U2 MCP3550-50-EMS, U3 AP63205WU, U4 ISO7731FQDBQQ1, U5 AZ1117-5.0, U6 ISO7730FQDBQQ1

Commit message: big relay alternative
Parts:
- removed C1, C6: 100n, Capacitor_SMD:C_1206_3216Metric_Pad1.33x1.80mm_HandSolder
- removed C2: 10u, Capacitor_SMD:C_1206_3216Metric_Pad1.33x1.80mm_HandSolder
- removed C3, C4, C5, C7: 22u, Capacitor_SMD:C_1206_3216Metric_Pad1.33x1.80mm_HandSolder
- removed J1, J2, J3: Conn_01x02_Pin, Connector_PinHeader_2.54mm:PinHeader_1x02_P2.54mm_Vertical
- removed J4: DCPS+, MountingHole:MountingHole_3mm_Pad_TopBottom
- removed J5: Conn_01x08_Pin, Connector_PinHeader_2.54mm:PinHeader_1x08_P2.54mm_Vertical
- removed J6: ~, MountingHole:MountingHole_3mm_Pad_TopBottom
- removed JP1, JP2, JP3, JP4: SolderJumper_2_Open, Jumper:SolderJumper-2_P1.3mm_Open_RoundedPad1.0x1.5mm
- removed L1: 4.7u, Inductor_SMD:L_0201_0603Metric_Pad0.64x0.40mm_HandSolder
- removed Q1, Q2, Q3, Q5: NTMFS0D8N03C, Package_SO:ONSemi_SO-8FL_488AA
- removed Q4: 2N7002K, Package_TO_SOT_SMD:SOT-23
- removed R1, R2, R3, R4, R5, R6: ~50k, Resistor_SMD:R_1206_3216Metric_Pad1.30x1.75mm_HandSolder
- removed U1, U2: MCP3550-50-EMS, Package_SO:MSOP-8_3x3mm_P0.65mm
- removed U3: AP63205WU, Package_TO_SOT_SMD:TSOT-23-6
- removed U4: ISO7731FQDBQQ1, HC_ohm_tester:DBQ16_TEX-M
- removed U5: AZ1117-5.0, Package_TO_SOT_SMD:SOT-223-3_TabPin2
- removed U6: ISO7730FQDBQQ1, HC_ohm_tester:DBQ16_TEX-M
Routing:
- net Net-(Q1-G): track 25.9 -> 0.00 mm
- removed copper zone on B.Cu, net /DCPS+
- removed copper zone on F.Cu, net /DCPS+
- removed copper zone on B.Cu, net /HC out
- removed copper zone on F.Cu, net /HC out

Commit message: final revision A
board shipped using GDL, "across the globe eventually" at the small price of $5
Parts:
- added C1: 100n, Capacitor_SMD:C_1206_3216Metric_Pad1.33x1.80mm_HandSolder, F.Cu at (169.8, 77.6)
- added C2: 10u, Capacitor_SMD:C_1206_3216Metric_Pad1.33x1.80mm_HandSolder, F.Cu at (171.6, 72.1)
- added C3: 22u, Capacitor_SMD:C_1206_3216Metric_Pad1.33x1.80mm_HandSolder, F.Cu at (164.3, 85.6)
- added C4: 22u, Capacitor_SMD:C_1206_3216Metric_Pad1.33x1.80mm_HandSolder, F.Cu at (171.1, 84.0)
- added C5: 22u, Capacitor_SMD:C_1206_3216Metric_Pad1.33x1.80mm_HandSolder, F.Cu at (154.9, 70.0)
- added C6: 100n, Capacitor_SMD:C_1206_3216Metric_Pad1.33x1.80mm_HandSolder, F.Cu at (152.7, 95.8)
- added C7: 22u, Capacitor_SMD:C_1206_3216Metric_Pad1.33x1.80mm_HandSolder, F.Cu at (170.2, 86.8)
- added J1: Conn_01x02_Pin, Connector_PinHeader_2.54mm:PinHeader_1x02_P2.54mm_Vertical, F.Cu at (174.6, 70.2)
- added J2: Conn_01x02_Pin, Connector_PinHeader_2.54mm:PinHeader_1x02_P2.54mm_Vertical, F.Cu at (151.2, 103.7)
- added J3: Conn_01x02_Pin, Connector_PinHeader_2.54mm:PinHeader_1x02_P2.54mm_Vertical, F.Cu at (151.2, 90.4)
- added J4: DCPS+, MountingHole:MountingHole_3mm_Pad_TopBottom, F.Cu at (153.1, 62.2)
- added J5: Conn_01x08_Pin, Connector_PinHeader_2.54mm:PinHeader_1x08_P2.54mm_Vertical, F.Cu at (174.6, 86.9)
- added J6: ~, MountingHole:MountingHole_3mm_Pad_TopBottom, F.Cu at (172.5, 62.1)
- added JP1: SolderJumper_2_Open, Jumper:SolderJumper-2_P1.3mm_Open_RoundedPad1.0x1.5mm, F.Cu at (154.7, 87.9)
- added JP2: SolderJumper_2_Open, Jumper:SolderJumper-2_P1.3mm_Open_RoundedPad1.0x1.5mm, F.Cu at (154.7, 90.5)
- added JP3: SolderJumper_2_Open, Jumper:SolderJumper-2_P1.3mm_Open_RoundedPad1.0x1.5mm, F.Cu at (154.7, 103.7)
- added JP4: SolderJumper_2_Open, Jumper:SolderJumper-2_P1.3mm_Open_RoundedPad1.0x1.5mm, F.Cu at (154.7, 101.1)
- added L1: 4.7u, Inductor_SMD:L_0603_1608Metric_Pad1.05x0.95mm_HandSolder, F.Cu at (173.2, 79.3)
- added Q1: 2N3904, Package_TO_SOT_THT:TO-92_Inline, F.Cu at (161.7, 70.9)
- added Q3: NTMFS0D8N03C, Package_SO:ONSemi_SO-8FL_488AA, F.Cu at (162.7, 62.0)
- added R1: ~50k, Resistor_SMD:R_1206_3216Metric_Pad1.30x1.75mm_HandSolder, F.Cu at (166.1, 70.3)
- added R2: ~50k, Resistor_SMD:R_1206_3216Metric_Pad1.30x1.75mm_HandSolder, F.Cu at (166.7, 97.0)
- added R3: ~50k, Resistor_SMD:R_1206_3216Metric_Pad1.30x1.75mm_HandSolder, F.Cu at (170.7, 96.9)
- added R6: ~50k, Resistor_SMD:R_1206_3216Metric_Pad1.30x1.75mm_HandSolder, F.Cu at (154.9, 72.5)
- added U1: MCP3550-50-EMS, Package_SO:MSOP-8_3x3mm_P0.65mm, F.Cu at (159.7, 89.0)
- added U2: MCP3550-50-EMS, Package_SO:MSOP-8_3x3mm_P0.65mm, F.Cu at (159.8, 102.2)
- added U3: AP63205WU, Package_TO_SOT_SMD:TSOT-23-6, F.Cu at (173.1, 76.7)
- added U4: ISO7731FQDBQQ1, HC_ohm_tester:DBQ16_TEX-M, F.Cu at (167.6, 102.8)
- added U5: AZ1117-5.0, Package_TO_SOT_SMD:SOT-223-3_TabPin2, F.Cu at (158.5, 95.7)
- added U6: ISO7730FQDBQQ1, HC_ohm_tester:DBQ16_TEX-M, F.Cu at (168.6, 91.3)
Routing:
- net +5V: track 0.00 -> 73.2 mm, vias 0 -> 5
- net /HS active: track 0.00 -> 31.0 mm, vias 0 -> 2
- net /+5Vref: track 0.00 -> 28.7 mm, vias 0 -> 2
- net GND: track 0.00 -> 26.1 mm, vias 0 -> 91
- net Net-(U1-SDO/~{RDY}): track 0.00 -> 24.3 mm, vias 0 -> 2
- net /Vio: track 0.00 -> 23.8 mm
- net Net-(U1-SCK): track 0.00 -> 20.4 mm
- net Net-(U4-EN1): track 0.00 -> 18.5 mm
- net /DCPS+: track 0.00 -> 17.0 mm, vias 0 -> 14
- net Net-(U2-~{CS}): track 0.00 -> 14.7 mm
- net Net-(Q1-E): track 0.00 -> 14.2 mm
- net Net-(U4-EN2): track 0.00 -> 8.62 mm
- net Net-(J1-Pin_2): track 0.00 -> 7.95 mm
- net /ADC2 CS: track 0.00 -> 6.74 mm
- net /GNDio: track 0.00 -> 5.87 mm, vias 0 -> 12
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- added copper zone on B.Cu, net /DCPS+
- added copper zone on F.Cu, net /DCPS+
- added copper zone on B.Cu, net /GNDio
- added copper zone on F.Cu, net /GNDio
- added copper zone on B.Cu, net GND
- added copper zone on F.Cu, net GND
Other:
- board outline added: 27.1 x 48.3 mm
- board text added: "+-5V abs MAX"
- board text added: "<1mOhm meter : LS driver : 2x +-5V 22b ADC : J5 isolated : requires external flyback protection"
- board text added: "ADC model: MCP3550"
- board text added: "ADC1 CS ADC2 CS ADC2 SDO/RDY"
- board text added: "ADC1 SDO/RDY SCK"
- board text added: "ADC1+ ADC1-"
- board text added: "ADC2+ ADC2-"
- board text added: "LS Switch +"
- board text added: "LS Switch - (PWR GND)"
- board text added: "SIG GND VDD [3.8V, 32V]"
- board text added: "Vio [0,5V] GND LS SW on/off AH"
- board text added: "eyeballed the layout. probably could be better"
- board text added: "github.com/Gregification/BeeMS /tree/main/hardware/HC ohm tester"
