File: hardware/HV_Sensor/HV_Sensor/HV_Sensor.kicad_sch (KiCad schematic)
At the start: 27 parts, among them J1 Conn_01x09_Socket, J2 Conn_02x05_Odd_Even, J3 Conn_01x04_Pin, SW1 SW_Push, U2 MCU-MSM0G3507SPM

Commit message: Update HV_Sensor.kicad_sch
Parts:
- added U4: AMC3330DWE, zzLocalLibraries-Footprints:SOIC_30DWER_TEX-M, symbol zzLocalLibrary:AMC3330DWE
Other:
- moved on the sheet: C12, C13, C3, C7, D3, J1, J2, J3, R1, R7, SW1, TP14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
