File: hardware/EVAL MSPM0lG3507 BQ76952/EVAL MSPM0lG3507 BQ76952.kicad_pcb (KiCad board)
At the start: 2 copper layers, 72.2 x 76.8 mm, 115 parts, among them J1 Conn_01x09_Socket, J10 Screw_Terminal_01x02, J11 Screw_Terminal_01x02, J12 Screw_Terminal_01x02, J13 Screw_Terminal_01x02, J14 Screw_Terminal_01x02, J15 Conn_02x04_Odd_Even, J16 USB_B_Micro, J18 Conn_01x17_Socket, J19 Screw_Terminal_01x02, J2 Conn_02x05_Odd_Even, J3 Conn_01x04_Socket, J4 Screw_Terminal_01x02, J5 Conn_01x07_Pin, J7 Screw_Terminal_01x02, J8 Screw_Terminal_01x02, J9 Screw_Terminal_01x02, Q6 2N7002, SW1 SW_Push, SW2 SW_Push, U1 MCP6L01Rx-xOT, U10 MCP2542FDxMF, U12 FT230XS, U13 PBQ76952PFBT, U14 FCX495, U2 MCU-MSM0G3507SPM, U3 STISO620, U4 RAA211805, U5 STISO620

Commit message: changes...awaiting oversight
Parts:
- added J18: Conn_01x04_Socket, Connector_PinHeader_2.54mm:PinHeader_1x04_P2.54mm_Vertical, F.Cu at (167.5, 103.0)
- added R10: 97.6k, Resistor_SMD:R_0805_2012Metric_Pad1.20x1.40mm_HandSolder, F.Cu at (195.5, 79.0)
- added R12: 97.6k, Resistor_SMD:R_0805_2012Metric_Pad1.20x1.40mm_HandSolder, F.Cu at (166.5, 83.0)
- added R13: 97.6k, Resistor_SMD:R_0805_2012Metric_Pad1.20x1.40mm_HandSolder, F.Cu at (177.5, 76.0)
- added R17: 24.9, Resistor_SMD:R_0805_2012Metric_Pad1.20x1.40mm_HandSolder, F.Cu at (201.5, 44.2)
- added R18: 24.9, Resistor_SMD:R_0805_2012Metric_Pad1.20x1.40mm_HandSolder, F.Cu at (201.5, 47.1)
- added R19: 24.9, Resistor_SMD:R_0805_2012Metric_Pad1.20x1.40mm_HandSolder, F.Cu at (201.5, 50.1)
- added R20: 24.9, Resistor_SMD:R_0805_2012Metric_Pad1.20x1.40mm_HandSolder, F.Cu at (201.5, 53.0)
- added R21: 24.9, Resistor_SMD:R_0805_2012Metric_Pad1.20x1.40mm_HandSolder, F.Cu at (201.5, 56.0)
- added R22: 24.9, Resistor_SMD:R_0805_2012Metric_Pad1.20x1.40mm_HandSolder, F.Cu at (206.2, 44.2)
- added R23: 24.9, Resistor_SMD:R_0805_2012Metric_Pad1.20x1.40mm_HandSolder, F.Cu at (206.2, 47.1)
- added R24: 24.9, Resistor_SMD:R_0805_2012Metric_Pad1.20x1.40mm_HandSolder, F.Cu at (206.2, 50.1)
- added R25: 24.9, Resistor_SMD:R_0805_2012Metric_Pad1.20x1.40mm_HandSolder, F.Cu at (206.2, 53.0)
- added R26: 24.9, Resistor_SMD:R_0805_2012Metric_Pad1.20x1.40mm_HandSolder, F.Cu at (206.2, 56.0)
- added R27: 24.9, Resistor_SMD:R_0805_2012Metric_Pad1.20x1.40mm_HandSolder, F.Cu at (211.0, 44.2)
- added R28: 24.9, Resistor_SMD:R_0805_2012Metric_Pad1.20x1.40mm_HandSolder, F.Cu at (211.0, 47.1)
- added R29: 24.9, Resistor_SMD:R_0805_2012Metric_Pad1.20x1.40mm_HandSolder, F.Cu at (211.0, 50.1)
- added R30: 24.9, Resistor_SMD:R_0805_2012Metric_Pad1.20x1.40mm_HandSolder, F.Cu at (211.0, 53.0)
- added R31: 24.9, Resistor_SMD:R_0805_2012Metric_Pad1.20x1.40mm_HandSolder, F.Cu at (211.0, 56.0)
- added R32: 24.9, Resistor_SMD:R_0805_2012Metric_Pad1.20x1.40mm_HandSolder, F.Cu at (215.8, 44.2)
- added R33: 24.9, Resistor_SMD:R_0805_2012Metric_Pad1.20x1.40mm_HandSolder, F.Cu at (215.8, 47.1)
- added R35: 3.32k, Resistor_SMD:R_0805_2012Metric_Pad1.20x1.40mm_HandSolder, F.Cu at (215.8, 50.1)
- added R36: 3.32k, Resistor_SMD:R_0805_2012Metric_Pad1.20x1.40mm_HandSolder, F.Cu at (215.8, 53.0)
- added R37: 3.32k, Resistor_SMD:R_0805_2012Metric_Pad1.20x1.40mm_HandSolder, F.Cu at (215.8, 56.0)
- added R5: 3.32k, Resistor_SMD:R_0805_2012Metric_Pad1.20x1.40mm_HandSolder, F.Cu at (182.0, 65.5)
- added R6: 97.6k, Resistor_SMD:R_0805_2012Metric_Pad1.20x1.40mm_HandSolder, F.Cu at (182.0, 59.5)
- added R7: 3.32k, Resistor_SMD:R_0805_2012Metric_Pad1.20x1.40mm_HandSolder, F.Cu at (196.5, 67.5)
- added R8: 3.32k, Resistor_SMD:R_0805_2012Metric_Pad1.20x1.40mm_HandSolder, F.Cu at (144.5, 73.0)
- added TP1: TestPoint, TestPoint:TestPoint_Loop_D2.50mm_Drill1.0mm_LowProfile, F.Cu at (161.0, 66.0)
- added TP2: TestPoint, TestPoint:TestPoint_Loop_D2.50mm_Drill1.0mm_LowProfile, F.Cu at (108.5, 104.5)
- R14: renamed from R10; value 750 -> 3.32k; footprint Resistor_SMD:R_1206_3216Metric_Pad1.30x1.75mm_HandSolder -> Resistor_SMD:R_0805_2012Metric_Pad1.20x1.40mm_HandSolder
- renumbered C17 to C1, C4 to C10, C30 to C11, C36 to C12, C37 to C13, C38 to C14, C42 to C15, C43 to C16, C44 to C17, C45 to C18, C46 to C19, C12 to C2, C47 to C20, C34 to C21, C48 to C22, C49 to C23, C50 to C24, C51 to C25, C52 to C26, C53 to C27, C54 to C28, C55 to C29, C13 to C3, C57 to C30, C2 to C31, C1 to C32, C14 to C4, C11 to C5, C5 to C6, C3 to C7, C6 to C8, C10 to C9, D4 to D2, D2 to D3, D5 to D4, D3 to D6, J2 to J1, J4 to J10, J19 to J11, J5 to J13, J15 to J14, J3 to J16, J16 to J17, J14 to J2, J13 to J3, J12 to J4, J11 to J5, J10 to J6, J9 to J7, J7 to J9, R14 to R1, R3 to R11, R25 to R15, R26 to R16, R4 to R2, R13 to R3, R12 to R34, R17 to R4, R8 to R9, SW2 to SW1, SW1 to SW2, TP14 to TP3, TP16 to TP4, TP9 to TP5, U2 to U1, U5 to U2, U4 to U3, U10 to U4, U12 to U5, U3 to U6, U13 to U7, U14 to U8
Connections:
- C1 pad 2: Net-(Q6-G) -> Net-(C1-Pad2)
- C11 pad 1: Net-(D6-COM) -> Net-(U7-SRP)
- C11 pad 2: Net-(D7-COM) -> Net-(U7-SRN)
- C12 pad 1: Net-(U13-VC16) -> Net-(U7-VC16)
- C12 pad 2: Net-(U13-VC15) -> Net-(U7-VC15)
- C13 pad 1: Net-(U13-VC14) -> Net-(U7-VC14)
- C13 pad 2: Net-(U13-VC13) -> Net-(U7-VC13)
- C14 pad 1: Net-(U13-VC12) -> Net-(U7-VC12)
- C14 pad 2: Net-(U13-VC11) -> Net-(U7-VC11)
- C15 pad 1: Net-(U13-VC10) -> Net-(U7-VC10)
- C15 pad 2: Net-(U13-VC9) -> Net-(U7-VC9)
- C16 pad 1: Net-(U13-VC8) -> Net-(U7-VC8)
- C16 pad 2: Net-(U13-VC7) -> Net-(U7-VC7)
- C17 pad 1: Net-(U13-VC6) -> Net-(U7-VC6)
- C17 pad 2: Net-(U13-VC5) -> Net-(U7-VC5)
- C18 pad 1: Net-(U13-VC4) -> Net-(U7-VC4)
- C18 pad 2: Net-(U13-VC3) -> Net-(U7-VC3)
- C19 pad 1: Net-(U13-VC2) -> Net-(U7-VC2)
- C19 pad 2: Net-(U13-VC1) -> Net-(U7-VC1)
- C20 pad 1: Net-(U13-VC0) -> Net-(U7-VC0)
- C21 pad 1: Net-(D6-COM) -> Net-(U7-SRP)
- C21 pad 2: Net-(D7-COM) -> Net-(U7-SRN)
- C22 pad 1: Net-(U13-VC15) -> Net-(U7-VC15)
- C22 pad 2: Net-(U13-VC14) -> Net-(U7-VC14)
- C23 pad 1: Net-(U13-VC13) -> Net-(U7-VC13)
- C23 pad 2: Net-(U13-VC12) -> Net-(U7-VC12)
- C24 pad 1: Net-(U13-VC11) -> Net-(U7-VC11)
- C24 pad 2: Net-(U13-VC10) -> Net-(U7-VC10)
- C25 pad 1: Net-(U13-VC9) -> Net-(U7-VC9)
- C25 pad 2: Net-(U13-VC8) -> Net-(U7-VC8)
- C26 pad 1: Net-(U13-VC7) -> Net-(U7-VC7)
- C26 pad 2: Net-(U13-VC6) -> Net-(U7-VC6)
- C27 pad 1: Net-(U13-VC5) -> Net-(U7-VC5)
- C27 pad 2: Net-(U13-VC4) -> Net-(U7-VC4)
- C28 pad 1: Net-(U13-VC3) -> Net-(U7-VC3)
- C28 pad 2: Net-(U13-VC2) -> Net-(U7-VC2)
- C29 pad 1: Net-(U13-VC1) -> Net-(U7-VC1)
- C30 pad 1: Net-(U1-+) -> Net-(U7-REG18)
- D6 pad 1: Net-(D3-K) (its old number) -> Net-(D6-K)
- J10 pad 2: -BATT -> /BQ76952 16C/1N
- J16 pad 1: /GLV interface/GLV+ -> /GLV interface/GLV-
- J16 pad 2: /GLV interface/CAN_H -> /GLV interface/GLV+
- J16 pad 3: /GLV interface/CAN_L -> /GLV interface/CAN_H
- J16 pad 4: /GLV interface/GLV- -> /GLV interface/CAN_L
- R15 pad 2: Net-(D6-COM) -> Net-(U7-SRP)
- R16 pad 2: Net-(D7-COM) -> Net-(U7-SRN)
- R34 pad 1: Net-(D3-K) (its old number) -> Net-(D6-K)
- SW1 pad 2: Net-(Q6-G) -> Net-(C1-Pad2)
- U2 pad 1: VDD -> -BATT
- U2 pad 4: -BATT -> VDD
- U2 pad 5: /GLV interface/GLV- -> /GLV interface/5v
- U2 pad 6: Net-(U10-RXD) -> Net-(U2-RXA)
- U2 pad 7: Net-(U10-TXD) -> Net-(U2-TXB)
- U2 pad 8: /GLV interface/5v -> /GLV interface/GLV-
- U3 pad 3: Net-(U4-EN) -> Net-(U3-EN)
- U4 pad 1: Net-(U10-TXD) -> Net-(U2-RXA)
- U4 pad 4: Net-(U10-RXD) -> Net-(U2-TXB)
- U4 pad 8: Net-(U10-STBY) -> Net-(U4-STBY)
- U7 pad 1: Net-(U13-VC15) -> Net-(U7-VC15)
- U7 pad 10: Net-(U13-VC6) -> Net-(U7-VC6)
- U7 pad 11: Net-(U13-VC5) -> Net-(U7-VC5)
- U7 pad 12: Net-(U13-VC4) -> Net-(U7-VC4)
- U7 pad 13: Net-(U13-VC3) -> Net-(U7-VC3)
- U7 pad 14: Net-(U13-VC2) -> Net-(U7-VC2)
- U7 pad 15: Net-(U13-VC1) -> Net-(U7-VC1)
- U7 pad 16: Net-(U13-VC0) -> Net-(U7-VC0)
- U7 pad 18: Net-(D6-COM) -> Net-(U7-SRP)
- U7 pad 2: Net-(U13-VC14) -> Net-(U7-VC14)
- U7 pad 20: Net-(D7-COM) -> Net-(U7-SRN)
- U7 pad 24: Net-(U1-+) -> Net-(U7-REG18)
- U7 pad 3: Net-(U13-VC13) -> Net-(U7-VC13)
- U7 pad 4: Net-(U13-VC12) -> Net-(U7-VC12)
- U7 pad 41: Net-(U13-LD) -> Net-(U7-LD)
- U7 pad 42: Net-(U13-PACK) -> Net-(U7-PACK)
- U7 pad 48: Net-(U13-VC16) -> Net-(U7-VC16)
- U7 pad 5: Net-(U13-VC11) -> Net-(U7-VC11)
- U7 pad 6: Net-(U13-VC10) -> Net-(U7-VC10)
- U7 pad 7: Net-(U13-VC9) -> Net-(U7-VC9)
- U7 pad 8: Net-(U13-VC8) -> Net-(U7-VC8)
- U7 pad 9: Net-(U13-VC7) -> Net-(U7-VC7)
- U8 pad 2: +BATT -> /BQ76952 16C/BAT
Routing:
- net (no net): track 0.00 -> 18.9 mm
- net Net-(J17-D-): track 13.2 -> 0.00 mm
- net Net-(U10-TXD): track 2.90 -> 0.00 mm
- net Net-(U10-RXD): track 2.89 -> 0.00 mm
- net Net-(D6-K): track 15.5 -> 18.1 mm
- net Net-(D3-K) (its old number): track 2.60 -> 0.00 mm
- net /BQ76952 16C/1N: track 0.00 -> 0.70 mm
- net -BATT: track 55.0 -> 54.3 mm
Other:
- board size 72.2 x 76.8 mm -> 72.2 x 83.8 mm

Commit message: changed
Parts:
- moved R7 82.7 mm to (116.0, 86.5)
Changed lines of the file:
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@@
 	(footprint "Resistor_SMD:R_0805_2012Metric_Pad1.20x1.40mm_HandSolder"
 		(layer "F.Cu")
-		(at 196.5 67.5)
+		(at 116 86.5)
 		(descr "Resistor SMD 0805 (2012 Metric), square (rectangular) end terminal, IPC-7351 nominal with elongated pad for handsoldering. (Body size source: IPC-SM-782 page 72, https://www.pcb-3d.com/wordpress/wp-content/uploads/ipc-sm-782a_amendment_1_and_2.pdf), generated with kicad-footprint-generator")
 		(tags "resistor handsolder")

Commit message: updating PCB
Parts:
- moved J18 14.8 mm to (153.0, 100.5), turned to 90 degrees
- moved D4 9.52 mm to (164.1, 100.5), turned to 0 degrees
- moved TP2 3.50 mm to (108.5, 101.0)
- moved R14 2.72 mm to (164.9, 97.4), turned to -90 degrees
Routing:
- net Net-(J17-D-): track 0.00 -> 17.1 mm, vias 0 -> 1
- net (no net): track 18.9 -> 5.79 mm
- net /XDS_3v_supply: track 26.0 -> 30.5 mm
- net Net-(J17-D+): track 22.1 -> 26.2 mm, vias 0 -> 1
- net /UART_USB/5V: track 35.5 -> 38.0 mm

Commit message: EDITING EVAL
Parts:
- moved TP1 57.0 mm to (104.5, 73.5)
- moved R7 4.92 mm to (114.0, 82.0), turned to -45 degrees
- moved D1 1.21 mm to (113.0, 83.5)
- moved R13 0.50 mm to (177.0, 76.0)
Routing:
- net VDD: track 68.8 -> 71.4 mm
- net Net-(D1-A): track 3.29 -> 4.36 mm
Changed lines of the file:
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@@
 		(tags "test point wire loop bead")
 		(property "Reference" "TP12"
-			(at -0.1 -3.8 0)
+			(at 2.5 0 180)
 			(layer "F.SilkS")
 			(effects
@@
 	(footprint "Resistor_SMD:R_0805_2012Metric_Pad1.20x1.40mm_HandSolder"
 		(layer "F.Cu")
-		(at 177.5 76 -90)
+		(at 177 76 -90)
 		(descr "Resistor SMD 0805 (2012 Metric), square (rectangular) end terminal, IPC-7351 nominal with elongated pad for handsoldering. (Body size source: IPC-SM-782 page 72, https://www.pcb-3d.com/wordpress/wp-content/uploads/ipc-sm-782a_amendment_1_and_2.pdf), generated with kicad-footprint-generator")
 		(tags "resistor handsolder")
@@
 	(footprint "LED_SMD:LED_0603_1608Metric"
 		(layer "F.Cu")
-		(at 113.5 82.4 -45)
+		(at 113 83.5 -45)
 		(descr "LED SMD 0603 (1608 Metric), square (rectangular) end terminal, IPC-7351 nominal, (Body size source: http://www.tortai-tech.com/upload/download/2011102023233369053.pdf), generated with kicad-footprint-generator")
 		(tags "LED")
@@
 	(footprint "Resistor_SMD:R_0805_2012Metric_Pad1.20x1.40mm_HandSolder"
 		(layer "F.Cu")
-		(at 116 86.5)
+		(at 114 82 -45)
 		(descr "Resistor SMD 0805 (2012 Metric), square (rectangular) end terminal, IPC-7351 nominal with elongated pad for handsoldering. (Body size source: IPC-SM-782 page 72, https://www.pcb-3d.com/wordpress/wp-content/uploads/ipc-sm-782a_amendment_1_and_2.pdf), generated with kicad-footprint-generator")
 		(tags "resistor handsolder")
 		(property "Reference" "R7"
-			(at 0 -1.65 0)
+			(at 0 -1.65 135)
 			(layer "F.SilkS")
 			(effects
@@
 		)
 		(property "Value" "3.32k"
-			(at 0 1.65 0)
+			(at 0 1.65 135)
 			(layer "F.Fab")
 			(effects
@@
 		)
 		(property "Datasheet" ""
-			(at 0 0 0)
+			(at 0 0 135)
 			(layer "F.Fab")
 			(hide yes)
@@
 		)
 		(property "Description" "Resistor, US symbol"
-			(at 0 0 0)
+			(at 0 0 135)
 			(layer "F.Fab")
 			(hide yes)
@@
 		)
 		(property "Sim.Device" ""
-			(at 0 0 0)
+			(at 0 0 315)
 			(unlocked yes)
 			(layer "F.Fab")
@@
 		)
 		(property "Sim.Type" ""
-			(at 0 0 0)
+			(at 0 0 315)
 			(unlocked yes)
 			(layer "F.Fab")
@@
 		)
 		(property "mouser" "https://www.mouser.com/ProductDetail/Walsin/WR08X3321FTL?qs=sGAEpiMZZMvdGkrng054twKDKoBh%252BscnhzVUopLjNIsmzZlnTa4U1w%3D%3D"
-			(at 0 0 0)
+			(at 0 0 315)
 			(unlocked yes)
 			(layer "F.Fab")
@@
 		)
 		(property "specs" "3.32kOhm, 1%, 150V, 125mW, 100ppm, -55C, 155C"
-			(at 0 0 0)
+			(at 0 0 315)
 			(unlocked yes)
 			(layer "F.Fab")
@@
 		)
 		(property "unit x10" "0.019"
-			(at 0 0 0)
+			(at 0 0 315)
 			(unlocked yes)
 			(layer "F.Fab")
@@
 		)
 		(property "unit x1" "0.1"
-			(at 0 0 0)
+			(at 0 0 315)
 			(unlocked yes)
 			(layer "F.Fab")
@@
 		(attr smd)
 		(fp_line
-			(start -0.227064 -0.735)
-			(end 0.227064 -0.735)
+			(start -0.227064 0.735)
+			(end 0.227064 0.735)
 			(stroke
 				(width 0.12)
@@
 		)
 		(fp_line
-			(start -0.227064 0.735)
-			(end 0.227064 0.735)
+			(start -0.227064 -0.735)
+			(end 0.227064 -0.735)
 			(stroke
 				(width 0.12)
@@
 		)
 		(fp_line
-			(start -1.85 -0.95)
-			(end 1.85 -0.95)
+			(start -1.85 0.95)
+			(end -1.85 -0.95)
 			(stroke
 				(width 0.05)
@@
 		)
 		(fp_line
-			(start -1.85 0.95)
-			(end -1.85 -0.95)
+			(start -1.85 -0.95)
+			(end 1.85 -0.95)
 			(stroke
 				(width 0.05)
@@
 		)
 		(fp_line
-			(start 1.85 -0.95)
-			(end 1.85 0.95)
+			(start 1.85 0.95)
+			(end -1.85 0.95)
 			(stroke
 				(width 0.05)
@@
 		)
 		(fp_line
-			(start 1.85 0.95)
-			(end -1.85 0.95)
+			(start 1.85 -0.95)
+			(end 1.85 0.95)
 			(stroke
 				(width 0.05)
@@
 		)
 		(fp_line
-			(start -1 -0.625)
-			(end 1 -0.625)
+			(start -1 0.625)
+			(end -1 -0.625)
 			(stroke
 				(width 0.1)
@@
 		)
 		(fp_line
-			(start -1 0.625)
-			(end -1 -0.625)
+			(start -1 -0.625)
+			(end 1 -0.625)
 			(stroke
 				(width 0.1)
@@
 		)
 		(fp_line
-			(start 1 -0.625)
-			(end 1 0.625)
+			(start 1 0.625)
+			(end -1 0.625)
 			(stroke
 				(width 0.1)
@@
 		)
 		(fp_line
-			(start 1 0.625)
-			(end -1 0.625)
+			(start 1 -0.625)
+			(end 1 0.625)
 			(stroke
 				(width 0.1)
@@
 		)
 		(fp_text user "${REFERENCE}"
-			(at 0 0 0)
+			(at 0 0 135)
 			(layer "F.Fab")
 			(effects
@@
 		)
 		(pad "1" smd roundrect
-			(at -1 0)
+			(at -1 0 315)
 			(size 1.2 1.4)
 			(layers "F.Cu" "F.Mask" "F.Paste")
@@
 		)
 		(pad "2" smd roundrect
-			(at 1 0)
+			(at 1 0 315)
 			(size 1.2 1.4)
 			(layers "F.Cu" "F.Mask" "F.Paste")
@@
 	(footprint "TestPoint:TestPoint_Loop_D2.50mm_Drill1.0mm_LowProfile"
 		(layer "F.Cu")
-		(at 161 66)
+		(at 104.5 73.5)
 		(descr "low profile wire loop as test point, loop diameter 2.5mm, hole diameter 1.0mm")
 		(tags "test point wire loop bead")
@@
 	)
 	(via
-		(at 112.75 85.35)
+		(at 111.5 84)
 		(size 0.6)
 		(drill 0.3)
@@
 	)
 	(segment
+		(start 114.503984 80.081802)
+		(end 113.292893 81.292893)
+		(width 0.3)
+		(layer "F.Cu")
+		(net 3)
+	)
+	(segment
 		(start 140.4 81.1)
 		(end 139.5 81.1)
@@
 	)
 	(segment
+		(start 114.503984 79.203984)
+		(end 114.503984 80.081802)
+		(width 0.3)
+		(layer "F.Cu")
+		(net 3)
+	)
+	(segment
 		(start 124.523223 86.423223)
 		(end 126.110051 84.836396)
@@
 	)
 	(segment
+		(start 113.556847 84.056847)
+		(end 113.556847 83.857367)
+		(width 0.3)
+		(layer "F.Cu")
+		(net 85)
+	)
+	(segment
 		(start 116.696016 81.396016)
-		(end 115.617678 81.396016)
+		(end 116.018198 81.396016)
+		(width 0.3)
+		(layer "F.Cu")
+		(net 85)
+	)
+	(segment
+		(start 116.018198 81.396016)
+		(end 114.707107 82.707107)
 		(width 0.3)
 		(layer "F.Cu")
@@
 	)
 	(segment
-		(start 115.617678 81.396016)
-		(end 114.056847 82.956847)
+		(start 113.556847 83.857367)
+		(end 114.707107 82.707107)
 		(width 0.3)
 		(layer "F.Cu")

Commit message: getting through PCB layout and schematic changes
Parts:
- removed C15, C16, C18, C19, C20, C22, C23, C24, C25, C26, C27, C28, C29, C8: 220n, Capacitor_SMD:C_1206_3216Metric_Pad1.33x1.80mm_HandSolder
- removed C21: 100p, Capacitor_SMD:C_1206_3216Metric_Pad1.33x1.80mm_HandSolder
- removed C31, C32, C8, C9: 10u, Capacitor_SMD:C_1206_3216Metric_Pad1.33x1.80mm_HandSolder
- removed C7: 100n, Capacitor_SMD:C_1206_3216Metric_Pad1.33x1.80mm_HandSolder
- removed D6, D7: BAT54S, Package_TO_SOT_SMD:SOT-23-3
- removed D6: ES1D, Diode_SMD:D_SMA
- removed the J1 at (111.0, 94.5)
- removed the J1 at (104.1, 78.7)
- removed the J18 at (153.0, 100.5)
- removed the J18 at (118.6, 25.8)
- removed JP1: SolderJumper_3_Open, Jumper:SolderJumper-3_P1.3mm_Open_Pad1.0x1.5mm
- removed Q6: 2N7002, Package_TO_SOT_SMD:SOT-23
- removed the R1 at (122.0, 63.7)
- removed the R11 at (135.1, 92.1)
- removed the R15 at (141.9, 64.0)
- removed the R16 at (117.3, 45.0)
- removed the R19 at (168.4, 38.4)
- removed the R2 at (136.2, 67.7)
- removed the R20 at (165.4, 38.4)
- removed the R21 at (162.3, 38.4)
- removed the R22 at (159.3, 38.4)
- removed the R23 at (159.8, 82.4)
- removed the R24 at (156.3, 38.4)
- removed the R32 at (153.3, 38.4)
- removed the R33 at (215.8, 47.1)
- removed the R34 at (147.3, 38.4)
- removed the R35 at (144.2, 38.4)
- removed the R36 at (141.2, 38.4)
- removed the R37 at (215.8, 56.0)
- removed R38, R40, R41, R42, R43, R44: 50, Resistor_SMD:R_1206_3216Metric_Pad1.30x1.75mm_HandSolder
- removed R5: 150, Resistor_SMD:R_1206_3216Metric_Pad1.30x1.75mm_HandSolder
- removed R5: 3.32k, Resistor_SMD:R_0805_2012Metric_Pad1.20x1.40mm_HandSolder
- removed R50: 4.99k, Resistor_SMD:R_1206_3216Metric_Pad1.30x1.75mm_HandSolder
- removed the R6 at (182.0, 59.5)
- removed the R7 at (114.0, 82.0)
- removed the R9 at (133.4, 93.8)
- removed TP12, TP3, TP4 (x2), TP5: TestPoint, TestPoint:TestPoint_Loop_D2.50mm_Drill1.0mm_LowProfile
- removed TP5: TestPoint, TestPoint:TestPoint_THTPad_3.0x3.0mm_Drill1.5mm
- removed the U1 at (112.3, 53.2)
- removed U2, U6: STISO620, Package_SO:SOIC-8_7.5x5.85mm_P1.27mm
- removed U7: PBQ76952PFBT, zzLocalLibraries-Footprints:BQ76952_PFB48_TEX
- removed U8: FCX495, Package_TO_SOT_SMD:SOT-89-3
- added C34: 100p, Capacitor_SMD:C_1206_3216Metric_Pad1.33x1.80mm_HandSolder, F.Cu at (31.7, 28.4)
- added C36: 220n, Capacitor_SMD:C_1206_3216Metric_Pad1.33x1.80mm_HandSolder, F.Cu at (31.7, 31.7)
- added C37: 220n, Capacitor_SMD:C_1206_3216Metric_Pad1.33x1.80mm_HandSolder, F.Cu at (31.7, 35.1)
- added C38: 220n, Capacitor_SMD:C_1206_3216Metric_Pad1.33x1.80mm_HandSolder, F.Cu at (31.7, 38.4)
- added C42: 220n, Capacitor_SMD:C_1206_3216Metric_Pad1.33x1.80mm_HandSolder, F.Cu at (31.7, 41.8)
- added C43: 220n, Capacitor_SMD:C_1206_3216Metric_Pad1.33x1.80mm_HandSolder, F.Cu at (31.7, 45.1)
- added C44: 220n, Capacitor_SMD:C_1206_3216Metric_Pad1.33x1.80mm_HandSolder, F.Cu at (31.7, 48.5)
- added C45: 220n, Capacitor_SMD:C_1206_3216Metric_Pad1.33x1.80mm_HandSolder, F.Cu at (37.7, 28.4)
- added C46: 220n, Capacitor_SMD:C_1206_3216Metric_Pad1.33x1.80mm_HandSolder, F.Cu at (37.7, 31.7)
- added C47: 220n, Capacitor_SMD:C_1206_3216Metric_Pad1.33x1.80mm_HandSolder, F.Cu at (37.7, 35.1)
- added C48: 220n, Capacitor_SMD:C_1206_3216Metric_Pad1.33x1.80mm_HandSolder, F.Cu at (37.7, 38.4)
- added C49: 220n, Capacitor_SMD:C_1206_3216Metric_Pad1.33x1.80mm_HandSolder, F.Cu at (37.7, 41.8)
- added C50: 220n, Capacitor_SMD:C_1206_3216Metric_Pad1.33x1.80mm_HandSolder, F.Cu at (37.7, 45.1)
- added C51: 220n, Capacitor_SMD:C_1206_3216Metric_Pad1.33x1.80mm_HandSolder, F.Cu at (37.7, 48.5)
- added C52: 220n, Capacitor_SMD:C_1206_3216Metric_Pad1.33x1.80mm_HandSolder, F.Cu at (43.8, 28.4)
- added C53: 220n, Capacitor_SMD:C_1206_3216Metric_Pad1.33x1.80mm_HandSolder, F.Cu at (43.8, 31.7)
- added C54: 220n, Capacitor_SMD:C_1206_3216Metric_Pad1.33x1.80mm_HandSolder, F.Cu at (43.8, 35.1)
- added C55: 220n, Capacitor_SMD:C_1206_3216Metric_Pad1.33x1.80mm_HandSolder, F.Cu at (43.8, 38.4)
- added C57: 10u, Capacitor_SMD:C_1206_3216Metric_Pad1.33x1.80mm_HandSolder, F.Cu at (43.8, 41.8)
- added D5: LED, LED_SMD:LED_0603_1608Metric, F.Cu at (62.7, 34.9)
- added J12: Screw_Terminal_01x02, TerminalBlock_MetzConnect:TerminalBlock_MetzConnect_Type059_RT06302HBWC_1x02_P3.50mm_Horizontal, F.Cu at (153.5, 20.2)
- added J15: Screw_Terminal_01x02, TerminalBlock_MetzConnect:TerminalBlock_MetzConnect_Type059_RT06302HBWC_1x02_P3.50mm_Horizontal, F.Cu at (106.4, 31.2)
- added J16: Conn_02x04_Odd_Even, Connector_PinHeader_2.54mm:PinHeader_2x04_P2.54mm_Vertical, F.Cu at (40.1, 54.4)
- added J2: Conn_01x10_Socket, Connector_PinHeader_2.54mm:PinHeader_1x10_P2.54mm_Vertical, F.Cu at (104.2, 83.0)
- added NT1: NetTie_2, NetTie:NetTie-2_SMD_Pad0.5mm, F.Cu at (48.0, 45.5)
- added R39: 3.32k, Resistor_SMD:R_0805_2012Metric_Pad1.20x1.40mm_HandSolder, F.Cu at (45.2, 65.8)
- added TP14: TestPoint, TestPoint:TestPoint_Loop_D2.50mm_Drill1.0mm_LowProfile, F.Cu at (47.2, 54.5)
- added TP16: TestPoint, TestPoint:TestPoint_Loop_D2.50mm_Drill1.0mm_LowProfile, F.Cu at (47.2, 59.1)
- added TP9: TestPoint, TestPoint:TestPoint_THTPad_3.0x3.0mm_Drill1.5mm, F.Cu at (40.3, 66.9)
- added U10: MCP2542FDxMF, Package_SO:JEITA_SOIC-8_3.9x4.9mm_P1.27mm, F.Cu at (55.7, 55.5)
- added U12: FT230XS, Package_SO:SSOP-16_3.9x4.9mm_P0.635mm, F.Cu at (155.5, 95.0)
- added U13: PBQ76952PFBT, zzLocalLibraries-Footprints:BQ76952_PFB48_TEX, F.Cu at (129.2, 55.5)
- added U14: FCX495, Package_TO_SOT_SMD:SOT-89-3, F.Cu at (50.1, 41.7)
- C1: value 100n -> 1u
- C11: value 100n -> 220n
- C14: value 220n -> 10u
- C17, C3: value 220n -> 100n
- C2, C6: value 220n -> 1u
- C30: value 10u -> 100n
- D2: value LED -> ES1D; footprint LED_SMD:LED_0603_1608Metric -> Diode_SMD:D_SMA
- J1: renamed from J2; value Screw_Terminal_01x02 -> Conn_02x05_Odd_Even; footprint TerminalBlock_MetzConnect:TerminalBlock_MetzConnect_Type059_RT06302HBWC_1x02_P3.50mm_Horizontal -> Connector_PinHeader_1.27mm:PinHeader_2x05_P1.27mm_Vertical_SMD
- J13: value Conn_01x07_Pin -> Screw_Terminal_01x02; footprint Connector_PinHeader_2.54mm:PinHeader_1x07_P2.54mm_Vertical -> TerminalBlock_MetzConnect:TerminalBlock_MetzConnect_Type059_RT06302HBWC_1x02_P3.50mm_Horizontal
- J14: value Conn_02x04_Odd_Even -> Screw_Terminal_01x02; footprint Connector_PinHeader_2.54mm:PinHeader_2x04_P2.54mm_Vertical -> TerminalBlock_MetzConnect:TerminalBlock_MetzConnect_Type059_RT06302HBWC_1x02_P3.50mm_Horizontal
- J17: renamed from J16; value Conn_01x04_Socket -> USB_B_Micro; footprint Connector_PinHeader_2.54mm:PinHeader_1x04_P2.54mm_Vertical -> Connector_USB:USB_Micro-B_Amphenol_10118194-0001LF_Horizontal
- J18: renamed from J17; value USB_B_Micro -> Conn_01x04_Socket; footprint Connector_USB:USB_Micro-B_Amphenol_10118194-0001LF_Horizontal -> Connector_PinHeader_2.54mm:PinHeader_1x04_P2.54mm_Vertical
- J3: renamed from J6; value Screw_Terminal_01x02 -> Conn_01x03_Pin; footprint TerminalBlock_MetzConnect:TerminalBlock_MetzConnect_Type059_RT06302HBWC_1x02_P3.50mm_Horizontal -> Connector_PinHeader_2.54mm:PinHeader_1x03_P2.54mm_Vertical
- J4: renamed from J3; value Screw_Terminal_01x02 -> Conn_01x04_Socket; footprint TerminalBlock_MetzConnect:TerminalBlock_MetzConnect_Type059_RT06302HBWC_1x02_P3.50mm_Horizontal -> Connector_PinHeader_2.54mm:PinHeader_1x04_P2.54mm_Vertical
- J5: value Screw_Terminal_01x02 -> Conn_01x07_Pin; footprint TerminalBlock_MetzConnect:TerminalBlock_MetzConnect_Type059_RT06302HBWC_1x02_P3.50mm_Horizontal -> Connector_PinHeader_2.54mm:PinHeader_1x07_P2.54mm_Vertical
- R1: value 4.99k -> 3.32k; footprint Resistor_SMD:R_1206_3216Metric_Pad1.30x1.75mm_HandSolder -> Resistor_SMD:R_0805_2012Metric_Pad1.20x1.40mm_HandSolder
- R10: value 97.6k -> 3.32k
- R11, R16, R7: value 200k -> 97.6k
- R12, R13: value 97.6k -> 150; footprint Resistor_SMD:R_0805_2012Metric_Pad1.20x1.40mm_HandSolder -> Resistor_SMD:R_1206_3216Metric_Pad1.30x1.75mm_HandSolder
- R14: value 3.32k -> 150; footprint Resistor_SMD:R_0805_2012Metric_Pad1.20x1.40mm_HandSolder -> Resistor_SMD:R_1206_3216Metric_Pad1.30x1.75mm_HandSolder
- R15: value 100 -> 3.32k; footprint Resistor_SMD:R_1206_3216Metric_Pad1.30x1.75mm_HandSolder -> Resistor_SMD:R_0805_2012Metric_Pad1.20x1.40mm_HandSolder
- R17: value 24.9 -> 150; footprint Resistor_SMD:R_0805_2012Metric_Pad1.20x1.40mm_HandSolder -> Resistor_SMD:R_1206_3216Metric_Pad1.30x1.75mm_HandSolder
- R18: value 24.9 -> 3.32k
- R2: value 150 -> 97.6k; footprint Resistor_SMD:R_1206_3216Metric_Pad1.30x1.75mm_HandSolder -> Resistor_SMD:R_0805_2012Metric_Pad1.20x1.40mm_HandSolder
- R3: value 150 -> 750
- R33: value 50 -> 24.9; footprint Resistor_SMD:R_1206_3216Metric_Pad1.30x1.75mm_HandSolder -> Resistor_SMD:R_0805_2012Metric_Pad1.20x1.40mm_HandSolder
- R34: value 150 -> 24.9; footprint Resistor_SMD:R_1206_3216Metric_Pad1.30x1.75mm_HandSolder -> Resistor_SMD:R_0805_2012Metric_Pad1.20x1.40mm_HandSolder
- R35: value 3.32k -> 24.9
- R36: value 3.32k -> 100; footprint Resistor_SMD:R_0805_2012Metric_Pad1.20x1.40mm_HandSolder -> Resistor_SMD:R_1206_3216Metric_Pad1.30x1.75mm_HandSolder
- R37: value 50 -> 100
- R6: value 750 -> 3.32k; footprint Resistor_SMD:R_1206_3216Metric_Pad1.30x1.75mm_HandSolder -> Resistor_SMD:R_0805_2012Metric_Pad1.20x1.40mm_HandSolder
- R8: value 3.32k -> 100k; footprint Resistor_SMD:R_0805_2012Metric_Pad1.20x1.40mm_HandSolder -> Resistor_SMD:R_1206_3216Metric_Pad1.30x1.75mm_HandSolder
- R9: value 10k -> 3.32k
- SW1, SW2: footprint Button_Switch_SMD:SW_SPST_PTS645 -> Button_Switch_SMD:SW_SPST_PTS645Sx43SMTR92
- U3: value RAA211805 -> STISO620; footprint Package_TO_SOT_SMD:TSOT-23-5 -> Package_SO:SOIC-8_7.5x5.85mm_P1.27mm
- U4: value MCP2542FDxMF -> RAA211805; footprint Package_SO:JEITA_SOIC-8_3.9x4.9mm_P1.27mm -> Package_TO_SOT_SMD:TSOT-23-5
- U5: value FT230XS -> STISO620; footprint Package_SO:SSOP-16_3.9x4.9mm_P0.635mm -> Package_SO:SOIC-8_7.5x5.85mm_P1.27mm
- moved R27 137.3 mm to (73.8, 42.5)
- moved R32 91.2 mm to (124.8, 38.8), turned to -90 degrees
- moved J1 85.4 mm to (111.0, 94.5), turned to 90 degrees
- moved R31 84.5 mm to (128.2, 38.8), turned to -90 degrees
- moved R30 80.5 mm to (131.8, 38.8), turned to -90 degrees
- moved R29 76.6 mm to (135.2, 38.8), turned to -90 degrees
- moved R28 73.0 mm to (138.5, 38.5), turned to -90 degrees
- moved R37 67.8 mm to (71.5, 26.4)
- moved R33 67.5 mm to (83.8, 27.0)
- moved J13 66.0 mm to (161.5, 20.2)
- moved R10 64.6 mm to (134.5, 100.2)
- moved R26 63.7 mm to (145.0, 38.5), turned to -90 degrees
- moved J14 61.9 mm to (169.5, 20.2), turned to 0 degrees
- moved R25 59.9 mm to (148.2, 38.2), turned to -90 degrees
- moved R24 56.0 mm to (151.5, 38.2), turned to -90 degrees
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- renumbered J4 to J6
Connections:
- C1 pad 1: -BATT -> /BQ76952 16C/BAT
- C1 pad 2: Net-(C1-Pad2) -> -BATT
- C10 pad 1: /UART_USB/5V -> /GLV interface/5v
- C10 pad 2: /UART_USB/GND -> /GLV interface/GLV-
- C11 pad 1: Net-(U7-SRP) -> Net-(U1-VCORE)
- C11 pad 2: Net-(U7-SRN) -> -BATT
- C12 pad 1: Net-(U7-VC16) -> VDD
- C12 pad 2: Net-(U7-VC15) -> -BATT
- C13 pad 1: Net-(U7-VC14) -> VDD
- C13 pad 2: Net-(U7-VC13) -> -BATT
- C14 pad 1: Net-(U7-VC12) -> VDD
- C14 pad 2: Net-(U7-VC11) -> -BATT
- C17 pad 1: Net-(U7-VC6) -> -BATT
- C17 pad 2: Net-(U7-VC5) -> Net-(C17-Pad2)
- C2 pad 1: VDD -> /BQ76952 16C/BAT
- C3 pad 1: VDD -> RST_N
- C30 pad 1: Net-(U7-REG18) -> Net-(U13-SRP)
- C30 pad 2: -BATT -> Net-(U13-SRN)
- C4 pad 1: VDD -> /UART_USB/5V
- C4 pad 2: -BATT -> /UART_USB/GND
- C6 pad 1: Net-(U1-VCORE) -> /GLV interface/GLV+
- C6 pad 2: -BATT -> /GLV interface/GLV-
- D2 pad 1: -BATT -> Net-(D2-K)
- D2 pad 2: Net-(D2-A) -> /GLV interface/GLV-
- D3 pad 2: /GLV interface/GLV- -> +BATT
- D4 pad 1: /UART_USB/GND -> -BATT
- J1 pad 1: /BQ76952 16C/15P -> /XDS_3v_supply
- J1 pad 2: +BATT -> PA19_SWDIO
- J10 pad 1: -BATT -> /BQ76952 16C/7P
- J10 pad 2: /BQ76952 16C/1N -> /BQ76952 16C/8P
- J11 pad 1: /BQ76952 16C/PACK- -> /BQ76952 16C/9P
- J11 pad 2: -BATT -> /BQ76952 16C/10P
- J13 pad 1: /BQ76952 16C/TS1 -> /BQ76952 16C/13P
- J13 pad 2: /BQ76952 16C/TS2 -> /BQ76952 16C/14P
- J14 pad 1: Net-(J14-Pin_1) -> /BQ76952 16C/15P
- J14 pad 2: PA18_SPI1_MOSI -> +BATT
- J17 pad 1: /GLV interface/GLV- -> /UART_USB/5V
- J17 pad 2: /GLV interface/GLV+ -> Net-(J17-D-)
- J17 pad 3: /GLV interface/CAN_H -> Net-(J17-D+)
- J17 pad 4: /GLV interface/CAN_L -> unconnected-(J17-ID-Pad4)
- J18 pad 2: Net-(J17-D-) -> Net-(J17-D+)
- J18 pad 3: Net-(J17-D+) -> Net-(J17-D-)
- J18 pad 4: unconnected-(J17-ID-Pad4) -> /UART_USB/GND
- J3 pad 1: /BQ76952 16C/7P -> onboard 3.3v src
- J3 pad 2: /BQ76952 16C/8P -> VDD
- J4 pad 1: /BQ76952 16C/13P -> /GLV interface/GLV-
- J4 pad 2: /BQ76952 16C/14P -> /GLV interface/GLV+
- J5 pad 1: /BQ76952 16C/9P -> /BQ76952 16C/TS1
- J5 pad 2: /BQ76952 16C/10P -> /BQ76952 16C/TS2
- J6 pad 1: /BQ76952 16C/11P -> -BATT
- J6 pad 2: /BQ76952 16C/12P -> /BQ76952 16C/1N
- J7 pad 1: /BQ76952 16C/5P -> /BQ76952 16C/1P
- J7 pad 2: /BQ76952 16C/6P -> /BQ76952 16C/2P
- J9 pad 1: /BQ76952 16C/1P -> /BQ76952 16C/5P
- J9 pad 2: /BQ76952 16C/2P -> /BQ76952 16C/6P
- L1 pad 1: Net-(D3-K) -> Net-(D2-K)
- R1 pad 1: Net-(Q6-G) -> Net-(C17-Pad2)
- R10 pad 1: RST_N -> /UART_USB/5V
- R10 pad 2: VDD -> Net-(D5-A)
- R11 pad 2: Net-(Q6-G) -> Net-(C17-Pad2)
- R12 pad 1: /GLV interface/GLV- -> Net-(D3-K)
- R12 pad 2: Net-(U4-STBY) -> /BQ76952 16C/BAT
- R13 pad 1: Net-(U3-EN) -> /BQ76952 16C/HDQ
- R13 pad 2: /GLV interface/GLV+ -> Net-(J16-Pin_1)
- R14 pad 1: /UART_USB/5V -> /BQ76952 16C/CFETOFF
- R14 pad 2: Net-(D4-A) -> Net-(J16-Pin_3)
- R15 pad 1: -BATT -> Net-(U13-LD)
- R15 pad 2: Net-(U7-SRP) -> /BQ76952 16C/BAT
- R16 pad 1: Net-(U4-EN) -> /GLV interface/GLV-
- R16 pad 2: /GLV interface/GLV+ -> Net-(U10-STBY)
- R17 pad 1: +BATT -> Net-(J16-Pin_7)
- R17 pad 2: Net-(U7-VC16) -> /BQ76952 16C/SDA
- R18 pad 1: /BQ76952 16C/15P -> Net-(R18-Pad1)
- R18 pad 2: Net-(U7-VC15) -> /BQ76952 16C/BAT
- R19 pad 1: /BQ76952 16C/14P -> +BATT
- R19 pad 2: Net-(U7-VC14) -> Net-(U13-VC16)
- R2 pad 1: Net-(J14-Pin_5) -> Net-(U4-EN)
- R2 pad 2: /BQ76952 16C/SCL -> /GLV interface/GLV+
- R20 pad 1: /BQ76952 16C/13P -> /BQ76952 16C/15P
- R20 pad 2: Net-(U7-VC13) -> Net-(U13-VC15)
- R21 pad 1: /BQ76952 16C/12P -> /BQ76952 16C/14P
- R21 pad 2: Net-(U7-VC12) -> Net-(U13-VC14)
- R22 pad 1: /BQ76952 16C/11P -> /BQ76952 16C/13P
- R22 pad 2: Net-(U7-VC11) -> Net-(U13-VC13)
- R23 pad 1: /BQ76952 16C/10P -> /BQ76952 16C/12P
- R24 pad 1: /BQ76952 16C/9P -> /BQ76952 16C/11P
- R25 pad 1: /BQ76952 16C/8P -> /BQ76952 16C/10P
- R26 pad 1: /BQ76952 16C/7P -> /BQ76952 16C/9P
- R27 pad 1: /BQ76952 16C/6P -> /BQ76952 16C/8P
- R27 pad 2: Net-(U7-VC6) -> Net-(U13-VC8)
- R28 pad 1: /BQ76952 16C/5P -> /BQ76952 16C/7P
- R28 pad 2: Net-(U7-VC5) -> Net-(U13-VC7)
- R29 pad 1: /BQ76952 16C/4P -> /BQ76952 16C/6P
- R3 pad 1: /BQ76952 16C/HDQ -> PA7
- R3 pad 2: Net-(J14-Pin_1) -> Net-(D4-A)
- R30 pad 1: /BQ76952 16C/3P -> /BQ76952 16C/5P
- R31 pad 1: /BQ76952 16C/2P -> /BQ76952 16C/4P
- R32 pad 1: /BQ76952 16C/1P -> /BQ76952 16C/3P
- R33 pad 1: /BQ76952 16C/9P -> /BQ76952 16C/2P
- R34 pad 1: Net-(D6-K) -> /BQ76952 16C/1P
- R34 pad 2: /BQ76952 16C/BAT -> Net-(U13-VC1)
- R35 pad 1: Net-(U7-PACK) -> /BQ76952 16C/1N
- R36 pad 1: Net-(U7-LD) -> -BATT
- R36 pad 2: /BQ76952 16C/BAT -> Net-(U13-SRP)
- R37 pad 1: /BQ76952 16C/5P -> /BQ76952 16C/PACK-
- R37 pad 2: Net-(U13-VC5) (its old number) -> Net-(U13-SRN)
- R4 pad 1: Net-(J14-Pin_7) -> Net-(J16-Pin_5)
- R4 pad 2: /BQ76952 16C/SDA -> /BQ76952 16C/SCL
- R6 pad 1: Net-(D1-A) -> VDD
- R6 pad 2: VDD -> Net-(D1-A)
- R8 pad 1: Net-(C1-Pad2) -> -BATT
- R8 pad 2: PA15_BBQ_RESET -> Net-(U1-PA2_ROSC)
- R9 pad 2: +BATT -> Net-(R18-Pad1)
- SW1 pad 1: onboard 3.3v src -> RST_N
- SW1 pad 2: Net-(C1-Pad2) -> -BATT
- SW2 pad 1: RST_N -> onboard 3.3v src
- SW2 pad 2: -BATT -> Net-(C17-Pad2)
- TP1 pad 1: onboard 3.3v src -> /XDS_3v_supply
- TP2 pad 1: /XDS_3v_supply -> onboard 3.3v src
- U3 pad 1: /GLV interface/5v -> /UART_USB/5V
- U3 pad 2: /GLV interface/GLV- -> Net-(U12-RXD)
- U3 pad 3: Net-(U3-EN) -> Net-(U12-TXD)
- U3 pad 4: /GLV interface/GLV+ -> /UART_USB/GND
- U3 pad 5: Net-(D3-K) -> -BATT
- U4 pad 1: Net-(U2-RXA) -> /GLV interface/5v
- U4 pad 3: /GLV interface/5v -> Net-(U4-EN)
- U4 pad 4: Net-(U2-TXB) -> /GLV interface/GLV+
- U4 pad 5: /GLV interface/5v -> Net-(D2-K)
- U5 pad 1: Net-(U5-TXD) -> -BATT
- U5 pad 2: unconnected-(U5-~{RTS}-Pad2) -> PA13_CAN_RX
- U5 pad 3: /UART_USB/5V -> PA12_CAN_TX
- U5 pad 4: Net-(U5-RXD) -> VDD
- U5 pad 5: /UART_USB/GND -> /GLV interface/5v
- U5 pad 6: unconnected-(U5-~{CTS}-Pad6) -> Net-(U10-TXD)
- U5 pad 7: unconnected-(U5-CBUS2-Pad7) -> Net-(U10-RXD)
- U5 pad 8: Net-(J17-D+) -> /GLV interface/GLV-
Routing:
- net (no net): track 5.79 -> 378.6 mm
- net +BATT: track 77.5 -> 0.00 mm
- net Net-(R18-Pad1): track 0.00 -> 65.1 mm
- net Net-(U13-VC16): track 45.2 -> 0.00 mm
- net Net-(U13-VC15): track 41.0 -> 0.00 mm
- net Net-(U13-VC14): track 38.2 -> 0.00 mm
- net Net-(U13-VC13): track 35.5 -> 0.00 mm
- net Net-(U13-VC12) (its old number): track 32.6 -> 0.00 mm
- net Net-(U13-VC11) (its old number): track 30.1 -> 0.00 mm
- net Net-(U13-VC12): track 0.00 -> 28.5 mm
- net /BQ76952 16C/1P: track 30.7 -> 2.60 mm
- net Net-(U13-VC10) (its old number): track 26.9 -> 0.00 mm
- net Net-(U13-VC11): track 0.00 -> 26.0 mm
- net Net-(U13-VC2): track 24.6 -> 0.00 mm
- net Net-(Q6-G): track 22.1 -> 0.00 mm
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Other:
- board size 72.2 x 83.8 mm -> 74.2 x 92.8 mm
- board text added: "${REFERENCE}"

Commit message: end the night with a push
Parts:
- moved C36 145.0 mm to (176.8, 33.5), turned to -90 degrees
- moved C37 137.0 mm to (168.8, 33.5), turned to -90 degrees
- moved C48 135.1 mm to (172.8, 33.5), turned to -90 degrees
- moved C38 129.1 mm to (160.8, 33.5), turned to -90 degrees
- moved C49 127.3 mm to (164.8, 33.5), turned to -90 degrees
- moved C42 121.3 mm to (152.8, 33.5), turned to -90 degrees
- moved C50 119.6 mm to (156.8, 33.5), turned to -90 degrees
- moved C43 113.6 mm to (144.8, 33.5), turned to -90 degrees
- moved C51 112.0 mm to (148.8, 33.5), turned to -90 degrees
- moved C44 106.1 mm to (136.8, 33.5), turned to -90 degrees
- moved C52 97.1 mm to (140.8, 33.5), turned to -90 degrees
- moved C45 91.2 mm to (128.8, 33.5), turned to -90 degrees
- moved C53 89.0 mm to (132.8, 33.5), turned to -90 degrees
- moved R35 83.1 mm to (112.5, 28.0), turned to -90 degrees
- moved C46 82.8 mm to (120.5, 33.5), turned to -90 degrees
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Routing:
- net (no net): track 378.6 -> 328.3 mm
- net Net-(U13-VC10): track 0.00 -> 37.8 mm
- net Net-(U13-VC9): track 0.00 -> 35.3 mm
- net Net-(U13-VC1): track 0.00 -> 27.4 mm
- net Net-(U13-VC2): track 0.00 -> 25.8 mm
- net /BQ76952 16C/BAT: track 0.00 -> 21.1 mm
- net Net-(U13-VC8): track 12.2 -> 31.8 mm
- net Net-(U13-VC12): track 28.5 -> 9.76 mm
- net Net-(U13-VC7): track 11.8 -> 28.6 mm
- net Net-(U13-VC11): track 26.0 -> 9.51 mm
- net -BATT: track 49.6 -> 33.4 mm
- net Net-(R18-Pad1): track 65.1 -> 49.2 mm
- net Net-(U13-VC15): track 0.00 -> 10.5 mm
- net Net-(U13-VC14): track 0.00 -> 10.3 mm
- net Net-(U13-VC13): track 0.00 -> 10.0 mm
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Other:
- board size 74.2 x 92.8 mm -> 78.5 x 92.8 mm

Commit message: trial 1...basically complete, going to come back tomorrow to make sure everything is right, logging off
Parts:
- removed J2: Conn_01x10_Socket, Connector_PinHeader_2.54mm:PinHeader_1x10_P2.54mm_Vertical
- moved D5 122.2 mm to (166.2, 99.8)
- moved J3 107.5 mm to (104.5, 93.2)
- moved U10 107.4 mm to (160.8, 78.0)
- moved U14 89.2 mm to (136.0, 66.0), turned to -45 degrees
- moved J16 86.7 mm to (125.8, 67.1), turned to -45 degrees
- moved R39 79.0 mm to (142.2, 70.8), turned to 90 degrees
- moved R14 71.4 mm to (113.0, 63.2), turned to -135 degrees
- moved R36 70.3 mm to (117.8, 42.1), turned to -45 degrees
- moved NT1 68.1 mm to (114.5, 30.8), turned to -90 degrees
- moved C12 66.5 mm to (112.5, 78.8), turned to -135 degrees
- moved C4 63.4 mm to (173.0, 96.5), turned to 90 degrees
- moved R17 62.2 mm to (118.2, 67.8), turned to 135 degrees
- moved C13 62.0 mm to (110.6, 77.1), turned to -135 degrees
- moved J4 60.0 mm to (179.0, 73.7)
- moved R2 54.8 mm to (173.8, 76.8), turned to 0 degrees
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Routing:
- net (no net): track 328.3 -> 0.00 mm
- net Net-(U13-VC16): track 5.47 -> 63.4 mm
- net onboard 3.3v src: track 71.6 -> 16.7 mm
- net Net-(U13-VC15): track 10.5 -> 61.7 mm
- net Net-(R18-Pad1): track 49.2 -> 1.75 mm
- net Net-(U13-VC14): track 10.3 -> 57.5 mm
- net Net-(U13-VC13): track 10.0 -> 53.8 mm
- net Net-(U13-VC12): track 9.76 -> 49.7 mm
- net Net-(U13-VC11): track 9.51 -> 46.6 mm
- net Net-(U13-VC6): track 8.96 -> 30.3 mm
- net Net-(D3-K): track 9.28 -> 28.8 mm
- net RST_N: track 35.4 -> 54.9 mm
- net /BQ76952 16C/BAT: track 21.1 -> 40.2 mm, vias 0 -> 2
- net Net-(U13-VC5): track 8.85 -> 27.7 mm
- net Net-(J17-D+): track 26.2 -> 44.9 mm
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Other:
- board size 78.5 x 92.8 mm -> 78.7 x 91.3 mm
