File: hardware/EVAL MSPM0lG3507 BQ76952/EVAL MSPM0lG3507 BQ76952.kicad_pcb (KiCad board)
At the start: 2 copper layers, 78.7 x 91.3 mm, 108 parts, among them J1 Conn_02x05_Odd_Even, J10 Screw_Terminal_01x02, J11 Screw_Terminal_01x02, J12 Screw_Terminal_01x02, J13 Screw_Terminal_01x02, J14 Screw_Terminal_01x02, J15 Screw_Terminal_01x02, J16 Conn_02x04_Odd_Even, J17 USB_B_Micro, J18 Conn_01x04_Socket, J3 Conn_01x03_Pin, J4 Conn_01x04_Socket, J5 Conn_01x07_Pin, J6 Screw_Terminal_01x02, J7 Screw_Terminal_01x02, J8 Screw_Terminal_01x02, J9 Screw_Terminal_01x02, SW1 SW_Push, SW2 SW_Push, U1 MCU-MSM0G3507SPM, U10 MCP2542FDxMF, U12 FT230XS, U13 PBQ76952PFBT, U14 FCX495, U3 STISO620, U4 RAA211805, U5 STISO620

Commit message: deep
Routing:
- net RST_N: track 54.9 -> 59.1 mm, vias 0 -> 2
- net -BATT: vias 62 -> 67
Changed lines of the file:
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@@
 	)
 	(segment
-		(start 139.087501 70.75)
-		(end 143.05 70.75)
+		(start 145.92 67.68)
+		(end 145.92 66.55)
 		(width 0.3)
 		(layer "F.Cu")
@@
 	)
 	(segment
-		(start 145.92 67.68)
-		(end 145.92 66.55)
+		(start 137.25 70.75)
+		(end 137.75 70.75)
 		(width 0.3)
 		(layer "F.Cu")
@@
 	(segment
 		(start 145.92 66.55)
-		(end 153.88 66.55)
+		(end 145.92 67.88)
 		(width 0.3)
 		(layer "F.Cu")
@@
 	)
 	(segment
-		(start 138.9 70.937501)
-		(end 139.087501 70.75)
+		(start 145.92 66.55)
+		(end 153.88 66.55)
 		(width 0.3)
 		(layer "F.Cu")
@@
 	)
 	(segment
-		(start 127 60.75)
-		(end 127.42246 61.17246)
+		(start 125.402944 84.129289)
+		(end 126.25 83.282233)
+		(width 0.3)
+		(layer "F.Cu")
+		(net 1)
+	)
+	(segment
+		(start 145.92 67.88)
+		(end 143.05 70.75)
 		(width 0.3)
 		(layer "F.Cu")
@@
 	)
 	(segment
-		(start 127.42246 61.17246)
-		(end 127.42246 62.72246)
+		(start 137.25 70.75)
+		(end 137 71)
 		(width 0.3)
 		(layer "F.Cu")
@@
 	)
 	(segment
+		(start 143.05 70.75)
+		(end 137.25 70.75)
+		(width 0.3)
+		(layer "F.Cu")
+		(net 1)
+	)
+	(segment
 		(start 116.645146 88.85936)
 		(end 118.688039 90.902253)
@@
 	)
 	(segment
-		(start 127.42246 62.72246)
-		(end 135.637501 70.937501)
+		(start 126.25 83.282233)
+		(end 126.25 82)
 		(width 0.3)
 		(layer "F.Cu")
@@
 	)
 	(segment
-		(start 135.637501 70.937501)
-		(end 138.9 70.937501)
+		(start 117.684996 89.984996)
+		(end 119.084996 88.584996)
 		(width 0.3)
 		(layer "F.Cu")
@@
 	)
 	(segment
-		(start 143.05 70.75)
-		(end 145.92 67.88)
-		(width 0.3)
+		(start 116.645146 88.854854)
+		(end 116.645146 88.85936)
+		(width 0.6)
 		(layer "F.Cu")
 		(net 1)
 	)
+	(via
+		(at 137 71)
+		(size 0.6)
+		(drill 0.3)
+		(layers "F.Cu" "B.Cu")
+		(net 1)
+	)
+	(via
+		(at 126.25 82)
+		(size 0.6)
+		(drill 0.3)
+		(layers "F.Cu" "B.Cu")
+		(net 1)
+	)
 	(segment
-		(start 145.92 67.88)
-		(end 145.92 66.55)
+		(start 126.671 81.579)
+		(end 128.171 81.579)
 		(width 0.3)
-		(layer "F.Cu")
+		(layer "B.Cu")
 		(net 1)
 	)
 	(segment
-		(start 117.684996 89.984996)
-		(end 119.084996 88.584996)
+		(start 128.171 81.579)
+		(end 134.25 75.5)
 		(width 0.3)
-		(layer "F.Cu")
+		(layer "B.Cu")
 		(net 1)
 	)
 	(segment
-		(start 116.645146 88.854854)
-		(end 116.645146 88.85936)
-		(width 0.6)
-		(layer "F.Cu")
+		(start 134.25 75.25)
+		(end 137 72.5)
+		(width 0.3)
+		(layer "B.Cu")
+		(net 1)
+	)
+	(segment
+		(start 134.25 75.5)
+		(end 134.25 75.25)
+		(width 0.3)
+		(layer "B.Cu")
+		(net 1)
+	)
+	(segment
+		(start 137 72.5)
+		(end 137 71)
+		(width 0.3)
+		(layer "B.Cu")
+		(net 1)
+	)
+	(segment
+		(start 126.25 82)
+		(end 126.671 81.579)
+		(width 0.3)
+		(layer "B.Cu")
 		(net 1)
 	)
@@
 	)
 	(via
+		(at 117.75 83.25)
+		(size 0.6)
+		(drill 0.3)
+		(layers "F.Cu" "B.Cu")
+		(free yes)
+		(net 2)
+	)
+	(via
 		(at 111.25 62.75)
 		(size 0.6)
@@
 	)
 	(via
+		(at 132.25 62.75)
+		(size 0.6)
+		(drill 0.3)
+		(layers "F.Cu" "B.Cu")
+		(net 2)
+	)
+	(via
 		(at 108 79.75)
 		(size 0.6)
@@
 	)
 	(via
+		(at 138.25 57)
+		(size 0.6)
+		(drill 0.3)
+		(layers "F.Cu" "B.Cu")
+		(net 2)
+	)
+	(via
 		(at 131.25 57.15)
 		(size 0.6)
@@
 	)
 	(via
+		(at 114.5 86.5)
+		(size 0.6)
+		(drill 0.3)
+		(layers "F.Cu" "B.Cu")
+		(free yes)
+		(net 2)
+	)
+	(via
+		(at 117.25 93)
+		(size 0.6)
+		(drill 0.3)
+		(layers "F.Cu" "B.Cu")
+		(net 2)
+	)
+	(via
 		(at 134.4 80.1)
 		(size 0.6)
@@
 	)
 	(segment
-		(start 120.75 80.7)
-		(end 109.73 91.72)
-		(width 0.3)
-		(layer "F.Cu")
-		(net 12)
-	)
-	(segment
 		(start 131.120729 76.079271)
 		(end 131.206498 76.16504)
@@
 	)
 	(segment
-		(start 121 80.7)
-		(end 120.75 80.7)
+		(start 114 88)
+		(end 113.45 88)
 		(width 0.3)
 		(layer "F.Cu")
@@
 		(net 12)
 	)
+	(segment
+		(start 121 80.7)
+		(end 121 81)
+		(width 0.3)
+		(layer "F.Cu")
+		(net 12)
+	)
+	(segment
+		(start 113.45 88)
+		(end 109.73 91.72)
+		(width 0.3)
+		(layer "F.Cu")
+		(net 12)
+	)
+	(segment
+		(start 121 81)
+		(end 114 88)
+		(width 0.3)
+		(layer "F.Cu")
+		(net 12)
+	)
 	(via
 		(at 131.120729 76.079271)
@@
 		(min_thickness 0.2)
 		(filled_areas_thickness no)
-		(fill
+		(fill yes
 			(thermal_gap 0.3)
 			(thermal_bridge_width 0.6)
@@
 		(min_thickness 0.2)
 		(filled_areas_thickness no)
-		(fill
+		(fill yes
 			(thermal_gap 0.3)
 			(thermal_bridge_width 0.6)
@@
 		(min_thickness 0.2)
 		(filled_areas_thickness no)
-		(fill
+		(fill yes
 			(thermal_gap 0.3)
 			(thermal_bridge_width 0.6)
