File: hardware/MasterBoard_A/PWM sig bank 1.kicad_sch (KiCad schematic)
At the start: 41 parts, among them Q16 MMBT5550L, Q17 MMBT5550L, Q4 MMBT5550L, Q6 MMBT5550L, Q7 MMBT5550L, Q8 MMBT5550L, U15 TLP155E, U16 TLP155E, U17 TLP155E, U20 DMN62D0U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

Commit message: mb v1.1 on da way
shuffled around stuff. review notes. made notes. glory to those who look forward and all that fuzz
Parts:
- removed D30, D32, D34: yellow, LED_SMD:LED_0805_2012Metric_Pad1.15x1.40mm_HandSolder, symbol Device:LED_Small
- removed Q16, Q17: MMBT5550L, Package_TO_SOT_SMD:SOT-23, symbol Transistor_BJT:MMBT5550L
- removed R106: 39k, Resistor_SMD:R_0805_2012Metric_Pad1.20x1.40mm_HandSolder, symbol Device:R_Small_US
- removed R36: 332, Resistor_SMD:R_1206_3216Metric_Pad1.30x1.75mm_HandSolder, symbol Device:R_Small_US
- added R13, R16: 750, Resistor_SMD:R_1206_3216Metric_Pad1.30x1.75mm_HandSolder, symbol Device:R_Small_US
- added R17: 97.6k, Resistor_SMD:R_0805_2012Metric_Pad1.20x1.40mm_HandSolder, symbol Device:R_Small_US
- added U11: AP7381-33SA-7, Package_TO_SOT_SMD:SOT-23, symbol Regulator_Linear:AP7381-33SA-7
Connections:
- net i-: now also R16.1
- net i1: now also Q8.1 (B)
- net o-: now also D25.1 (K), R17.1, U11.3 (GND)
- net at C27.1, C28.1, C29.1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: now also U11.1 (VI); no longer D25.2 (A)
- net at R46.1, U21.1 (EN/UVLO): now also R17.2
- net at D28.1 (K): now also R16.2; no longer Q8.1 (B)
- new net: D25.2 (A), R13.1
- new net: R13.2, U11.2 (VO)
Other:
- note added: "(2.28, 31)V"
- note removed: "(6, 30)V"
- company: (none) -> UTA Racing
- title: (none) -> BeeMS Master Board (A)
- moved on the sheet: C38, D25, D28, R46
