File: hardware/W5500 testing/W5500 testing.kicad_sch (KiCad schematic)
At the start: 1 part, among them J4 Conn_01x08_Pin

Commit message: mb v1.1 on da way
shuffled around stuff. review notes. made notes. glory to those who look forward and all that fuzz
Other:
- company: (none) -> BeeMS
- title: (none) -> spi ethernet controller
Changed lines of the file:
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@@
 	(generator_version "9.0")
 	(paper "A4")
+	(title_block
+		(title "spi ethernet controller")
+		(company "BeeMS")
+	)
 	(text "screwed this up a few times :( , test board to lock in on"
 		(exclude_from_sim no)
