File: hardware/W5500 testing/wizard.kicad_sch (KiCad schematic)
At the start: 43 parts, among them J10 RJ45_Amphenol_RJMG1BD3B8K1ANR, U18 W5500, Y1 25MHz

Commit message: test
Parts:
- removed C1, C12, C17, C3, C46, C48, C50, C51, C56: 220n, Capacitor_SMD:C_0805_2012Metric_Pad1.18x1.45mm_HandSolder, symbol Device:C_Small
- removed C16, C47, C55, C67: 10n, Capacitor_SMD:C_0805_2012Metric_Pad1.18x1.45mm_HandSolder, symbol Device:C_Small
- removed C54, C57: 10u, Capacitor_SMD:C_1206_3216Metric_Pad1.33x1.80mm_HandSolder, symbol Device:C_Small
- removed C69: 1n 2kV, Capacitor_SMD:C_1206_3216Metric_Pad1.33x1.80mm_HandSolder, symbol Device:C_Small
- removed NT2: NetTie_2, NetTie:NetTie-2_SMD_Pad2.0mm, symbol Device:NetTie_2
- removed R74, R75, R76, R77: 3.3, Resistor_SMD:R_1206_3216Metric_Pad1.30x1.75mm_HandSolder, symbol Device:R_Small_US
- removed R80: 10, Resistor_SMD:R_1206_3216Metric_Pad1.30x1.75mm_HandSolder, symbol Device:R_Small_US
- removed R81, R82: 750, Resistor_SMD:R_1206_3216Metric_Pad1.30x1.75mm_HandSolder, symbol Device:R_Small_US
- removed R87: 226, Resistor_SMD:R_0805_2012Metric_Pad1.20x1.40mm_HandSolder, symbol Device:R_Small_US
- removed Y1: 25MHz, Crystal:Crystal_SMD_ECS_CSM3X-2Pin_7.6x4.1mm, symbol Device:Crystal
- added C22, C29, C39: 10u, Capacitor_SMD:C_1206_3216Metric_Pad1.33x1.80mm_HandSolder, symbol Device:C_Small
- added C23, C25, C27, C28, C30, C38, C40: 100n, Capacitor_SMD:C_0603_1608Metric_Pad1.08x0.95mm_HandSolder, symbol Device:C_Small
- added C37: 1n 2kV, Capacitor_SMD:C_1206_3216Metric_Pad1.33x1.80mm_HandSolder, symbol Device:C_Small
- added FB2: ~, Inductor_SMD:L_0603_1608Metric_Pad1.05x0.95mm_HandSolder, symbol Device:FerriteBead
- added Q4, Q5: MMBT5550L, Package_TO_SOT_SMD:SOT-23, symbol Transistor_BJT:MMBT5550L
- added R35: 0, Resistor_SMD:R_0805_2012Metric_Pad1.20x1.40mm_HandSolder, symbol Device:R_Small_US
- added R37, R38, R39, R40: 14.3, Resistor_SMD:R_0805_2012Metric_Pad1.20x1.40mm_HandSolder, symbol Device:R_Small_US
- added R43, R44: 4.99k, Resistor_SMD:R_1206_3216Metric_Pad1.30x1.75mm_HandSolder, symbol Device:R_Small_US
- added R47: 10, Resistor_SMD:R_0805_2012Metric_Pad1.20x1.40mm_HandSolder, symbol Device:R_Small_US
- added R48, R49: 332, Resistor_SMD:R_1206_3216Metric_Pad1.30x1.75mm_HandSolder, symbol Device:R_Small_US
- added Y1: Crystal_GND24, Crystal:Crystal_SMD_2016-4Pin_2.0x1.6mm, symbol Device:Crystal_GND24
- R34: renamed from R86; footprint Resistor_SMD:R_0805_2012Metric_Pad1.20x1.40mm_HandSolder -> Resistor_SMD:R_0603_1608Metric_Pad0.98x0.95mm_HandSolder; mouser https://www.mouser.com/ProductDetail/Vishay-Beyschlag/MCU08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 -> https://www.mouser.com/ProductDetail/Bourns/CRT0603-DZ-1004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; specs 1M, 125mW, 150V, 1%, 50ppm, -55C, +125C -> 1M, 100mW, 750V, 0.5%, 50ppm, -55C, +155C; unit x1 0.1 -> 0.10; unit x10 0.07 -> 0.031
- renumbered C72 to C24, C71 to C26, C65 to C31, C70 to C32, C63 to C33, C64 to C34, C68 to C35, C62 to C36, J10 to J5, R84 to R36, R72 to R41, R78 to R42, R73 to R45, R79 to R46, U18 to U22
Connections:
- net +3.3V: now also C29.1, FB2.1; no longer NT1.1
- net +3.3VA: now also C22.1, C23.1, C25.1, C27.1, C28.1, C30.1, C38.1, C39.1, C40.1, FB2.2, R47.1; no longer NT1.2
- net GND: now also NT1.2, C29.2, C37.1, Q4.2 (E), Q5.2 (E), Y1.2, Y1.4; no longer C31.2
- net RX+: now also U22.6 (RXP), R39.2; no longer R46.2, U22.5 (RXN)
- net RX-: now also U22.5 (RXN), R40.1; no longer R42.2, U22.6 (RXP)
- net RX_1+: now also R46.2, R39.1
- net RX_1-: now also R42.2, R40.2
- net TD+: now also R41.1, R37.1
- net TD-: now also R45.1, R38.2
- net TX+: now also U22.2 (TXP), R37.2; no longer R41.1, U22.1 (TXN)
- net TX-: now also U22.1 (TXN), R38.1; no longer R45.1, U22.2 (TXP)
- net at U22.27 (ACTLED): now also R44.2
- net at J5.L3: now also R49.1
- net at U22.25 (LINKLED): now also R43.1
- net at R34.1, U22.30 (XI/CLKIN): now also C24.1, Y1.1
- net at R34.2, U22.31 (XO): now also R35.1; no longer C26.1
- net at J5.R5 (RCT): now also C36.1, R42.1, R46.1
- net at C35.1, J5.R4 (TCT): now also R47.2
- net at J5.L2: now also R48.2
- net GNDA renamed AGND
- net AGND: now also C31.2, NT1.1, C22.2, C23.2, C25.2, C27.2, C28.2, C30.2, C37.2, C38.2, C39.2, C40.2
- new net: Q5.3 (C), R49.2
- new net: Q5.1 (B), R44.1
- new net: C26.1, R35.2, Y1.3
- new net: Q4.3 (C), R48.1
- new net: Q4.1 (B), R43.2
Other:
- note added: "PMODE has internal PU"
- note removed: "(WORK IN PROGRESS ...)"
- note removed: "- 99% chance does not meet FCC standards"
- note removed: "DUMPSTER FIRE !!! DO NOT USE !!!!"
- note removed: "design guide: https://docs.wiznet.io/img/design_guide/Wiznet%20Ethernet%20Design%20Guide_ENG.pdf"
- note removed: "eyeballed this value idk, its to prevent over power"
- company: (none) -> BeeMS
- title: (none) -> spi ethernet controller
- moved on the sheet: C24, C26, C31, C32, C33, C34, C35, C36, J5, R34, R36, R41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

Commit message: joined wizards
wizz chip no more split ground. seems scuffed before, less scuffed
Parts:
- removed NT1: NetTie_2, NetTie:NetTie-2_SMD_Pad2.0mm, symbol Device:NetTie_2
Connections:
- net AGND is gone; now on net GND: C22.2, C23.2, C25.2, C27.2, C28.2, C30.2, C31.2, C32.2, C35.2, C36.2, C37.2, C38.2, C39.2, C40.2, R36.2, U22.14 (AGND), U22.16 (AGND), U22.19 (AGND), U22.3 (AGND), U22.48 (AGND), U22.9 (AGND)
Changed lines of the file:
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@@
 	(wire
 		(pts
-			(xy 36.83 33.02) (xy 52.07 33.02)
-		)
-		(stroke
-			(width 0)
-			(type default)
-		)
-	)
-	(wire
-		(pts
 			(xy 154.94 97.79) (xy 163.83 97.79)
 		)
@@
 	(wire
 		(pts
-			(xy 26.67 33.02) (xy 31.75 33.02)
+			(xy 26.67 33.02) (xy 52.07 33.02)
 		)
 		(stroke
@@
 					(unit 1)
 				)
-			)
-		)
-	)
-	(symbol
-		(lib_id "Device:NetTie_2")
-		(at 34.29 33.02 180)
-		(unit 1)
-		(exclude_from_sim no)
-		(in_bom no)
-		(on_board yes)
-		(dnp no)
-		(property "Reference" "NT1"
-			(at 34.29 35.56 0)
-			(effects
-				(font
-					(size 1.27 1.27)
-				)
-			)
-		)
-		(property "Value" "NetTie_2"
-			(at 34.29 38.1 0)
-			(effects
-				(font
-					(size 1.27 1.27)
-				)
-				(hide yes)
-			)
-		)
-		(property "Footprint" "NetTie:NetTie-2_SMD_Pad2.0mm"
-			(at 34.29 33.02 0)
-			(effects
-				(font
-					(size 1.27 1.27)
-				)
-				(hide yes)
-			)
-		)
-		(property "Datasheet" "~"
-			(at 34.29 33.02 0)
-			(effects
-				(font
-					(size 1.27 1.27)
-				)
-				(hide yes)
-			)
-		)
-		(property "Description" "Net tie, 2 pins"
-			(at 34.29 33.02 0)
-			(effects
-				(font
-					(size 1.27 1.27)
-				)
-				(hide yes)
-			)
-		)
-		(pin "2"
-		)
-		(pin "1"
-		)
-		(instances
-			(project ""
-				(path "/3cda9d14-c948-44fe-9af9-6daef6da768c/575b4cdf-c54c-463c-83fa-7ec0ac8843d7"
-					(reference "NT1")
-					(unit 1)
-				)

Commit message: mb v1.1 on da way
shuffled around stuff. review notes. made notes. glory to those who look forward and all that fuzz
Parts:
- C37: now not fitted; now left out of the parts list
- R35: value 0 -> 14.3; mouser (none) -> https://www.mouser.com/ProductDetail/KOA-Speer/RK73H2ATTD14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; specs usr a random resistor or something -> 14.3R, 250mW, 1%, 100ppm, 150V, -55C, +155C; unit x1 (none) -> 0.10; unit x10 (none) -> 0.02
Connections:
- net at R34.2, U22.31 (XO): now also R35.2; no longer R35.1
- net at C26.1, Y1.3: now also R35.1; no longer R35.2
Changed lines of the file:
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@@
 	(title_block
 		(title "spi ethernet controller")
+		(date "2025-12-26")
 		(rev "1.0")
 		(company "BeeMS")
@@
 		)
 	)
-	(text_box "sheilding note\n- rj45 sheilding sucks. sheild goes elsewhere"
+	(text_box "miscellaneous\n- rj45 sheilding sucks. sheild goes elsewhere\n- FSAE rule (updated 2026) : \"\"\"\n		EV.5.2.5 Each wire used in a Tractive Battery Container, whether it is part of the GLV or Tractive System, must be rated to the maximum Tractive System voltage\n	\"\"\"\n	i know other teams use ethernet for segment interconnects, not sure how they get away with it.\n- smallest part 0805 inch. is hand solderable\n- suggest paste + heatgun oscillator on first, then iron everything else starting with w5500 and ending with rj45 jack\n- \"RSVD\" pins can be GND to for routing ease"
 		(exclude_from_sim no)
 		(at 119.38 154.94 0)
@@
 	)
 	(no_connect
-		(at 92.71 125.73)
+		(at 92.71 115.57)
+	)
+	(no_connect
+		(at 92.71 123.19)
 	)
 	(no_connect
@@
 	)
 	(no_connect
-		(at 92.71 115.57)
+		(at 92.71 130.81)
 	)
 	(no_connect
-		(at 92.71 118.11)
+		(at 92.71 125.73)
 	)
 	(no_connect
@@
 	)
 	(no_connect
-		(at 92.71 130.81)
-	)
-	(no_connect
-		(at 92.71 123.19)
+		(at 92.71 118.11)
 	)
 	(no_connect
@@
 	(symbol
 		(lib_id "Device:R_Small_US")
+		(at 81.28 119.38 0)
+		(mirror x)
+		(unit 1)
+		(exclude_from_sim no)
+		(in_bom yes)
+		(on_board yes)
+		(dnp no)
+		(property "Reference" "R35"
+			(at 86.868 118.364 0)
+			(effects
+				(font
+					(size 1.27 1.27)
+				)
+				(justify right)
+			)
+		)
+		(property "Value" "14.3"
+			(at 86.868 120.142 0)
+			(effects
+				(font
+					(size 1.27 1.27)
+				)
+				(justify right)
+			)
+		)
+		(property "Footprint" "Resistor_SMD:R_0805_2012Metric_Pad1.20x1.40mm_HandSolder"
+			(at 81.28 119.38 0)
+			(effects
+				(font
+					(size 1.27 1.27)
+				)
+				(hide yes)
+			)
+		)
+		(property "Datasheet" ""
+			(at 81.28 119.38 0)
+			(effects
+				(font
+					(size 1.27 1.27)
+				)
+				(hide yes)
+			)
+		)
+		(property "Description" "Resistor, US symbol"
+			(at 81.28 119.38 0)
+			(effects
+				(font
+					(size 1.27 1.27)
+				)
+				(hide yes)
+			)
+		)
+		(property "mouser" "https://www.mouser.com/ProductDetail/KOA-Speer/RK73H2ATTD14R3F?qs=sGAEpiMZZMvdGkrng054tzl5geC4ftCS2xF%2Fs66%2F7iY%3D"
+			(at 81.28 119.38 0)
+			(effects
+				(font
+					(size 1.27 1.27)
+				)
+				(hide yes)
+			)
+		)
+		(property "specs" "14.3R, 250mW, 1%, 100ppm, 150V, -55C, +155C"
+			(at 81.28 119.38 0)
+			(effects
+				(font
+					(size 1.27 1.27)
+				)
+				(hide yes)
+			)
+		)
+		(property "unit x1" "0.10"
+			(at 81.28 119.38 0)
+			(effects
+				(font
+					(size 1.27 1.27)
+				)
+				(hide yes)
+			)
+		)
+		(property "unit x10" "0.02"
+			(at 81.28 119.38 0)
+			(effects
+				(font
+					(size 1.27 1.27)
+				)
+				(hide yes)
+			)
+		)
+		(property "note" ""
+			(at 81.28 119.38 0)
+			(effects
+				(font
+					(size 1.27 1.27)
+				)
+				(hide yes)
+			)
+		)
+		(pin "2"
+		)
+		(pin "1"
+		)
+		(instances
+			(project "W5500 testing"
+				(path "/3cda9d14-c948-44fe-9af9-6daef6da768c/575b4cdf-c54c-463c-83fa-7ec0ac8843d7"
+					(reference "R35")
+					(unit 1)
+				)
+			)
+		)
+	)
+	(symbol
+		(lib_id "Device:R_Small_US")
 		(at 157.48 118.11 270)
 		(mirror x)
@@
 		(unit 1)
 		(exclude_from_sim no)
-		(in_bom yes)
-		(on_board yes)
-		(dnp no)
+		(in_bom no)
+		(on_board no)
+		(dnp yes)
 		(property "Reference" "C37"
 			(at 202.438 99.822 90)
@@
 					(unit 1)
 				)
-			)
-		)
-	)
-	(symbol
-		(lib_id "Device:R_Small_US")
-		(at 81.28 119.38 0)
-		(unit 1)
-		(exclude_from_sim no)
-		(in_bom yes)
-		(on_board yes)
-		(dnp no)
-		(property "Reference" "R35"
-			(at 82.804 118.618 0)
-			(effects
-				(font
-					(size 1.27 1.27)
-				)
-				(justify left)
-			)
-		)
-		(property "Value" "0"
-			(at 82.804 120.396 0)
-			(effects
-				(font
-					(size 1.27 1.27)
-				)
-				(justify left)
-			)
-		)
-		(property "Footprint" "Resistor_SMD:R_0805_2012Metric_Pad1.20x1.40mm_HandSolder"
-			(at 81.28 119.38 0)
-			(effects
-				(font
-					(size 1.27 1.27)
-				)
-				(hide yes)
-			)
-		)
-		(property "Datasheet" ""
-			(at 81.28 119.38 0)
-			(effects
-				(font
-					(size 1.27 1.27)
-				)
-				(hide yes)
-			)
-		)
-		(property "Description" "Resistor, US symbol"
-			(at 81.28 119.38 0)
-			(effects
-				(font
-					(size 1.27 1.27)
-				)
-				(hide yes)
-			)
-		)
-		(property "Sim.Device" ""
-			(at 81.28 119.38 0)
-			(effects
-				(font
-					(size 1.27 1.27)
-				)
-				(hide yes)
-			)
-		)
-		(property "Sim.Type" ""
-			(at 81.28 119.38 0)
-			(effects
-				(font
-					(size 1.27 1.27)
-				)
-				(hide yes)
-			)
-		)
-		(property "mouser" ""
-			(at 81.28 119.38 0)
-			(effects
-				(font
-					(size 1.27 1.27)
-				)
-				(hide yes)
-			)
-		)
-		(property "specs" "usr a random resistor or something"
-			(at 81.28 119.38 0)
-			(effects
-				(font
-					(size 1.27 1.27)
-				)
-				(hide yes)
-			)
-		)
-		(property "unit x1" ""
-			(at 81.28 119.38 0)
-			(effects
-				(font
-					(size 1.27 1.27)
-				)
-				(hide yes)
-			)
-		)
-		(property "unit x10" ""
-			(at 81.28 119.38 0)
-			(effects
-				(font
-					(size 1.27 1.27)
-				)
-				(hide yes)
-			)
-		)
-		(property "Sim.Pins" ""
-			(at 81.28 119.38 90)
-			(effects
-				(font
-					(size 1.27 1.27)
-				)
-				(hide yes)
-			)
-		)
-		(property "note" ""
-			(at 81.28 119.38 90)
-			(effects
-				(font
-					(size 1.27 1.27)
-				)
-				(hide yes)
-			)
-		)
-		(pin "2"
-		)
-		(pin "1"
-		)
-		(instances
-			(project "W5500 testing"
-				(path "/3cda9d14-c948-44fe-9af9-6daef6da768c/575b4cdf-c54c-463c-83fa-7ec0ac8843d7"
-					(reference "R35")
-					(unit 1)
-				)
