File: hardware/VoltageTap_A/BQ76952 1.kicad_sch (KiCad schematic)
At the start: 116 parts, among them U1 2PD2150-QX, U36 PBQ76952PFBT, U37 FCX495, U40 2PD2150-QX, U41 2PD2150-QX, U42 2PD2150-QX, U43 2PD2150-QX, U44 2PD2150-QX, U45 2PD2150-QX, U46 2PD2150-QX, U47 2PD2150-QX, U48 2PD2150-QX, U49 2PD2150-QX, U50 2PD2150-QX, U51 2PD2150-QX, U52 2PD2150-QX, U53 2PD2150-QX, U54 2PD2150-QX

Commit message: VT stuff
Parts:
- removed C54: 10n, Capacitor_SMD:C_0805_2012Metric_Pad1.18x1.45mm_HandSolder, symbol Device:C_Small
Changed lines of the file:
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@@
 	)
 	(junction
+		(at 234.95 53.34)
+		(diameter 0)
+		(color 0 0 0 0)
+	)
+	(junction
 		(at 107.95 142.24)
 		(diameter 0)
@@
 	)
 	(junction
-		(at 224.79 53.34)
-		(diameter 0)
-		(color 0 0 0 0)
-	)
-	(junction
 		(at 124.46 68.58)
 		(diameter 0)
@@
 	)
 	(junction
-		(at 234.95 45.72)
-		(diameter 0)
-		(color 0 0 0 0)
-	)
-	(junction
 		(at 53.34 135.89)
 		(diameter 0)
@@
 	)
 	(junction
-		(at 234.95 53.34)
-		(diameter 0)
-		(color 0 0 0 0)
-	)
-	(junction
 		(at 36.83 92.71)
 		(diameter 0)
@@
 	(wire
 		(pts
-			(xy 234.95 53.34) (xy 234.95 52.07)
-		)
-		(stroke
-			(width 0)
-			(type default)
-		)
-	)
-	(wire
-		(pts
 			(xy 82.55 144.78) (xy 82.55 129.54)
 		)
@@
 	(wire
 		(pts
-			(xy 224.79 46.99) (xy 224.79 45.72)
-		)
-		(stroke
-			(width 0)
-			(type default)
-		)
-	)
-	(wire
-		(pts
 			(xy 53.34 109.22) (xy 55.88 109.22)
 		)
@@
 	(wire
 		(pts
-			(xy 224.79 45.72) (xy 234.95 45.72)
-		)
-		(stroke
-			(width 0)
-			(type default)
-		)
-	)
-	(wire
-		(pts
 			(xy 124.46 91.44) (xy 127 91.44)
 		)
@@
 	(wire
 		(pts
-			(xy 234.95 53.34) (xy 252.73 53.34)
+			(xy 231.14 53.34) (xy 234.95 53.34)
 		)
 		(stroke
@@
 	(wire
 		(pts
-			(xy 224.79 52.07) (xy 224.79 53.34)
-		)
-		(stroke
-			(width 0)
-			(type default)
-		)
-	)
-	(wire
-		(pts
 			(xy 161.29 59.69) (xy 193.04 59.69)
 		)
@@
 	(wire
 		(pts
+			(xy 234.95 53.34) (xy 252.73 53.34)
+		)
+		(stroke
+			(width 0)
+			(type default)
+		)
+	)
+	(wire
+		(pts
 			(xy 36.83 190.5) (xy 120.65 190.5)
 		)
@@
 	(wire
 		(pts
+			(xy 234.95 52.07) (xy 234.95 53.34)
+		)
+		(stroke
+			(width 0)
+			(type default)
+		)
+	)
+	(wire
+		(pts
 			(xy 85.09 99.06) (xy 86.36 99.06)
 		)
@@
 	(wire
 		(pts
-			(xy 224.79 53.34) (xy 234.95 53.34)
-		)
-		(stroke
-			(width 0)
-			(type default)
-		)
-	)
-	(wire
-		(pts
 			(xy 243.84 35.56) (xy 243.84 38.1)
 		)
@@
 	(wire
 		(pts
-			(xy 223.52 53.34) (xy 224.79 53.34)
-		)
-		(stroke
-			(width 0)
-			(type default)
-		)
-	)
-	(wire
-		(pts
 			(xy 252.73 90.17) (xy 236.22 90.17)
 		)
@@
 	)
 	(label "GND"
-		(at 223.52 53.34 180)
+		(at 231.14 53.34 180)
 		(effects
 			(font
@@
 					(unit 1)
 				)
-			)
-		)
-	)
-	(symbol
-		(lib_id "Device:C_Small")
-		(at 224.79 49.53 0)
-		(unit 1)
-		(exclude_from_sim no)
-		(in_bom yes)
-		(on_board yes)
-		(dnp no)
-		(property "Reference" "C54"
-			(at 227.33 48.2662 0)
-			(effects
-				(font
-					(size 1.27 1.27)
-				)
-				(justify left)
-			)
-		)
-		(property "Value" "10n"
-			(at 227.33 50.8062 0)
-			(effects
-				(font
-					(size 1.27 1.27)
-				)
-				(justify left)
-			)
-		)
-		(property "Footprint" "Capacitor_SMD:C_0805_2012Metric_Pad1.18x1.45mm_HandSolder"
-			(at 224.79 49.53 0)
-			(effects
-				(font
-					(size 1.27 1.27)
-				)
-				(hide yes)
-			)
-		)
-		(property "Datasheet" ""
-			(at 224.79 49.53 0)
-			(effects
-				(font
-					(size 1.27 1.27)
-				)
-				(hide yes)
-			)
-		)
-		(property "Description" ""
-			(at 224.79 49.53 0)
-			(effects
-				(font
-					(size 1.27 1.27)
-				)
-				(hide yes)
-			)
-		)
-		(property "Sim.Device" ""
-			(at 224.79 49.53 0)
-			(effects
-				(font
-					(size 1.27 1.27)
-				)
-				(hide yes)
-			)
-		)
-		(property "Sim.Type" ""
-			(at 224.79 49.53 0)
-			(effects
-				(font
-					(size 1.27 1.27)
-				)
-				(hide yes)
-			)
-		)
-		(property "mouser" "https://www.mouser.com/ProductDetail/KYOCERA-AVX/08051C103J4Z2A?qs=k4kUdCzLgS7mcJ89o4qEaA%3D%3D"
-			(at 224.79 49.53 0)
-			(effects
-				(font
-					(size 1.27 1.27)
-				)
-				(hide yes)
-			)
-		)
-		(property "specs" "10nF, 5%, 100VDC, X7R, MLCC"
-			(at 224.79 49.53 0)
-			(effects
-				(font
-					(size 1.27 1.27)
-				)
-				(hide yes)
-			)
-		)
-		(property "unit x10" "0.04"
-			(at 224.79 49.53 0)
-			(effects
-				(font
-					(size 1.27 1.27)
-				)
-				(hide yes)
-			)
-		)
-		(property "unit x1" "0.10"
-			(at 224.79 49.53 0)
-			(effects
-				(font
-					(size 1.27 1.27)
-				)
-				(hide yes)
-			)
-		)
-		(property "Sim.Pins" ""
-			(at 224.79 49.53 0)
-			(effects
-				(font
-					(size 1.27 1.27)
-				)
-				(hide yes)
-			)
-		)
-		(property "note" ""
-			(at 224.79 49.53 0)
-			(effects
-				(font
-					(size 1.27 1.27)
-				)
-				(hide yes)
-			)
-		)
-		(pin "2"
-		)
-		(pin "1"
-		)
-		(instances
-			(project "VoltageTap_A"
-				(path "/4b33f365-f3e6-4257-876a-be65258e9424/edbaa468-55b2-41bb-a58d-8607a0c68a40"
-					(reference "C54")
-					(unit 1)
-				)

Commit message: check
Parts:
- removed R78: 10k, Resistor_SMD:R_0805_2012Metric_Pad1.20x1.40mm_HandSolder, symbol Device:R_Small_US
Connections:
- net 7P: now also R96.2; no longer R96.1
- net at C41.2, C42.1, R111.1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: now also R96.1; no longer R96.2
Other:
- moved on the sheet: NT2, R96

Commit message: R96 move
Connections:
- net 7P: now also C41.2, R111.1, R112.2, R96.1; no longer R96.2
- new net: C42.1, R96.2, U36.9 (VC7)
Other:
- moved on the sheet: C41, R96
Changed lines of the file:
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@@
 	(wire
 		(pts
-			(xy 60.96 179.07) (xy 77.47 179.07)
-		)
-		(stroke
-			(width 0)
-			(type default)
-		)
-	)
-	(wire
-		(pts
 			(xy 147.32 74.93) (xy 182.88 74.93)
 		)
@@
 	(wire
 		(pts
-			(xy 77.47 168.91) (xy 77.47 165.1)
+			(xy 77.47 168.91) (xy 77.47 166.37)
 		)
 		(stroke
@@
 	(wire
 		(pts
+			(xy 132.08 41.91) (xy 147.32 41.91)
+		)
+		(stroke
+			(width 0)
+			(type default)
+		)
+	)
+	(wire
+		(pts
 			(xy 124.46 101.6) (xy 124.46 102.87)
 		)
@@
 	(wire
 		(pts
-			(xy 53.34 179.07) (xy 55.88 179.07)
+			(xy 53.34 179.07) (xy 77.47 179.07)
 		)
 		(stroke
@@
 	(wire
 		(pts
-			(xy 107.95 41.91) (xy 147.32 41.91)
+			(xy 107.95 41.91) (xy 127 41.91)
 		)
 		(stroke
@@
 	(wire
 		(pts
-			(xy 77.47 158.75) (xy 77.47 160.02)
+			(xy 77.47 158.75) (xy 77.47 161.29)
 		)
 		(stroke
@@
 	(symbol
 		(lib_id "Device:R_Small_US")
-		(at 58.42 179.07 270)
+		(at 129.54 41.91 90)
+		(mirror x)
 		(unit 1)
 		(exclude_from_sim no)
@@
 		(dnp no)
 		(property "Reference" "R96"
-			(at 59.944 176.53 90)
+			(at 128.016 39.37 90)
 			(effects
 				(font
@@
 		)
 		(property "Value" "100"
-			(at 59.69 181.356 90)
+			(at 128.27 44.196 90)
 			(effects
 				(font
@@
 		)
 		(property "Footprint" "Resistor_SMD:R_1206_3216Metric_Pad1.30x1.75mm_HandSolder"
-			(at 58.42 179.07 0)
+			(at 129.54 41.91 0)
 			(effects
 				(font
@@
 		)
 		(property "Datasheet" ""
-			(at 58.42 179.07 0)
+			(at 129.54 41.91 0)
 			(effects
 				(font
@@
 		)
 		(property "Description" "Resistor, US symbol"
-			(at 58.42 179.07 0)
+			(at 129.54 41.91 0)
 			(effects
 				(font
@@
 		)
 		(property "Sim.Device" ""
-			(at 58.42 179.07 0)
+			(at 129.54 41.91 0)
 			(effects
 				(font
@@
 		)
 		(property "Sim.Type" ""
-			(at 58.42 179.07 0)
+			(at 129.54 41.91 0)
 			(effects
 				(font
@@
 		)
 		(property "mouser" "https://www.mouser.com/ProductDetail/ROHM-Semiconductor/ESR18EZPF1000?qs=sGAEpiMZZMvdGkrng054t4QdAY%2FQ0LwebVJAgfAYbMs%3D"
-			(at 58.42 179.07 0)
+			(at 129.54 41.91 0)
 			(effects
 				(font
@@
 		)
 		(property "specs" "100 omh, thick, anti surge, 1%, 750mW, 200V, -55C, +155C, 100ppm"
-			(at 58.42 179.07 0)
+			(at 129.54 41.91 0)
 			(effects
 				(font
@@
 		)
 		(property "unit x10" "0.055"
-			(at 58.42 179.07 0)
+			(at 129.54 41.91 0)
 			(effects
 				(font
@@
 		)
 		(property "unit x1" "0.17"
-			(at 58.42 179.07 0)
+			(at 129.54 41.91 0)
 			(effects
 				(font
@@
 	(symbol
 		(lib_id "Device:C_Small")
-		(at 77.47 162.56 0)
+		(at 77.47 163.83 0)
 		(mirror y)
 		(unit 1)
@@
 		(dnp no)
 		(property "Reference" "C41"
-			(at 74.93 161.2962 0)
+			(at 74.93 162.5662 0)
 			(effects
 				(font
@@
 		)
 		(property "Value" "100n"
-			(at 74.93 163.8362 0)
+			(at 74.93 165.1062 0)
 			(effects
 				(font
@@
 		)
 		(property "Footprint" "Capacitor_SMD:C_0603_1608Metric_Pad1.08x0.95mm_HandSolder"
-			(at 77.47 162.56 0)
+			(at 77.47 163.83 0)
 			(effects
 				(font
@@
 		)
 		(property "Datasheet" ""
-			(at 77.47 162.56 0)
+			(at 77.47 163.83 0)
 			(effects
 				(font
@@
 		)
 		(property "Description" ""
-			(at 77.47 162.56 0)
+			(at 77.47 163.83 0)
 			(effects
 				(font
@@
 		)
 		(property "mouser" "https://www.mouser.com/ProductDetail/Wurth-Elektronik/885012206095?qs=0KOYDY2FL2%2FIErXVpcsrTQ%3D%3D"
-			(at 77.47 162.56 0)
+			(at 77.47 163.83 0)
 			(effects
 				(font
@@
 		)
 		(property "specs" "100nF, 10%, 50V, X7R, -55C, +125C"
-			(at 77.47 162.56 0)
+			(at 77.47 163.83 0)
 			(effects
 				(font
@@
 		)
 		(property "unit x10" "0.029"
-			(at 77.47 162.56 0)
+			(at 77.47 163.83 0)
 			(effects
 				(font
@@
 		)
 		(property "unit x1" "0.10"
-			(at 77.47 162.56 0)
+			(at 77.47 163.83 0)
 			(effects
 				(font
@@
 		)
 		(property "Sim.Pins" ""
-			(at 77.47 162.56 0)
+			(at 77.47 163.83 0)
 			(effects
 				(font
@@
 		)
 		(property "Sim.Type" ""
-			(at 77.47 162.56 0)
+			(at 77.47 163.83 0)
 			(effects
 				(font
@@
 		)
 		(property "Sim.Device" ""
-			(at 77.47 162.56 0)
+			(at 77.47 163.83 0)
 			(effects
 				(font
@@
 		)
 		(property "note" ""
-			(at 77.47 162.56 0)
+			(at 77.47 163.83 0)
 			(effects
 				(font
@@
 		)
 		(property "unit x50" "0.02"
-			(at 77.47 162.56 0)
+			(at 77.47 163.83 0)
 			(effects
 				(font
@@
 		)
 		(property "unit x100" "0.017"
-			(at 77.47 162.56 0)
+			(at 77.47 163.83 0)
 			(effects
 				(font

Commit message: moo
Connections:
- net 7P: no longer C41.2, R111.1
- net at C42.1, R96.2, U36.9 (VC7): now also C41.2, R111.1
Changed lines of the file:
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@@
 	)
 	(junction
+		(at 77.47 168.91)
+		(diameter 0)
+		(color 0 0 0 0)
+	)
+	(junction
 		(at 24.13 26.67)
 		(diameter 0)
@@
 	)
 	(junction
-		(at 77.47 179.07)
-		(diameter 0)
-		(color 0 0 0 0)
-	)
-	(junction
 		(at 53.34 43.18)
 		(diameter 0)
@@
 	)
 	(junction
-		(at 77.47 168.91)
-		(diameter 0)
-		(color 0 0 0 0)
-	)
-	(junction
 		(at 147.32 107.95)
 		(diameter 0)
@@
 	(wire
 		(pts
-			(xy 77.47 168.91) (xy 77.47 179.07)
-		)
-		(stroke
-			(width 0)
-			(type default)
-		)
-	)
-	(wire
-		(pts
 			(xy 67.31 86.36) (xy 77.47 86.36)
 		)
@@
 	(wire
 		(pts
+			(xy 92.71 40.64) (xy 146.05 40.64)
+		)
+		(stroke
+			(width 0)
+			(type default)
+		)
+	)
+	(wire
+		(pts
 			(xy 60.96 76.2) (xy 77.47 76.2)
 		)
@@
 	(wire
 		(pts
+			(xy 92.71 40.64) (xy 92.71 168.91)
+		)
+		(stroke
+			(width 0)
+			(type default)
+		)
+	)
+	(wire
+		(pts
 			(xy 53.34 119.38) (xy 62.23 119.38)
 		)
@@
 	(wire
 		(pts
-			(xy 77.47 179.07) (xy 93.98 179.07)
+			(xy 53.34 179.07) (xy 93.98 179.07)
 		)
 		(stroke
@@
 	(wire
 		(pts
-			(xy 53.34 179.07) (xy 77.47 179.07)
-		)
-		(stroke
-			(width 0)
-			(type default)
-		)
-	)
-	(wire
-		(pts
 			(xy 134.62 191.77) (xy 134.62 190.5)
 		)
@@
 	(wire
 		(pts
+			(xy 146.05 40.64) (xy 147.32 41.91)
+		)
+		(stroke
+			(width 0)
+			(type default)
+		)
+	)
+	(wire
+		(pts
 			(xy 36.83 157.48) (xy 36.83 158.75)
 		)
@@
 		)
 		(stroke
+			(width 0)
+			(type default)
+		)
+	)
+	(wire
+		(pts
+			(xy 77.47 168.91) (xy 92.71 168.91)
+		)
+		(stroke

Commit message: halp
Parts:
- removed NT2: NetTie_2, NetTie:NetTie-2_SMD_Pad0.5mm, symbol Device:NetTie_2
Connections:
- net Series Sense P is gone; now on net 1N: C53.2, C55.2, C56.2, R56.1, R80.1, U36.17 (VSS)
Changed lines of the file:
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@@
 	)
 	(junction
-		(at 36.83 189.23)
-		(diameter 0)
-		(color 0 0 0 0)
-	)
-	(junction
 		(at 124.46 125.73)
 		(diameter 0)
@@
 	)
 	(junction
+		(at 36.83 189.23)
+		(diameter 0)
+		(color 0 0 0 0)
+	)
+	(junction
 		(at 124.46 68.58)
 		(diameter 0)
@@
 	(wire
 		(pts
-			(xy 36.83 193.04) (xy 36.83 194.31)
-		)
-		(stroke
-			(width 0)
-			(type default)
-		)
-	)
-	(wire
-		(pts
 			(xy 138.43 101.6) (xy 147.32 101.6)
 		)
@@
 	(wire
 		(pts
-			(xy 36.83 189.23) (xy 107.95 189.23)
-		)
-		(stroke
-			(width 0)
-			(type default)
-		)
-	)
-	(wire
-		(pts
 			(xy 182.88 90.17) (xy 195.58 90.17)
 		)
@@
 	(wire
 		(pts
+			(xy 36.83 189.23) (xy 36.83 194.31)
+		)
+		(stroke
+			(width 0)
+			(type default)
+		)
+	)
+	(wire
+		(pts
 			(xy 147.32 97.79) (xy 147.32 101.6)
 		)
@@
 	(wire
 		(pts
+			(xy 36.83 189.23) (xy 107.95 189.23)
+		)
+		(stroke
+			(width 0)
+			(type default)
+		)
+	)
+	(wire
+		(pts
 			(xy 243.84 29.21) (xy 243.84 38.1)
 		)
@@
 					(unit 1)
 				)
-			)
-		)
-	)
-	(symbol
-		(lib_id "Device:NetTie_2")
-		(at 36.83 191.77 270)
-		(unit 1)
-		(exclude_from_sim no)
-		(in_bom no)
-		(on_board yes)
-		(dnp no)
-		(property "Reference" "NT2"
-			(at 39.116 193.04 90)
-			(effects
-				(font
-					(size 1.27 1.27)
-				)
-				(justify left)
-			)
-		)
-		(property "Value" "NetTie_2"
-			(at 35.56 190.5001 90)
-			(effects
-				(font
-					(size 1.27 1.27)
-				)
-				(justify right)
-				(hide yes)
-			)
-		)
-		(property "Footprint" "NetTie:NetTie-2_SMD_Pad0.5mm"
-			(at 36.83 191.77 0)
-			(effects
-				(font
-					(size 1.27 1.27)
-				)
-				(hide yes)
-			)
-		)
-		(property "Datasheet" "~"
-			(at 36.83 191.77 0)
-			(effects
-				(font
-					(size 1.27 1.27)
-				)
-				(hide yes)
-			)
-		)
-		(property "Description" "Net tie, 2 pins"
-			(at 36.83 191.77 0)
-			(effects
-				(font
-					(size 1.27 1.27)
-				)
-				(hide yes)
-			)
-		)
-		(pin "1"
-		)
-		(pin "2"
-		)
-		(instances
-			(project "EVAL MSPM0lG3507 BQ76952"
-				(path "/20ac6af0-79b5-4ba6-aad3-75081d02c913/ba45ce94-ada4-466b-9390-9916681e599d"
-					(reference "NT1")
-					(unit 1)
-				)
-			)
-			(project "EVAL MSPM0lG3507 BQ76952"
-				(path "/4b33f365-f3e6-4257-876a-be65258e9424/edbaa468-55b2-41bb-a58d-8607a0c68a40"
-					(reference "NT2")
-					(unit 1)
-				)

Commit message: dollar store tetris
Parts:
- removed R58, R59, R62, R65, R68, R71, R74, R75, R79, R88, R90, R91, R92, R93, R94, R95, R96, R97, R98: 100, Resistor_SMD:R_1206_3216Metric_Pad1.30x1.75mm_HandSolder, symbol Device:R_Small_US
- added R210, R211, R212, R213, R214, R215, R216, R217, R218, R237, R238, R239, R240, R241, R242, R243, R244, R252, R255: 100, Resistor_SMD:R_0805_2012Metric, symbol Device:R_Small_US
- C201: renamed from C28; now not fitted; now left out of the parts list
- C202: renamed from C29; now not fitted; now left out of the parts list
- C210: renamed from C34; now not fitted; now left out of the parts list
- C218: renamed from C44; now not fitted; now left out of the parts list
- D201: renamed from D22; now not fitted; now left out of the parts list
- D202: renamed from D23; now not fitted; now left out of the parts list
- R201: renamed from R86; now not fitted; now left out of the parts list
- R202: renamed from R61; now not fitted; now left out of the parts list
- R219: renamed from R60; now not fitted; now left out of the parts list
- R220: renamed from R63; now not fitted; now left out of the parts list
- R235: renamed from R56; now not fitted; now left out of the parts list
- R236: renamed from R57; now not fitted; now left out of the parts list
- U201: renamed from U1; footprint Package_TO_SOT_SMD:SOT-89-3_Handsoldering -> Package_TO_SOT_SMD:SOT-89-3; now not fitted; now left out of the parts list
- U202: renamed from U40; footprint Package_TO_SOT_SMD:SOT-89-3_Handsoldering -> Package_TO_SOT_SMD:SOT-89-3; now not fitted; now left out of the parts list
- U203: renamed from U41; footprint Package_TO_SOT_SMD:SOT-89-3_Handsoldering -> Package_TO_SOT_SMD:SOT-89-3
- U204: renamed from U42; footprint Package_TO_SOT_SMD:SOT-89-3_Handsoldering -> Package_TO_SOT_SMD:SOT-89-3
- U205: renamed from U43; footprint Package_TO_SOT_SMD:SOT-89-3_Handsoldering -> Package_TO_SOT_SMD:SOT-89-3
- U206: renamed from U44; footprint Package_TO_SOT_SMD:SOT-89-3_Handsoldering -> Package_TO_SOT_SMD:SOT-89-3
- U207: renamed from U45; footprint Package_TO_SOT_SMD:SOT-89-3_Handsoldering -> Package_TO_SOT_SMD:SOT-89-3
- U208: renamed from U46; footprint Package_TO_SOT_SMD:SOT-89-3_Handsoldering -> Package_TO_SOT_SMD:SOT-89-3
- U209: renamed from U47; footprint Package_TO_SOT_SMD:SOT-89-3_Handsoldering -> Package_TO_SOT_SMD:SOT-89-3
- U210: renamed from U48; footprint Package_TO_SOT_SMD:SOT-89-3_Handsoldering -> Package_TO_SOT_SMD:SOT-89-3
- U211: renamed from U49; footprint Package_TO_SOT_SMD:SOT-89-3_Handsoldering -> Package_TO_SOT_SMD:SOT-89-3
- U212: renamed from U50; footprint Package_TO_SOT_SMD:SOT-89-3_Handsoldering -> Package_TO_SOT_SMD:SOT-89-3
- U213: renamed from U51; footprint Package_TO_SOT_SMD:SOT-89-3_Handsoldering -> Package_TO_SOT_SMD:SOT-89-3
- U214: renamed from U52; footprint Package_TO_SOT_SMD:SOT-89-3_Handsoldering -> Package_TO_SOT_SMD:SOT-89-3
- U215: renamed from U53; footprint Package_TO_SOT_SMD:SOT-89-3_Handsoldering -> Package_TO_SOT_SMD:SOT-89-3
- U216: renamed from U54; footprint Package_TO_SOT_SMD:SOT-89-3_Handsoldering -> Package_TO_SOT_SMD:SOT-89-3
- renumbered C35 to C203, C36 to C204, C37 to C205, C38 to C206, C39 to C207, C40 to C208, C41 to C209, C42 to C211, C43 to C212, C45 to C213, C46 to C214, C47 to C215, C48 to C216, C49 to C217, C53 to C219, C55 to C220, C56 to C221, D24 to D203, D25 to D204, D26 to D205, D27 to D206, D28 to D207, D29 to D208, D30 to D209, D31 to D210, D32 to D211, D33 to D212, D34 to D213, D35 to D214, D36 to D215, D37 to D216, D17 to D217, D18 to D218, R64 to R203, R67 to R204, R70 to R205, R73 to R206, R103 to R207, R106 to R208, R109 to R209, R66 to R221, R69 to R222, R72 to R223, R102 to R224, R105 to R225, R108 to R226, R111 to R227, R112 to R228, R115 to R229, R118 to R230, R121 to R231, R124 to R232, R127 to R233, R87 to R234, R114 to R245, R117 to R246, R120 to R247, R123 to R248, R126 to R249, R129 to R250, R89 to R251, R76 to R253, R77 to R254, R80 to R256, U36 to U217, U37 to U218
Connections:
- net 10P: now also R216.2
- net 11P: now also R215.2
- net 12P: now also R214.2
- net 13P: now also R213.2
- net 14P: now also R212.2
- net 15P: now also R211.2
- net 16P: now also R210.2
- net 1N: now also R244.2
- net 1P: now also R243.2
- net 2P: now also R242.2
- net 3P: now also R241.2
- net 4P: now also R240.2
- net 5P: now also R239.2
- net 6P: now also R238.2
- net 7P: now also R237.2
- net 8P: now also R218.2
- net 9P: now also R217.2
- net BAT: now also R252.1
- net C14Jc: now reaches R203.1, U203.2 (C)
- net at C208.2, C209.1, R226.1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: now also R218.1
- net C13Jc: now reaches R204.1, U204.2 (C)
- net at C204.2, C205.1, R222.1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: now also R214.1
- net at C201.1, U217.48 (VC16): now also C201.2, C202.1, C202.2, C203.1, R219.1, R220.1, U217.1 (VC15), U217.2 (VC14), R210.1, R211.1, R212.1
- net C12Jc: now reaches R205.1, U205.2 (C)
- net at C213.2, C214.1, R247.1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: now also R240.1
- net C7Jc: now reaches R228.1, U210.2 (C)
- net C11Jc: now reaches R206.1, U206.2 (C)
- net C15Jc: now reaches R202.1, U202.2 (C)
- net C4Jc: now reaches R231.1, U213.2 (C)
- net C1Jc: now reaches R234.1, U216.2 (C)
- net at C211.2, C212.1, R245.1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: now also R238.1
- net at C214.2, C215.1, R248.1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: now also R241.1
- net at C221.1, U218.2: now also R255.1
- net C10Jc: now reaches R207.1, U207.2 (C)
- net at C205.2, C206.1, R223.1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: now also R215.1
- net at C215.2, C216.1, R249.1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: now also R242.1
- net at C216.2, C217.1, R250.1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: now also R243.1
- net C2Jc: now reaches R233.1, U215.2 (C)
- net at C212.2, C213.1, R246.1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: now also R239.1
- net at C217.2, R251.1, U217.16 (VC0): now also R244.1
- net C9Jc: now reaches R208.1, U208.2 (C)
- net C3Jc: now reaches R232.1, U214.2 (C)
- net C6Jc: now reaches R229.1, U211.2 (C)
- net at C207.2, C208.1, R225.1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: now also R217.1
- net at C209.2, C211.1, R227.1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: now also R237.1
- net at D218.1 (K): now also R255.2
- net at C206.2, C207.1, R224.1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: now also R216.1
- net at C203.2, C204.1, R221.1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: now also R213.1
- net C8Jc: now reaches R209.1, U209.2 (C)
- net C5Jc: now reaches R230.1, U212.2 (C)
- net C16Jc: now reaches R201.1, U201.2 (C)
- net at D217.1 (K): now also R252.2

Commit message: one must imagine the project being complete
finished voltage tap. should double check wiring
Connections:
- net 1N: now also C210.1, C218.1, R235.2, U217.18 (SRP)
- net Series Sense N: now also C210.2, C218.2, R236.2, U217.20 (SRN)

Commit message: big things are comming
still cheaper than OSHPARK .
Parts:
- U217: mouser https://www.mouser.com/ProductDetail/Texas-Instruments/BQ7695204PFBR?qs=iLbezkQI%252BsiEQall6bGLHw%3D%3D&srsltid=AfmBOortQS0ZF7nyGONpPu2GM9H0Yt_aAZOvNG6JzQEqbOzrseuaG7sd -> https://www.mouser.com/ProductDetail/Texas-Instruments/BQ7697204PFBR?qs=mELouGlnn3d1bfb90Grt5w%3D%3D&srsltid=AfmBOorK_P5jnZWaZmdvfsHDZVrwPG13jxJWTt6B3VclUTUR5_6Rvmss
Changed lines of the file:
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@@
 			)
 		)
-		(property "mouser" "https://www.mouser.com/ProductDetail/Texas-Instruments/BQ7695204PFBR?qs=iLbezkQI%252BsiEQall6bGLHw%3D%3D&srsltid=AfmBOortQS0ZF7nyGONpPu2GM9H0Yt_aAZOvNG6JzQEqbOzrseuaG7sd"
+		(property "mouser" "https://www.mouser.com/ProductDetail/Texas-Instruments/BQ7697204PFBR?qs=mELouGlnn3d1bfb90Grt5w%3D%3D&srsltid=AfmBOorK_P5jnZWaZmdvfsHDZVrwPG13jxJWTt6B3VclUTUR5_6Rvmss"
 			(at 195.58 62.23 0)
 			(effects
