File: hardware/mini Orion TEM/thermistors.kicad_sch (KiCad schematic)
At the start: 21 parts

Commit message: shuflle master
Parts:
- added C208, C209: 220n, Capacitor_SMD:C_0805_2012Metric_Pad1.18x1.45mm_HandSolder, symbol Device:C_Small
- added R208: 2.4k, Resistor_SMD:R_0805_2012Metric_Pad1.20x1.40mm_HandSolder, symbol Device:R_Small_US
- added TH208: Thermistor_US, Resistor_SMD:R_1206_3216Metric, symbol Device:Thermistor_US
- added U201: SN74LV4051A-Q1, Package_SO:Texas_DYY0016A_TSOT-23-16_2x4.2mm_P0.5mm, symbol zzLocalLibrary:SN74LV4051ADYYR
Connections:
- net GND: now also C208.2, C209.2, TH208.2, U201.6 (Inh), U201.7 (GND), U201.8 (GND)
- net at R202.2: now also U201.14 (X1)
- net at R201.2: now also U201.13 (X0)
- net at R204.2: now also U201.12 (X3)
- net at R207.2: now also U201.2 (X6)
- net at R203.2: now also U201.15 (X2)
- net at R205.2: now also U201.1 (X4)
- net at R206.2: now also U201.5 (X5)
- new net: C208.1, R208.1, TH208.1
- new net: R208.2, U201.4 (X7)
- new net A: U201.11 (A)
- new net Aout1: U201.3 (X)
- new net B: U201.10 (B)
- new net C: U201.9 (C)
- new net VDD: C209.1, U201.16 (VCC)
Other:
- moved on the sheet: C201, C202, C203, C204, C205, C206, C207, R201, R202, R203, R204, R205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

Commit message: NOTHING MATCHES CAD!!!!!!!!!
YIPPERS!!
Parts:
- TH201, TH202, TH203, TH204, TH205, TH206, TH207, TH208: footprint Resistor_SMD:R_1206_3216Metric -> zzLocalLibraries-Footprints:FPC thermistor strip 2x2mm
Other:
- moved on the sheet: C206, C207, C208, R206, R207, R208

Commit message: more shuffling
Connections:
- net Aout1: now also C209.1
- net VDD: no longer C209.1
Other:
- moved on the sheet: C209
Changed lines of the file:
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@@
-	)
-	(junction
-		(at 114.3 71.12)
-		(diameter 0)
-		(color 0 0 0 0)
 	)
 	(junction
@@
 	)
 	(junction
-		(at 116.84 63.5)
-		(diameter 0)
-		(color 0 0 0 0)
-	)
-	(junction
-		(at 116.84 71.12)
-		(diameter 0)
-		(color 0 0 0 0)
-	)
-	(junction
 		(at 74.93 45.72)
 		(diameter 0)
@@
 	)
 	(junction
+		(at 125.73 71.12)
+		(diameter 0)
+		(color 0 0 0 0)
+	)
+	(junction
+		(at 113.03 71.12)
+		(diameter 0)
+		(color 0 0 0 0)
+	)
+	(junction
 		(at 64.77 57.15)
 		(diameter 0)
@@
 	)
 	(junction
+		(at 125.73 45.72)
+		(diameter 0)
+		(color 0 0 0 0)
+	)
+	(junction
 		(at 74.93 67.31)
 		(diameter 0)
@@
 	(wire
 		(pts
+			(xy 125.73 60.96) (xy 125.73 71.12)
+		)
+		(stroke
+			(width 0)
+			(type default)
+		)
+	)
+	(wire
+		(pts
 			(xy 64.77 111.76) (xy 64.77 118.11)
 		)
@@
 	(wire
 		(pts
-			(xy 116.84 63.5) (xy 116.84 64.77)
-		)
-		(stroke
-			(width 0)
-			(type default)
-		)
-	)
-	(wire
-		(pts
 			(xy 74.93 85.09) (xy 74.93 90.17)
 		)
@@
 	(wire
 		(pts
-			(xy 116.84 71.12) (xy 124.46 71.12)
-		)
-		(stroke
-			(width 0)
-			(type default)
-		)
-	)
-	(wire
-		(pts
 			(xy 73.66 57.15) (xy 74.93 57.15)
 		)
@@
 	(wire
 		(pts
+			(xy 125.73 45.72) (xy 113.03 45.72)
+		)
+		(stroke
+			(width 0)
+			(type default)
+		)
+	)
+	(wire
+		(pts
 			(xy 83.82 48.26) (xy 83.82 57.15)
 		)
@@
 	(wire
 		(pts
-			(xy 116.84 69.85) (xy 116.84 71.12)
-		)
-		(stroke
-			(width 0)
-			(type default)
-		)
-	)
-	(wire
-		(pts
 			(xy 64.77 90.17) (xy 64.77 95.25)
 		)
@@
 	(wire
 		(pts
-			(xy 113.03 63.5) (xy 116.84 63.5)
-		)
-		(stroke
-			(width 0)
-			(type default)
-		)
-	)
-	(wire
-		(pts
 			(xy 64.77 118.11) (xy 67.31 118.11)
 		)
@@
 	(wire
 		(pts
+			(xy 125.73 45.72) (xy 125.73 55.88)
+		)
+		(stroke
+			(width 0)
+			(type default)
+		)
+	)
+	(wire
+		(pts
 			(xy 86.36 78.74) (xy 82.55 78.74)
 		)
@@
 	(wire
 		(pts
+			(xy 113.03 71.12) (xy 113.03 68.58)
+		)
+		(stroke
+			(width 0)
+			(type default)
+		)
+	)
+	(wire
+		(pts
 			(xy 72.39 118.11) (xy 74.93 118.11)
 		)
@@
 	(wire
 		(pts
+			(xy 129.54 45.72) (xy 125.73 45.72)
+		)
+		(stroke
+			(width 0)
+			(type default)
+		)
+	)
+	(wire
+		(pts
 			(xy 64.77 118.11) (xy 64.77 123.19)
 		)
@@
 	(wire
 		(pts
+			(xy 129.54 71.12) (xy 125.73 71.12)
+		)
+		(stroke
+			(width 0)
+			(type default)
+		)
+	)
+	(wire
+		(pts
 			(xy 74.93 45.72) (xy 77.47 45.72)
 		)
@@
 	(wire
 		(pts
-			(xy 113.03 71.12) (xy 114.3 71.12)
-		)
-		(stroke
-			(width 0)
-			(type default)
-		)
-	)
-	(wire
-		(pts
 			(xy 74.93 40.64) (xy 74.93 45.72)
 		)
@@
 	(wire
 		(pts
-			(xy 114.3 68.58) (xy 114.3 71.12)
-		)
-		(stroke
-			(width 0)
-			(type default)
-		)
-	)
-	(wire
-		(pts
 			(xy 82.55 90.17) (xy 87.63 90.17)
 		)
@@
 	(wire
 		(pts
-			(xy 113.03 68.58) (xy 114.3 68.58)
-		)
-		(stroke
-			(width 0)
-			(type default)
-		)
-	)
-	(wire
-		(pts
 			(xy 74.93 52.07) (xy 74.93 57.15)
 		)
@@
 	(wire
 		(pts
-			(xy 116.84 63.5) (xy 124.46 63.5)
+			(xy 125.73 71.12) (xy 113.03 71.12)
 		)
 		(stroke
@@
 		(pts
 			(xy 73.66 123.19) (xy 74.93 123.19)
-		)
-		(stroke
-			(width 0)
-			(type default)
-		)
-	)
-	(wire
-		(pts
-			(xy 114.3 71.12) (xy 116.84 71.12)
 		)
 		(stroke
@@
 	(hierarchical_label "Aout1"
 		(shape bidirectional)
-		(at 113.03 45.72 0)
+		(at 129.54 45.72 0)
 		(effects
 			(font
@@
 	(hierarchical_label "VDD"
 		(shape input)
-		(at 124.46 63.5 0)
+		(at 113.03 63.5 0)
 		(effects
 			(font
@@
 	(hierarchical_label "GND"
 		(shape input)
-		(at 124.46 71.12 0)
+		(at 129.54 71.12 0)
 		(effects
 			(font
@@
 	(symbol
 		(lib_id "Device:C_Small")
-		(at 116.84 67.31 0)
+		(at 125.73 58.42 0)
 		(unit 1)
 		(exclude_from_sim no)
@@
 		(dnp no)
 		(property "Reference" "C209"
-			(at 119.38 66.0462 0)
+			(at 128.27 57.1562 0)
 			(effects
 				(font
@@
 		)
 		(property "Value" "220n"
-			(at 119.38 68.5862 0)
+			(at 128.27 59.6962 0)
 			(effects
 				(font
@@
 		)
 		(property "Footprint" "Capacitor_SMD:C_0805_2012Metric_Pad1.18x1.45mm_HandSolder"
-			(at 116.84 67.31 0)
+			(at 125.73 58.42 0)
 			(effects
 				(font
@@
 		)
 		(property "Datasheet" "https://www.mouser.com/ProductDetail/Samsung-Electro-Mechanics/CL31B224KBFNNNF?qs=sGAEpiMZZMsh%252B1woXyUXj7iNKXiFkBmw7C%252BUlKpuDJ8%3D"
-			(at 116.84 67.31 0)
+			(at 125.73 58.42 0)
 			(effects
 				(font
@@
 		)
 		(property "Description" ""
-			(at 116.84 67.31 0)
+			(at 125.73 58.42 0)
 			(effects
 				(font
@@
 		)
 		(property "Sim.Device" ""
-			(at 116.84 67.31 0)
+			(at 125.73 58.42 0)
 			(effects
 				(font
@@
 		)
 		(property "Sim.Type" ""
-			(at 116.84 67.31 0)
+			(at 125.73 58.42 0)
 			(effects
 				(font
@@
 		)
 		(property "mouser" "https://www.mouser.com/ProductDetail/Samsung-Electro-Mechanics/CL21B224KCFSFNE?qs=664zcAxDQ0l4Y1eUk6Zc1g%3D%3D"
-			(at 116.84 67.31 0)
+			(at 125.73 58.42 0)
 			(effects
 				(font
@@
 		)
 		(property "specs" "100VDC, X7R, 10%, -55C, +125C, 220nF"
-			(at 116.84 67.31 0)
+			(at 125.73 58.42 0)
 			(effects
 				(font
@@
 		)
 		(property "unit x10" "0.054"
-			(at 116.84 67.31 0)
+			(at 125.73 58.42 0)
 			(effects
 				(font
@@
 		)
 		(property "Sim.Pins" ""
-			(at 116.84 67.31 0)
+			(at 125.73 58.42 0)
 			(effects
 				(font
@@
 		)
 		(property "note" ""
-			(at 116.84 67.31 0)
-			(effects
-				(font
+			(at 125.73 58.42 0)
+			(effects
+				(font
