File: hardware/mini Orion TEM/mini Orion TEM.kicad_pcb (KiCad board)
At the start: 2 copper layers, 319.7 x 58.4 mm, 109 parts, among them J101 HRLV, J102 VT bridge, SW101 SW_DIP_x06, U101 VT harness, U102 AP7384-50SA, U103 MCP2542FDxMF, U104 ISOW7741, U105 XMSM0G3507SDGS28R, U201 SN74LV4051A-Q1, U301 SN74LV4051A-Q1

Commit message: NOTHING MATCHES CAD!!!!!!!!!
YIPPERS!!
Parts:
- added R104: 100k, Resistor_SMD:R_1206_3216Metric_Pad1.30x1.75mm_HandSolder, F.Cu at (153.4, 99.6)
- R102: value 4.99k -> 22.1k; footprint Resistor_SMD:R_1206_3216Metric_Pad1.30x1.75mm_HandSolder -> Resistor_SMD:R_0805_2012Metric_Pad1.20x1.40mm_HandSolder
- R103: value 100k -> 4.99k
- TH201, TH202, TH203, TH204, TH205, TH206, TH207, TH208, TH301, TH302, TH303, TH304, TH305, TH306, TH307, TH308: footprint Resistor_SMD:R_1206_3216Metric -> zzLocalLibraries-Footprints:FPC thermistor strip 2x2mm
- moved H101 9.87 mm to (76.6, 160.2)
- moved U101 4.05 mm to (53.2, 123.9)
- moved TP101 1.20 mm to (44.0, 169.6)
- moved TP115 1.20 mm to (44.0, 120.2)
Connections:
- C107 pad 2: Net-(U105-VCORE) -> +3V3
- C108 pad 2: +3V3 -> Net-(U105-VCORE)
- D102 pad 2: Net-(D102-A) -> unconnected-(D102-A-Pad2)
- R102 pad 1: GND -> Net-(U105-NRST)
- R102 pad 2: Net-(D102-K) -> +3V3
- R103 pad 1: Net-(U105-PA2_/_ROSC) -> GND
- R103 pad 2: GND -> Net-(D102-K)
- U105 pad 14: Net-(D102-A) -> unconnected-(U105-PA9_/_RTC_OUT_/_CLK_OUT-Pad14)
- U105 pad 22: unconnected-(U105-PA19/SWDIO-Pad22) -> /SWDIO
- U105 pad 23: unconnected-(U105-PA20/SWCLK-Pad23) -> /SWCLK
- U105 pad 4: unconnected-(U105-PA0-Pad4) -> /UART_TX
- U105 pad 5: unconnected-(U105-PA1-Pad5) -> /UART_A1
- U105 pad 6: unconnected-(U105-NRST-Pad6) -> Net-(U105-NRST)

Commit message: vt routing complete
Parts:
- moved F114 267.8 mm to (327.1, 118.8)
- moved F113 262.9 mm to (305.2, 171.0)
- moved F111 226.6 mm to (260.2, 171.0)
- moved F112 226.0 mm to (282.3, 118.8)
- moved TH306 205.2 mm to (344.1, 135.5)
- moved F109 189.6 mm to (215.1, 171.0)
- moved F110 189.2 mm to (237.5, 118.8)
- moved F107 159.0 mm to (170.1, 171.0)
- moved F108 148.7 mm to (192.8, 118.8)
- moved F105 124.6 mm to (125.0, 171.0)
- moved F106 112.4 mm to (148.0, 118.8)
- moved F103 109.4 mm to (80.0, 171.0)
- moved F101 93.2 mm to (44.0, 152.0), turned to -90 degrees
- moved F104 76.1 mm to (103.3, 118.8)
- moved F115 64.5 mm to (44.0, 139.0), turned to 90 degrees
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Routing:
- net /VT9: track 0.00 -> 427.3 mm
- net /VT10/-13: track 0.00 -> 400.5 mm, vias 0 -> 3
- net /VT1: track 0.00 -> 389.5 mm, vias 0 -> 1
- net /VT5: track 0.00 -> 378.8 mm, vias 0 -> 1
- net /VT8: track 0.00 -> 374.3 mm, vias 0 -> 1
- net /VT15: track 0.00 -> 353.3 mm, vias 0 -> 1
- net /VT6: track 0.00 -> 336.3 mm, vias 0 -> 3
- net /VT4: track 0.00 -> 334.5 mm, vias 0 -> 1
- net /VT2: track 0.00 -> 325.0 mm, vias 0 -> 2
- net /VT13: track 0.00 -> 324.8 mm, vias 0 -> 4
- net /VT-1: track 0.00 -> 322.5 mm, vias 0 -> 2
- net /VT16: track 0.00 -> 319.0 mm
- net /VT14: track 0.00 -> 312.7 mm, vias 0 -> 4
- net /VT3: track 0.00 -> 302.7 mm, vias 0 -> 2
- net /VT7: track 0.00 -> 298.4 mm, vias 0 -> 2
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
Commit message: brain rot maxxing
rout rout trout rout
Parts:
- added REF**: Symbol_HighVoltage_Triangle_8x7mm_Copper, Symbol:Symbol_HighVoltage_Triangle_8x7mm_Copper, B.Cu at (69.1, 168.3)
- U102: footprint Package_TO_SOT_SMD:SOT-23 -> Package_TO_SOT_SMD:SOT-23-3
- moved C301 129.6 mm to (277.2, 191.8)
- moved C302 129.6 mm to (277.2, 194.8)
- moved C303 129.6 mm to (277.2, 197.8)
- moved C304 129.6 mm to (277.2, 200.8)
- moved C305 129.6 mm to (277.2, 203.8)
- moved C306 129.6 mm to (277.2, 206.9)
- moved C307 129.6 mm to (277.2, 209.9)
- moved C308 129.6 mm to (277.2, 212.9)
- moved C309 129.6 mm to (277.2, 215.9)
- moved R301 129.6 mm to (287.6, 191.8)
- moved R302 129.6 mm to (287.6, 194.7)
- moved R303 129.6 mm to (287.6, 197.7)
- moved R304 129.6 mm to (287.6, 200.6)
- moved R305 129.6 mm to (287.6, 203.6)
- moved R306 129.6 mm to (287.6, 206.5)
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Routing:
- net Net-(U102-VO): track 0.00 -> 38.4 mm
- net Net-(U104-V_{ISOIN}): track 0.00 -> 25.6 mm, vias 0 -> 2
- net /CAN-: track 0.00 -> 20.9 mm
- net /CAN+: track 0.00 -> 20.6 mm
- net /GLV+: track 0.00 -> 11.7 mm
- net /GLV-: track 0.00 -> 8.23 mm, vias 0 -> 19
- net Net-(U103-TXD): track 0.00 -> 7.44 mm
- net Net-(D101-K): track 0.00 -> 7.42 mm
- net Net-(U103-RXD): track 0.00 -> 6.64 mm
- net /IL+: track 0.00 -> 5.92 mm
- net GND: track 0.00 -> 4.71 mm, vias 0 -> 78
- net Net-(FB101-Pad2): track 0.00 -> 3.68 mm
- net +3V3: track 0.00 -> 2.41 mm
- added copper zone on B.Cu, net /GLV-
- added copper zone on F.Cu, net /GLV-
- added copper zone on B.Cu, net GND
- added copper zone on F.Cu, net GND
Other:
- board text added: "HV Isolation 600Vdc"
- board text added: "High Voltage"
- board text added: "Low Voltage"
- board text added: "TEM integrated Voltage Tap 1.0 github.com/Gregification/BeeMS/ 1/22/2025 - pinning & hardware info: {dblquote}/hardware/mini Orion TEM/{dblquote} - software: {dblquote}/miniOrionTEM{dblquote}"
- board text added: "extra safety isolation 600Vdc"

Commit message: more shuffling
Parts:
- removed C103: 10u, Capacitor_SMD:C_1206_3216Metric_Pad1.33x1.80mm_HandSolder
- removed C107: 220n, Capacitor_SMD:C_0805_2012Metric_Pad1.18x1.45mm_HandSolder
- removed R102: 22.1k, Resistor_SMD:R_0805_2012Metric_Pad1.20x1.40mm_HandSolder
- removed REF**: Symbol_HighVoltage_Triangle_8x7mm_Copper, Symbol:Symbol_HighVoltage_Triangle_8x7mm_Copper
- added C109: 10u, Capacitor_SMD:C_1206_3216Metric_Pad1.33x1.80mm_HandSolder, F.Cu at (181.6, 150.2)
- added C110: 10u, Capacitor_SMD:C_1206_3216Metric_Pad1.33x1.80mm_HandSolder, F.Cu at (181.6, 145.5)
- added J103: SWD, Connector_PinHeader_2.54mm:PinHeader_1x02_P2.54mm_Vertical, F.Cu at (201.2, 143.9)
- moved C204 204.3 mm to (340.4, 134.9)
- moved R204 194.8 mm to (340.4, 136.9), turned to 180 degrees
- moved TH204 193.6 mm to (334.9, 135.0), turned to 180 degrees
- moved TH304 156.5 mm to (133.5, 153.8), turned to 180 degrees
- moved R304 156.2 mm to (139.2, 151.8)
- moved C201 155.8 mm to (285.6, 136.1), turned to 180 degrees
- moved TH201 155.4 mm to (290.5, 136.0)
- moved R201 147.1 mm to (285.6, 138.1), turned to 180 degrees
- moved C304 145.8 mm to (139.2, 153.8)
- moved R301 132.7 mm to (161.0, 152.0)
- moved TH301 132.1 mm to (155.9, 154.0), turned to 180 degrees
- moved C301 122.2 mm to (161.0, 154.0)
- moved R302 121.0 mm to (173.8, 153.6), turned to 90 degrees
- moved TH202 113.7 mm to (245.7, 135.4)
- moved C202 113.2 mm to (239.8, 135.2), turned to 180 degrees
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Connections:
- net /UART_A1 renamed /UART_RX
- C209 pad 1: +3V3 -> /TB1_out
- C309 pad 1: +3V3 -> /TB2_out
- D102 pad 2: unconnected-(D102-A-Pad2) -> Net-(D102-A)
- U105 pad 11: unconnected-(U105-PA4_/_LFCLK_IN_/_LFXOUT-Pad11) -> +3V3
- U105 pad 12: unconnected-(U105-PA5/HFXIN/FCC_IN-Pad12) -> /TB2_A
- U105 pad 13: unconnected-(U105-PA6/HFCLK_IN/HFXOUT-Pad13) -> /TB2_B
- U105 pad 14: unconnected-(U105-PA9_/_RTC_OUT_/_CLK_OUT-Pad14) -> /TB2_C
- U105 pad 15: unconnected-(U105-PA10/CLK_OUT-Pad15) -> Net-(D102-A)
- U105 pad 16: unconnected-(U105-PA11-Pad16) -> /sw_unit_id_4
- U105 pad 17: unconnected-(U105-PA14/CLK_OUT/A0_12-Pad17) -> /TB2_out
- U105 pad 18: unconnected-(U105-PA15/A1_0-Pad18) -> /sw_unit_id_3
- U105 pad 19: unconnected-(U105-PA16/A1_1/FCC_IN-Pad19) -> /sw_unit_id_2
- U105 pad 20: unconnected-(U105-PA17/A1_2-Pad20) -> /sw_unit_id_1
- U105 pad 21: unconnected-(U105-PA18/A1_3-Pad21) -> /sw_can_baud_2
- U105 pad 24: unconnected-(U105-PA21/A1_7/VREF--Pad24) -> /sw_can_baud_1
- U105 pad 25: unconnected-(U105-PA22/CLK_OUT/A0_7-Pad25) -> /TB1_out
- U105 pad 26: unconnected-(U105-PA23/VREF+-Pad26) -> /TB1_A
- U105 pad 27: unconnected-(U105-PA24/A0_3-Pad27) -> /TB1_B
- U105 pad 28: unconnected-(U105-PA25/A0_2-Pad28) -> /TB1_C
- U105 pad 6: Net-(U105-NRST) -> +3V3
- U201 pad 10: /thermistor bank 1/B -> /TB1_B
- U201 pad 11: /thermistor bank 1/A -> /TB1_A
- U201 pad 3: /thermistor bank 1/Aout1 -> /TB1_out
- U201 pad 9: /thermistor bank 1/C -> /TB1_C
- U301 pad 10: /thermistor bank 1/B -> /TB2_B
- U301 pad 11: /thermistor bank 1/A -> /TB2_A
- U301 pad 3: /thermistor bank 2/Aout1 -> /TB2_out
- U301 pad 9: /thermistor bank 1/C -> /TB2_C
Routing:
- net Net-(U201-X3): track 0.00 -> 149.6 mm
- net Net-(U301-X5): track 0.00 -> 120.5 mm
- net +3V3: track 2.41 -> 103.8 mm
- net Net-(U301-X7): track 0.00 -> 96.3 mm
- net Net-(U201-X0): track 0.00 -> 93.8 mm
- net Net-(U104-OUTC): track 0.00 -> 83.3 mm
- net Net-(U104-IND): track 0.00 -> 79.7 mm
- net Net-(U201-X5): track 0.00 -> 75.2 mm
- net Net-(U301-X6): track 0.00 -> 70.3 mm
- net Net-(U201-X7): track 0.00 -> 69.9 mm
- net Net-(U201-X6): track 0.00 -> 65.0 mm
- net Net-(U301-X3): track 0.00 -> 50.2 mm
- net Net-(U301-X4): track 0.00 -> 49.6 mm
- net Net-(U201-X1): track 0.00 -> 48.1 mm
- net Net-(D102-A): track 0.00 -> 34.6 mm
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
Commit message: drc passing
Parts:
- added H106: MountingHole, MountingHole:MountingHole_3.5mm, F.Cu at (156.9, 146.2)
- added J104: Conn_01x02_Socket, Connector_PinHeader_2.00mm:PinHeader_1x02_P2.00mm_Vertical, F.Cu at (83.7, 144.7)
- moved D102 48.9 mm to (273.0, 146.4)
- moved R103 48.9 mm to (273.0, 144.3)
- moved H104 32.9 mm to (237.6, 143.6)
- moved D101 2.01 mm to (84.2, 150.4)
- moved C101 1.90 mm to (84.5, 155.3), turned to 180 degrees
- moved C204 1.00 mm to (339.4, 134.9)
- moved R204 1.00 mm to (339.4, 136.9)
Routing:
- net Net-(D102-A): track 34.6 -> 83.1 mm
- net /VT9: track 427.3 -> 408.2 mm
- net GND: track 20.4 -> 31.4 mm
- net /VT5: track 378.8 -> 371.8 mm
- net /VT6: track 336.3 -> 330.2 mm
- net /VT15: track 353.3 -> 348.0 mm
- net /VT14: track 312.7 -> 308.0 mm
- net /VT13: track 324.8 -> 320.2 mm
- net /VT8: track 374.3 -> 369.8 mm
- net /GLV+: track 6.37 -> 10.8 mm
- net /VT10/-13: track 400.5 -> 396.2 mm
- net /VT3: track 302.7 -> 298.5 mm
- net /VT4: track 334.5 -> 330.4 mm
- net /VT2: track 325.0 -> 321.0 mm
- net /VT7: track 298.4 -> 296.3 mm
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Other:
- outline, holes or cut-outs redrawn
- board text added: "0 : 250k 1 : 500k 2 : 1M 3 : 1Ma 2Md"
- board text added: "CAN baud A"
- board text added: "CAN+ CAN-"
- board text added: "GLV+"
- board text added: "GLV-"
- board text added: "IL+"
- board text added: "IL-"
- board text added: "TOP"
- board text added: "Unit ID"
- board text added: "^ 0"
- board text added: "blink == good no-blink == bad"
- board text added: "bridge connection to bottom board"
- board text added: "stuff fan connector here"
- board text removed: "extra safety isolation 600Vdc"

Commit message: Masterboard modbus working
Parts:
- added U106: TLP290, Package_SO:SOP-4_4.4x2.6mm_P1.27mm, F.Cu at (364.2, 145.7)
- added U705: TLP155E, zzLocalLibraries-Footprints:U_SO6_11-4L1_TOS-M, F.Cu at (357.4, 154.3)

Commit message: kil!
Parts:
- removed U106: TLP290, Package_SO:SOP-4_4.4x2.6mm_P1.27mm
- removed U705: TLP155E, zzLocalLibraries-Footprints:U_SO6_11-4L1_TOS-M
- added J2: Fan enable, Connector_PinHeader_2.00mm:PinHeader_1x02_P2.00mm_Vertical, F.Cu at (146.2, 147.8)
- added R151: 220, Resistor_SMD:R_1206_3216Metric, F.Cu at (165.6, 146.6)
- added U1: TLP290, Package_SO:SOP-4_4.4x2.6mm_P1.27mm, F.Cu at (152.1, 146.9)
- moved H106 21.7 mm to (135.2, 145.8)
- moved TH308 3.20 mm to (290.7, 151.0)
- moved TH307 2.74 mm to (268.3, 151.5)
- moved F112 2.69 mm to (282.3, 121.5)
- moved TH305 2.13 mm to (245.7, 152.3)
- moved TH301 1.93 mm to (157.7, 153.4)
- moved F108 1.75 mm to (192.5, 120.6)
- moved TH202 1.71 mm to (245.8, 137.1)
- moved F110 1.55 mm to (237.6, 120.4)
- moved TH303 1.46 mm to (224.0, 152.7)
- moved TH205 1.45 mm to (156.9, 136.8)
- moved C301 1.43 mm to (162.1, 154.8)
- moved R304 1.42 mm to (138.6, 153.1)
- moved R301 1.35 mm to (162.1, 152.8)
- moved F114 1.35 mm to (326.9, 120.2)
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Connections:
- U105 pad 4: /UART_TX -> /TIMG8_C2
- U105 pad 5: /UART_RX -> unconnected-(U105-PA1-Pad5)
Routing:
- net /TIMG8_C2: track 0.00 -> 22.3 mm, vias 0 -> 2
- net Net-(R151-Pad1): track 0.00 -> 9.02 mm
- net +3V3: track 103.8 -> 112.1 mm
- net Net-(U301-X3): track 50.2 -> 56.0 mm
- net Net-(U104-OUTC): track 83.3 -> 88.8 mm
- net GND: track 31.4 -> 25.9 mm, vias 116 -> 114
- net Net-(U104-IND): track 79.7 -> 83.4 mm
- net Net-(J2-Pin_2): track 0.00 -> 2.91 mm
- net Net-(J2-Pin_1): track 0.00 -> 2.88 mm
- net Net-(U201-X5): track 75.2 -> 77.2 mm
- net Net-(C308-Pad1): track 4.91 -> 6.75 mm
- net Net-(C307-Pad1): track 8.30 -> 10.00 mm
- net Net-(C303-Pad1): track 4.44 -> 5.76 mm
- net Net-(F110-Pad2): track 6.20 -> 4.90 mm
- net Net-(F106-Pad2): track 6.10 -> 4.89 mm
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
Commit message: aeclnkaeckl
Parts:
- moved H105 3.94 mm to (74.0, 133.0)
- moved H101 3.18 mm to (74.0, 160.0)
Other:
- outline, holes or cut-outs redrawn
- board text added: "0 : 250k 1 : 500k 2 : 500k/A 2M/D 3 : 1M"
- board text removed: "0 : 250k 1 : 500k 2 : 1M 3 : 1Ma 2Md"
