File: hardware/mini Orion TEM/thermistor bank 2.kicad_sch (KiCad schematic)
At the start: 26 parts, among them U201 SN74LV4051A-Q1

Commit message: grunt
review
Parts:
- renumbered C201 to C301, C202 to C302, C203 to C303, C204 to C304, C205 to C305, C206 to C306, C207 to C307, C208 to C308, C209 to C309, R201 to R301, R202 to R302, R203 to R303, R204 to R304, R205 to R305, R206 to R306, R207 to R307, R208 to R308, TH201 to TH301, TH202 to TH302, TH203 to TH303, TH204 to TH304, TH205 to TH305, TH206 to TH306, TH207 to TH307, TH208 to TH308, U201 to U301
Connections:
- net at R308.2: now also U301.2 (X6); no longer U301.1 (X4)
- net at R302.2: now also U301.5 (X5); no longer U301.14 (X1)
- net at R301.2: now also U301.4 (X7); no longer U301.15 (X2)
- net at U301.12 (X3): now also R307.2; no longer R303.2
- net at U301.13 (X0): now also R305.2; no longer R304.2
- net at R306.2: now also U301.1 (X4); no longer U301.2 (X6)
- new net: R304.2, U301.14 (X1)
- new net: R303.2, U301.15 (X2)
