File: hardware/mini Orion TEM/mini Orion TEM.kicad_sch (KiCad schematic)
At the start: 86 parts, among them J101 HRLV, J102 bridge to bottom board, J103 SWD, J104 fan pwr source, J105 VT harness, J106 fan PWR, J2 Fan enable, Q101 DI035P04PT, Q102 MMBT5550L, SW101 SW_DIP_x06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

Commit message: freecad is yippie
Parts:
- removed C113, C114: 10u, Capacitor_SMD:C_1206_3216Metric_Pad1.33x1.80mm_HandSolder, symbol Device:C_Small
- added C102: 22u, Capacitor_SMD:C_0805_2012Metric_Pad1.18x1.45mm_HandSolder, symbol Device:C_Small
- C101: value 10u -> 1u; footprint Capacitor_SMD:C_1206_3216Metric_Pad1.33x1.80mm_HandSolder -> Capacitor_SMD:C_0603_1608Metric_Pad1.08x0.95mm_HandSolder; mouser https://www.mouser.com/ProductDetail/Samsung-Electro-Mechanics/CL31A106KBHNNNE?qs=sGAEpiMZZMsh%252B1woXyUXjxqcB7t9naYpzWmpMbMJIKQ%3D -> https://www.mouser.com/ProductDetail/Samsung-Electro-Mechanics/CL10A105KA8NNND?qs=sGAEpiMZZMsh%252B1woXyUXj9e2R%2FOkAO5oyLEB2KToctI%3D; specs 10uF, 50VDC, X5R, 10%, -55C, +85C -> 1uF, 25VDC, 10%, -55C, +125C; unit x1 (none) -> 0.15; unit x10 0.07 -> 0.061
- C104, C105, C107, C110, C111: value 10u -> 22u; footprint Capacitor_SMD:C_1206_3216Metric_Pad1.33x1.80mm_HandSolder -> Capacitor_SMD:C_0805_2012Metric_Pad1.18x1.45mm_HandSolder; mouser https://www.mouser.com/ProductDetail/Samsung-Electro-Mechanics/CL31A106KBHNNNE?qs=sGAEpiMZZMsh%252B1woXyUXjxqcB7t9naYpzWmpMbMJIKQ%3D -> https://www.mouser.com/ProductDetail/Samsung-Electro-Mechanics/CL21A226MAYNNNE?qs=sGAEpiMZZMsh%252B1woXyUXj9e2R%2FOkAO5o4FNiyGuFzx8%3D; specs 10uF, 50VDC, X5R, 10%, -55C, +85C -> 22uF, 25V, 20%, X5R, -55C, +85C, mlcc; unit x10 0.07 -> 0.043
- C109, C112: value 10u -> 220n; footprint Capacitor_SMD:C_1206_3216Metric_Pad1.33x1.80mm_HandSolder -> Capacitor_SMD:C_0805_2012Metric_Pad1.18x1.45mm_HandSolder; mouser https://www.mouser.com/ProductDetail/Samsung-Electro-Mechanics/CL31A106KBHNNNE?qs=sGAEpiMZZMsh%252B1woXyUXjxqcB7t9naYpzWmpMbMJIKQ%3D -> https://www.mouser.com/ProductDetail/Samsung-Electro-Mechanics/CL21B224KCFSFNE?qs=664zcAxDQ0l4Y1eUk6Zc1g%3D%3D; specs 10uF, 50VDC, X5R, 10%, -55C, +85C -> 100VDC, X7R, 10%, -55C, +125C, 220nF; unit x10 0.07 -> 0.054
Connections:
- net +3V3: now also C105.1, C111.1, C112.2; no longer C112.1
- net GND: now also C105.2, C112.1, C102.2; no longer C105.1, C112.2
- net at C103.1, C104.2, U103.7 (SEL)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: now also C102.1; no longer C105.2, C111.1

Commit message: jlc my bovine
bawk bawk
Parts:
- U101: mouser https://www.mouser.com/ProductDetail/Texas-Instruments/ISOM8110DFSR?qs=2FehpBK1j96965pfOjJBkA%3D%3D -> https://www.mouser.com/ProductDetail/Texas-Instruments/ISOM8110DFSRQ1?qs=2FehpBK1j95ipI81oj%252BjEg%3D%3D; unit x1 2 -> 2.01; unit x10 1.5 -> 1.44
Changed lines of the file:
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@@
 	(generator_version "9.0")
 	(paper "A4")
+	(title_block
+		(date "2026-03-14")
+		(rev "1")
+	)
 	(rectangle
 		(start 25.4 15.24)
@@
 			)
 		)
-		(property "mouser" "https://www.mouser.com/ProductDetail/Texas-Instruments/ISOM8110DFSR?qs=2FehpBK1j96965pfOjJBkA%3D%3D"
+		(property "mouser" "https://www.mouser.com/ProductDetail/Texas-Instruments/ISOM8110DFSRQ1?qs=2FehpBK1j95ipI81oj%252BjEg%3D%3D"
 			(at 136.144 72.136 0)
 			(effects
@@
 			)
 		)
-		(property "unit x10" "1.5"
+		(property "unit x10" "1.44"
 			(at 134.62 81.28 0)
 			(effects
@@
 			)
 		)
-		(property "unit x1" "2"
+		(property "unit x1" "2.01"
 			(at 134.62 81.28 0)
 			(effects
