File: hardware/mini Orion TEM before the clone/mini Orion TEM.kicad_pcb (KiCad board)
At the start: 2 copper layers, 319.7 x 58.4 mm, 112 parts, among them J101 HRLV, J102 VT bridge, J103 SWD, J104 Conn_01x02_Socket, SW101 SW_DIP_x06, U101 VT harness, U102 AP7384-50SA, U103 MCP2542FDxMF, U104 ISOW7741, U105 XMSM0G3507SDGS28R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

Commit message: made a few changes
Parts:
- added R151: 220, Resistor_SMD:R_1206_3216Metric, F.Cu at (172.7, 146.3)
- added U705: TLP155E, zzLocalLibraries-Footprints:U_SO6_11-4L1_TOS-M, F.Cu at (165.5, 146.4)
- moved TH308 3.20 mm to (290.7, 151.0)
- moved TH307 2.97 mm to (268.4, 151.2)
- moved F112 2.69 mm to (282.3, 121.5)
- moved TH305 2.13 mm to (245.7, 152.3)
- moved F108 1.75 mm to (192.5, 120.6)
- moved TH303 1.74 mm to (224.0, 152.4)
- moved TH202 1.71 mm to (245.8, 137.1)
- moved TH301 1.61 mm to (155.7, 152.4)
- moved F110 1.55 mm to (237.6, 120.4)
- moved TH205 1.45 mm to (156.9, 136.8)
- moved TH304 1.35 mm to (133.4, 152.5)
- moved F114 1.35 mm to (326.9, 120.2)
- moved TH201 1.26 mm to (290.5, 137.3)
- moved F106 1.19 mm to (147.9, 120.0)
- moved F104 0.63 mm to (103.2, 119.5)
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Connections:
- U105 pad 4: /UART_TX -> /TIMG8_C2
- U105 pad 5: /UART_RX -> unconnected-(U105-PA1-Pad5)
Routing:
- net /TIMG8_C2: track 0.00 -> 15.0 mm, vias 0 -> 2
- net Net-(R151-Pad1): track 0.00 -> 3.14 mm
- net Net-(C308-Pad1): track 4.91 -> 6.75 mm
- net Net-(C307-Pad1): track 8.30 -> 10.00 mm
- net Net-(C303-Pad1): track 4.44 -> 5.76 mm
- net Net-(F110-Pad2): track 6.20 -> 4.90 mm
- net Net-(F106-Pad2): track 6.10 -> 4.89 mm
- net Net-(F114-Pad2): track 5.98 -> 4.90 mm
- net Net-(C202-Pad1): track 6.08 -> 7.12 mm
- net /VT18: track 261.2 -> 260.2 mm
- net /VT25: track 171.9 -> 171.0 mm
- net Net-(F108-Pad2): track 6.15 -> 5.22 mm
- net Net-(F104-Pad2): track 6.05 -> 5.13 mm
- net Net-(C305-Pad1): track 6.17 -> 7.05 mm
- net Net-(F112-Pad2): track 6.25 -> 5.42 mm
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