File: hardware/mini Orion TEM before the clone/mini Orion TEM.kicad_sch (KiCad schematic)
At the start: 60 parts, among them J101 HRLV, J102 VT bridge, J103 SWD, J104 Conn_01x02_Socket, SW101 SW_DIP_x06, U101 VT harness, U102 AP7384-50SA, U103 MCP2542FDxMF, U104 ISOW7741, U105 XMSM0G3507SDGS28R

Commit message: made a few changes
Parts:
- added R151: 220, Resistor_SMD:R_1206_3216Metric, symbol Device:R_Small_US
- added U705: TLP155E, zzLocalLibraries-Footprints:U_SO6_11-4L1_TOS-M, symbol zzLocalLibrary:TLP155E
Connections:
- net GND: now also U705.3, U705.4 (-)
- net UART_RX: no longer names the net of U105.5 (PA1)
- net UART_TX renamed TIMG8_C2
- net TIMG8_C2: now also R151.2
- new net: R151.1, U705.1
- new net Fan control: U705.5
- no-connect marks 10 -> 9
Other:
- moved on the sheet: F102, F104, F106, J102, TP102, TP104, TP106, U101
