File: hardware/VoltageTap_Bee/UART_USB.kicad_sch (KiCad schematic)
At the start: 6 parts, among them J16 USB_B_Micro, U12 FT230XS, U3 STISO620

Commit message: baeckbjlnacnklac
Parts:
- renumbered C4 to C401, D5 to D401, J16 to J401, R10 to R401, U12 to U401, U3 to U402
Changed lines of the file:
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@@
 		(dnp no)
 		(fields_autoplaced yes)
-		(property "Reference" "J16"
+		(property "Reference" "J401"
 			(at 25.4 24.13 0)
 			(effects
@@
 			(project "VoltageTap_B"
 				(path "/24c6cb45-cbeb-4148-a23c-ec2e76234670/61266382-19ea-4f72-94ef-47ef11de2113"
-					(reference "J16")
+					(reference "J401")
 					(unit 1)
 				)
@@
 		(on_board yes)
 		(dnp no)
-		(property "Reference" "U3"
+		(property "Reference" "U402"
 			(at 119.38 40.64 0)
 			(effects
@@
 			(project "VoltageTap_B"
 				(path "/24c6cb45-cbeb-4148-a23c-ec2e76234670/61266382-19ea-4f72-94ef-47ef11de2113"
-					(reference "U3")
+					(reference "U402")
 					(unit 1)
 				)
@@
 		(on_board yes)
 		(dnp no)
-		(property "Reference" "D5"
+		(property "Reference" "D401"
 			(at 54.61 51.054 90)
 			(effects
@@
 			(project "VoltageTap_B"
 				(path "/24c6cb45-cbeb-4148-a23c-ec2e76234670/61266382-19ea-4f72-94ef-47ef11de2113"
-					(reference "D5")
+					(reference "D401")
 					(unit 1)
 				)
@@
 		(on_board yes)
 		(dnp no)
-		(property "Reference" "R10"
+		(property "Reference" "R401"
 			(at 52.832 43.18 0)
 			(effects
@@
 			(project "VoltageTap_B"
 				(path "/24c6cb45-cbeb-4148-a23c-ec2e76234670/61266382-19ea-4f72-94ef-47ef11de2113"
-					(reference "R10")
+					(reference "R401")
 					(unit 1)
 				)
@@
 		(on_board yes)
 		(dnp no)
-		(property "Reference" "C4"
+		(property "Reference" "C401"
 			(at 38.1 53.3462 0)
 			(effects
@@
 			(project "VoltageTap_B"
 				(path "/24c6cb45-cbeb-4148-a23c-ec2e76234670/61266382-19ea-4f72-94ef-47ef11de2113"
-					(reference "C4")
+					(reference "C401")
 					(unit 1)
 				)
@@
 		(dnp no)
 		(fields_autoplaced yes)
-		(property "Reference" "U12"
+		(property "Reference" "U401"
 			(at 82.1533 20.32 0)
 			(effects
@@
 			(project "VoltageTap_B"
 				(path "/24c6cb45-cbeb-4148-a23c-ec2e76234670/61266382-19ea-4f72-94ef-47ef11de2113"
-					(reference "U12")
+					(reference "U401")
 					(unit 1)
 				)
