File: hardware/VoltageTap_Bee/VoltageTap_B.kicad_sch (KiCad schematic)
At the start: 43 parts, among them J1 Conn_01x09_Socket, J102 Conn_01x18_Pin, J15 Conn_02x04_Odd_Even, J2 Conn_02x05_Odd_Even, Q6 2N7002, SW1 SW_Push, U2 MCU-MSM0G3507SPM

Commit message: aenllaec
Other:
- sheet (lib_symbols 	(symbol "Regulator_Linear:AP7384-50SA" 		(pin_names 			(offset 0.254) 		) 		(exclude_from_sim no) 		(in_bom yes) 		(on_board yes) 		(property "Reference" "U" 			(at -3.81 3.175 0) 			(effects 				(font (size 1.27 1.27)) 			) 		) 		(property "Value" "AP7384-50SA" 			(at 0 3.175 0) 			(effects 				(font (size 1.27 1.27)) 				(justify left) 			) 		) 		(property "Footprint" "Package_TO_SOT_SMD:SOT-23" 			(at 0 5.715 0) 			(effects 				(font (size 1.27 1.27) (italic yes)) 				(hide yes) 			) 		) 		(property "Datasheet" "https://www.diodes.com/assets/Datasheets/AP7384.pdf" 			(at 0 -1.27 0) 			(effects 				(font (size 1.27 1.27)) 				(hide yes) 			) 		) 		(property "Description" "50mA Low Dropout Voltage Regulator, Fixed Output 5V, Wide Input Voltage Range 40V, SOT-23" 			(at 0 0 0) 			(effects 				(font (size 1.27 1.27)) 				(hide yes) 			) 		) 		(property "ki_keywords" "50mA LDO Regulator Fixed Positive" 			(at 0 0 0) 			(effects 				(font (size 1.27 1.27)) 				(hide yes) 			) 		) 		(property "ki_fp_filters" "SOT?23*" 			(at 0 0 0) 			(effects 				(font (size 1.27 1.27)) 				(hide yes) 			) 		) 		(symbol "AP7384-50SA_0_1" 			(rectangle 				(start -5.08 1.905) 				(end 5.08 -5.08) 				(stroke (width 0.254) (type default)) 				(fill (type background)) 			) 		) 		(symbol "AP7384-50SA_1_1" 			(pin power_in line 				(at -7.62 0 0) 				(length 2.54) 				(name "VI" 					(effects 						(font (size 1.27 1.27)) 					) 				) 				(number "1" 					(effects 						(font (size 1.27 1.27)) 					) 				) 			) 			(pin power_in line 				(at 0 -7.62 90) 				(length 2.54) 				(name "GND" 					(effects 						(font (size 1.27 1.27)) 					) 				) 				(number "3" 					(effects 						(font (size 1.27 1.27)) 					) 				) 			) 			(pin power_out line 				(at 7.62 0 180) 				(length 2.54) 				(name "VO" 					(effects 						(font (size 1.27 1.27)) 					) 				) 				(number "2" 					(effects 						(font (size 1.27 1.27)) 					) 				) 			) 		) 		(embedded_fonts no) 	) ) (symbol 	(lib_id "Regulator_Linear:AP7384-50SA") 	(at 270.51 26.67 0) 	(unit 1) 	(exclude_from_sim no) 	(in_bom yes) 	(on_board yes) 	(dnp no) 	(fields_autoplaced yes) 	(uuid "63645a03-0dcf-4de9-9155-a6ccb0705d23") 	(property "Reference" "U26" 		(at 270.51 20.32 0) 		(effects 			(font (size 1.27 1.27)) 		) 	) 	(property "Value" "AP7384-50SA" 		(at 270.51 22.86 0) 		(effects 			(font (size 1.27 1.27)) 		) 	) 	(property "Footprint" "Package_TO_SOT_SMD:SOT-23" 		(at 270.51 20.955 0) 		(effects 			(font (size 1.27 1.27) (italic yes)) 			(hide yes) 		) 	) 	(property "Datasheet" "https://www.diodes.com/assets/Datasheets/AP7384.pdf" 		(at 270.51 27.94 0) 		(effects 			(font (size 1.27 1.27)) 			(hide yes) 		) 	) 	(property "Description" "50mA Low Dropout Voltage Regulator, Fixed Output 5V, Wide Input Voltage Range 40V, SOT-23" 		(at 270.51 26.67 0) 		(effects 			(font (size 1.27 1.27)) 			(hide yes) 		) 	) 	(property "mouser" "https://www.mouser.com/ProductDetail/Diodes-Incorporated/AP7375-50SA-7?qs=t7xnP681wgX8yYKy1Pe5iA%3D%3D" 		(at 270.51 26.67 0) 		(effects 			(font (size 1.27 1.27)) 			(hide yes) 		) 	) 	(property "unit x1" "0.25" 		(at 270.51 26.67 0) 		(effects 			(font (size 1.27 1.27)) 			(hide yes) 		) 	) 	(property "unit x10" "0.174" 		(at 270.51 26.67 0) 		(effects 			(font (size 1.27 1.27)) 			(hide yes) 		) 	) 	(property "unit x25" "0.154" 		(at 270.51 26.67 0) 		(effects 			(font (size 1.27 1.27)) 			(hide yes) 		) 	) 	(pin "3" 		(uuid "9ddd95e1-ca1e-416e-9dfe-24d7a0b4d0e6") 	) 	(pin "2" 		(uuid "ab10e457-2625-421f-8a82-9adf340550bb") 	) 	(pin "1" 		(uuid "b619a3b1-fac7-4971-8cb9-ac4027e9c86d") 	) 	(instances 		(project "VoltageTap_B" 			(path "" 				(reference "U26") 				(unit 1) 			) 			(path "/24c6cb45-cbeb-4148-a23c-ec2e76234670/443e7a8e-9df5-428f-9d56-3f2b4e9a9ffe/50286653-b14c-419a-bf32-2b9dde1a77b3" 				(reference "U46") 				(unit 1) 			) 		) 	) ) renamed moo
- sheet something renamed common
Changed lines of the file:
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@@
 	)
 	(sheet
-		(at 426.72 194.31)
+		(at 426.72 295.91)
 		(size 27.94 22.86)
 		(exclude_from_sim yes)
@@
 			(color 0 0 0 0.0000)
 		)
-		(property "Sheetname" "something"
-			(at 426.72 193.5984 0)
+		(property "Sheetname" "common"
+			(at 426.72 295.1984 0)
 			(effects
 				(font
@@
 		)
 		(property "Sheetfile" "../common designs.kicad_sch"
-			(at 426.72 217.7546 0)
+			(at 426.72 319.3546 0)
 			(effects
 				(font
@@
 		)
 		(property "Field2" ""
-			(at 426.72 194.31 0)
+			(at 426.72 295.91 0)
 			(effects
 				(font
@@
 			(project "VoltageTap_B"
 				(path "/24c6cb45-cbeb-4148-a23c-ec2e76234670"
-					(page "5")
+					(page "999")
 				)
 			)
@@
 			(color 0 0 0 0.0000)
 		)
+		(property "Sheetname" "moo"
+			(at 336.55 226.6184 0)
+			(effects
+				(font
+					(size 1.27 1.27)
+				)
+				(justify left bottom)
+				(hide yes)
+			)
+		)
 		(property "Sheetfile" "GLV CAN TRX.kicad_sch"

Commit message: nlaeclnaec
Parts:
- removed C12: 220n, Capacitor_SMD:C_1206_3216Metric_Pad1.33x1.80mm_HandSolder, symbol Device:C_Small
- removed Q6: 2N7002, Package_TO_SOT_SMD:SOT-23, symbol Transistor_FET:2N7002
- removed R13, R14, R17, R4: 150, Resistor_SMD:R_1206_3216Metric_Pad1.30x1.75mm_HandSolder, symbol Device:R_US
- added Q101: TSM2328CX, Package_TO_SOT_SMD:SOT-23-3, symbol Transistor_FET:Q_NMOS_GSD
- added R101, R102, R103, R104: 750, Resistor_SMD:R_1206_3216Metric_Pad1.30x1.75mm_HandSolder, symbol Device:R_US
- C11, C13, C5: value 220n -> 100n; footprint Capacitor_SMD:C_1206_3216Metric_Pad1.33x1.80mm_HandSolder -> Capacitor_SMD:C_0603_1608Metric_Pad1.08x0.95mm_HandSolder; mouser https://www.mouser.com/ProductDetail/Samsung-Electro-Mechan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 -> https://www.mouser.com/ProductDetail/Wurth-Elektronik/88501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; specs 50VDC, X7R, 10%, -55C, +125C, 220nF -> 100nF, 10%, 50V, X7R, -55C, +125C; unit x1 (none) -> 0.10; unit x10 0.054 -> 0.029; unit x100 (none) -> 0.017; unit x50 (none) -> 0.02
- R11, R2, R7: value 200k -> 88.7k; mouser https://www.mouser.com/ProductDetail/KOA-Speer/RK73H2ATTDD2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 -> https://www.mouser.com/ProductDetail/YAGEO/AC0805FR-0788K7L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; specs (none) -> 88.7kR, 125mW, 150V, 100ppm, 1%, -55C, +155C; specs  250mW, 200k, 1% -> (none); unit x1 0.02 -> 0.01; unit x10 0.1 -> 0.011
Connections:
- net BQ76952 1/CFETOFF: now also R102.2
- net BQ76952 1/HDQ: now also R101.2
- net BQ76952 1/SCL: now also R103.1
- net BQ76952 1/SDA: now also R104.1
- net PA16_SPI1_MISO: now also R104.2
- net PA17_SPI1_SCK: now also R103.2
- net PA18_SPI1_MOSI: now also R101.1
- net PB19_BBQ_CS: now also R102.1
- net onboard 3.3v src: now also Q101.3 (D)
- net at C17.2, R1.1, R11.2: now also Q101.1 (G)
- net at R2.2, R50.2: now also Q101.2 (S)

Commit message: baeckbjlnacnklac
Parts:
- removed J15: Conn_02x04_Odd_Even, Connector_PinHeader_2.54mm:PinHeader_2x04_P2.54mm_Vertical, symbol Connector_Generic:Conn_02x04_Odd_Even
- added U101: XMSM0G3507SDGS28R, zzLocalLibraries-Footprints:VSSOP28_DGS_TEX-M, symbol zzLocalLibrary:XMSM0G3507SDGS28R
- renumbered C17 to C101, C3 to C102, C13 to C103, C14 to C104, C11 to C105, C5 to C106, D1 to D101, D4 to D102, J2 to J101, J1 to J103, JP1 to JP101, R102 to R101, R103 to R102, R101 to R103, R6 to R105, R50 to R106, R2 to R107, R11 to R108, R1 to R109, R7 to R110, R3 to R111, R8 to R112, SW1 to SW101, TP14 to TP101, TP16 to TP102, TP9 to TP103, TP12 to TP104, TP5 to TP105, TP4 to TP106, U2 to U102
Connections:
- net RST_N: no longer J103.6 (Pin_6)
- net XDS_5v_supply: no longer names the net of J103.2 (Pin_2)

Commit message: schematic updates
Parts:
- removed J103: Conn_01x09_Socket, Connector_PinHeader_2.54mm:PinHeader_1x09_P2.54mm_Vertical, symbol Connector:Conn_01x09_Socket
- added C1, C3, C4: 100n, Capacitor_SMD:C_0603_1608Metric_Pad1.08x0.95mm_HandSolder, symbol Device:C_Small
- added C2: 10u, Capacitor_SMD:C_1206_3216Metric_Pad1.33x1.80mm_HandSolder, symbol Device:C_Small
- added J104: Conn_01x06_Pin, Connector_PinHeader_2.54mm:PinHeader_1x06_P2.54mm_Vertical, symbol Connector:Conn_01x06_Pin
- added R1: 100k, Resistor_SMD:R_1206_3216Metric_Pad1.30x1.75mm_HandSolder, symbol Device:R_US
Connections:
- net +3.3V: now also U101.7 (VDD), C3.1, C4.1
- net -BATT: now also U101.8 (VSS), C1.2, C2.2, C3.2, C4.2, J104.1 (Pin_1), R1.2
- net PA10_UART0-TX_XDS: now also U101.15 (PA10/CLK_OUT), J104.4 (Pin_4)
- net PA11_UART0-RX_XDS: now also U101.16 (PA11), J104.3 (Pin_3)
- net PA15_BBQ_RESET: now also U101.18 (PA15/A1_0)
- net PA16_SPI1_MISO: now also U101.19 (PA16/A1_1/FCC_IN)
- net PA17_SPI1_SCK: now also U101.20 (PA17/A1_2)
- net PA18_SPI1_MOSI: now also U101.21 (PA18/A1_3)
- net PA19_SWDIO: now also U101.22 (PA19/SWDIO), J104.5 (Pin_5)
- net PA20_SWCLK: now also U101.23 (PA20/SWCLK), J104.6 (Pin_6)
- net PA7: no longer R111.1
- net PB19_BBQ_CS: no longer R101.1
- net RST_N: now also U101.6 (NRST)
- net XDS_3v_supply: now also J104.2 (Pin_2)
- net at D102.2 (A): now also R111.1; no longer R111.2
- net PA26_CAN_TX: now reaches U101.1 (PA26/A0_1)
- net BLINK: now reaches U101.10 (PA3_/_LFXIN)
- net BLINK: now also R111.2
- net IL_EN: now reaches U101.11 (PA4_/_LFCLK_IN_/_LFXOUT)
- net PB14_BBQ_CS: now reaches U101.17 (PA14/CLK_OUT/A0_12)
- net PB14_BBQ_CS: now also R101.1
- net PA27_CAN_RX: now reaches U101.2 (PA27/RTC_OUT/A0_0)
- net at U101.3 (VCORE): now also C1.1, C2.1
- net at U101.9 (PA2_/_ROSC): now also R1.1
- no-connect marks 59 -> 58
Other:
- sheet moo renamed GLV
- removed sheet UART_USB
- note added: "TODO: CHANGE CAN TX, CAN RX, BLINK,IL ENABLE AND BBQ CS IN CODE"
- note removed: "user uart"
- moved on the sheet: D102, R111, U101
