File: hardware/CAN_Eth_Bridge/CAN_Eth_Bridge.kicad_sch (KiCad schematic)
At the start: 31 parts, among them J101 Global LV and CAN, J102 Conn_01x05_Pin, Q101 TSM2328CX, Q102 TSM2328CX, SW102 SW_Push, U101 AP7384-50SA, U103 MCP2542FDxMF, U104 XMSM0G3507SDGS28R, U105 LM74502, U106 BD33FC0FP

Commit message: calknaeclkac
lkaececa
Connections:
- net GLV+: now also J101.2 (Pin_2); no longer J101.5 (Pin_5)
- net GND: now also J101.5 (Pin_5); no longer J101.2 (Pin_2)
- net G_CAN+: now also J101.3 (Pin_3); no longer J101.6 (Pin_6)
- net G_CAN-: now also J101.6 (Pin_6); no longer J101.3 (Pin_3)
Changed lines of the file:
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@@
 	(symbol
 		(lib_id "Connector_Generic:Conn_02x03_Top_Bottom")
-		(at 31.75 29.21 0)
+		(at 34.29 29.21 0)
+		(mirror y)
 		(unit 1)
 		(exclude_from_sim no)
@@
 		)
 		(property "Footprint" "Connector_Molex:Molex_Micro-Fit_3.0_43045-0600_2x03_P3.00mm_Horizontal"
-			(at 31.75 29.21 0)
+			(at 34.29 29.21 0)
 			(effects
 				(font
@@
 		)
 		(property "Datasheet" "~"
-			(at 31.75 29.21 0)
+			(at 34.29 29.21 0)
 			(effects
 				(font
@@
 		)
 		(property "Description" "Generic connector, double row, 02x03, top/bottom pin numbering scheme (row 1: 1...pins_per_row, row2: pins_per_row+1 ... num_pins), script generated (kicad-library-utils/schlib/autogen/connector/)"
-			(at 31.75 29.21 0)
+			(at 34.29 29.21 0)
 			(effects
 				(font
@@
 		)
 		(property "mouser" "https://www.mouser.com/ProductDetail/Molex/43045-0600?qs=mrPiglD9aYJ8CzJ%2FE2PNbw%3D%3D&srsltid=AfmBOop7-nikRF2atEfFslZtuPWfqFOihNLqcdVlYseRCGCFOiFBx6Nk"
-			(at 31.75 29.21 0)
+			(at 34.29 29.21 0)
 			(effects
 				(font
@@
 		)
 		(property "unit x10" "1.19"
-			(at 31.75 29.21 0)
+			(at 34.29 29.21 0)
 			(effects
 				(font
@@
 		)
 		(property "unit x1" "1.46"
-			(at 31.75 29.21 0)
+			(at 34.29 29.21 0)
 			(effects
 				(font
@@
 		)
 		(property "Sim.Pins" ""
-			(at 31.75 29.21 0)
+			(at 34.29 29.21 0)
 			(effects
 				(font
@@
 		)
 		(property "note" ""
-			(at 31.75 29.21 0)
+			(at 34.29 29.21 0)
 			(effects
 				(font
