File: hardware/CANE Junction/CANE Junction.kicad_pcb (KiCad board)
At the start: 2 copper layers, 22.6 x 60.7 mm, 78 parts, among them J1 Global LV and CAN, J101 Global LV and CAN, J102 Conn_01x05_Pin, J104 Conn_02x05_Odd_Even, J2 glv interface, J301 RJ45_Amphenol_RJMG1BD3B8K1ANR, Q301 MMBT5550L, Q302 MMBT5550L, SW101 SW_Push, U1 ISO1044BD, U101 TPSM33606S5QRDNRQ1, U102 TPS26625DRCR, U103 MCP2542FDxMF, U104 XMSM0G3507SDGS28R, U106 NCP163ASN330T1G, U2 ISOM8110DFS, U3 TPS7B4254, U301 W5500, U509 ISO1044BD, Y301 Crystal_GND24

Commit message: shuffle master 2000
nearing terminal shuffle . main components in, awaiting general and layout tie ins
Parts:
- removed C1, C106, C110, C2, C3, C4, C5: 220n, Capacitor_SMD:C_0805_2012Metric_Pad1.18x1.45mm_HandSolder
- removed C101: 1u, Capacitor_SMD:C_0603_1608Metric_Pad1.08x0.95mm_HandSolder
- removed C102: 10n, Capacitor_SMD:C_0805_2012Metric_Pad1.18x1.45mm_HandSolder
- removed C309: 22u, Capacitor_SMD:C_0805_2012Metric_Pad1.18x1.45mm_HandSolder
- removed CR1, CR501: ESD2CAN36DBZRQ1, Package_TO_SOT_SMD:TSOT-23_HandSoldering
- removed D105: blue, LED_SMD:LED_0805_2012Metric_Pad1.15x1.40mm_HandSolder
- removed FL1, FL101: Choke_CommonMode_FerriteCore_1243, zzLocalLibraries-Footprints:L_CommonModeChoke_Coilcraft_1812CAN
- removed G***: LOGO, zzLocal Library:UTARacingSilkscreen
- removed G***: LOGO, LOGO
- removed J102: Conn_01x05_Pin, Connector_PinHeader_2.54mm:PinHeader_1x05_P2.54mm_Vertical
- removed J104: Conn_02x05_Odd_Even, Connector_PinHeader_1.27mm:PinHeader_2x05_P1.27mm_Vertical_SMD
- removed Q301, Q302: MMBT5550L, Package_TO_SOT_SMD:SOT-23
- removed R101: 22.1k, Resistor_SMD:R_0805_2012Metric_Pad1.20x1.40mm_HandSolder
- removed R102, R311, R312: 2.4k, Resistor_SMD:R_0805_2012Metric_Pad1.20x1.40mm_HandSolder
- removed R105, R111: 100k, Resistor_SMD:R_1206_3216Metric_Pad1.30x1.75mm_HandSolder
- removed R106: 40.2k, Resistor_SMD:R_0805_2012Metric_Pad1.20x1.40mm_HandSolder
- removed R107: 1M, Resistor_SMD:R_0805_2012Metric_Pad1.20x1.40mm_HandSolder
- removed R108: 33.2k, Resistor_SMD:R_0805_2012Metric_Pad1.20x1.40mm_HandSolder
- removed R110: 10k, Resistor_SMD:R_0805_2012Metric_Pad1.20x1.40mm_HandSolder
- removed U101: TPSM33606S5QRDNRQ1, zzLocalLibraries-Footprints:RDN0011A_TEX
- removed U103: MCP2542FDxMF, Package_SO:SOIC-8_3.9x4.9mm_P1.27mm
- removed U104: XMSM0G3507SDGS28R, zzLocalLibraries-Footprints:VSSOP28_DGS_TEX-M
- removed U106: NCP163ASN330T1G, Package_TO_SOT_SMD:SOT-23-5_HandSoldering
- removed U509: ISO1044BD, Package_SO:SOIC-8_5.3x5.3mm_P1.27mm
- added BZ1: Buzzer, Buzzer_Beeper:MagneticBuzzer_ProSignal_ABI-009-RC, F.Cu at (107.1, 125.2)
- added C107: 220n, Capacitor_SMD:C_0805_2012Metric_Pad1.18x1.45mm_HandSolder, F.Cu at (80.4, 92.2)
- added C201: 220n, Capacitor_SMD:C_0805_2012Metric_Pad1.18x1.45mm_HandSolder, F.Cu at (59.4, 54.4)
- added C202: 220n, Capacitor_SMD:C_0805_2012Metric_Pad1.18x1.45mm_HandSolder, F.Cu at (59.4, 57.4)
- added C203: 220n, Capacitor_SMD:C_0805_2012Metric_Pad1.18x1.45mm_HandSolder, F.Cu at (59.4, 60.4)
- added C204: 22u, Capacitor_SMD:C_0805_2012Metric_Pad1.18x1.45mm_HandSolder, F.Cu at (59.4, 63.4)
- added C205: 22u, Capacitor_SMD:C_0805_2012Metric_Pad1.18x1.45mm_HandSolder, F.Cu at (59.4, 66.4)
- added C401: 220n, Capacitor_SMD:C_0805_2012Metric_Pad1.18x1.45mm_HandSolder, F.Cu at (66.3, 139.6)
- added C402: 220n, Capacitor_SMD:C_0805_2012Metric_Pad1.18x1.45mm_HandSolder, F.Cu at (69.3, 139.6)
- added C403: 220n, Capacitor_SMD:C_0805_2012Metric_Pad1.18x1.45mm_HandSolder, F.Cu at (72.3, 139.6)
- added C404: 22u, Capacitor_SMD:C_0805_2012Metric_Pad1.18x1.45mm_HandSolder, F.Cu at (75.3, 139.6)
- added C405: 22u, Capacitor_SMD:C_0805_2012Metric_Pad1.18x1.45mm_HandSolder, F.Cu at (78.3, 139.6)
- added CR201: ESD2CAN36DBZRQ1, Package_TO_SOT_SMD:TSOT-23_HandSoldering, F.Cu at (78.1, 43.4)
- added CR401: ESD2CAN36DBZRQ1, Package_TO_SOT_SMD:TSOT-23_HandSoldering, F.Cu at (55.3, 120.8)
- added D1: SD0805S020S1R0, Diode_SMD:D_0805_2012Metric_Pad1.15x1.40mm_HandSolder, F.Cu at (75.6, 83.2)
- added D101: green, LED_SMD:LED_0805_2012Metric_Pad1.15x1.40mm_HandSolder, F.Cu at (75.6, 89.3)
- added D2: SD0805S020S1R0, Diode_SMD:D_0805_2012Metric_Pad1.15x1.40mm_HandSolder, F.Cu at (75.6, 86.2)
- added D201: TS4148, Diode_SMD:D_0805_2012Metric_Pad1.15x1.40mm_HandSolder, F.Cu at (64.2, 67.1)
- added D401: TS4148, Diode_SMD:D_0805_2012Metric_Pad1.15x1.40mm_HandSolder, F.Cu at (79.0, 134.8)
- added FL201: Choke_CommonMode_FerriteCore_1243, zzLocalLibraries-Footprints:L_CommonModeChoke_Coilcraft_1812CAN, F.Cu at (77.2, 49.0)
- added FL401: Choke_CommonMode_FerriteCore_1243, zzLocalLibraries-Footprints:L_CommonModeChoke_Coilcraft_1812CAN, F.Cu at (60.9, 121.8)
- added IC1: PAM8904QJER, zzLocalLibraries-Footprints:QFN50P300X300X65-17N-D, F.Cu at (102.2, 119.7)
- added R2: 40.2k, Resistor_SMD:R_0805_2012Metric_Pad1.20x1.40mm_HandSolder, F.Cu at (85.2, 83.2)
- added R205: 121, Resistor_SMD:R_0805_2012Metric_Pad1.20x1.40mm_HandSolder, F.Cu at (81.9, 47.1)
- added R3: 100k, Resistor_SMD:R_0805_2012Metric_Pad1.20x1.40mm_HandSolder, F.Cu at (85.2, 86.1)
- added R405: 121, Resistor_SMD:R_0805_2012Metric_Pad1.20x1.40mm_HandSolder, F.Cu at (59.0, 117.0)
- added R406: 750, Resistor_SMD:R_0805_2012Metric_Pad1.20x1.40mm_HandSolder, F.Cu at (81.9, 50.0)
- added R407: 750, Resistor_SMD:R_0805_2012Metric_Pad1.20x1.40mm_HandSolder, F.Cu at (61.9, 117.0)
- added RN1: 56K, zzLocalLibraries-Footprints:R_array_YCJ164_4, F.Cu at (81.0, 62.6)
- added RN2: 56K, zzLocalLibraries-Footprints:R_array_YCJ164_4, F.Cu at (74.5, 118.0)
- added U201: TL432DBZ, Package_TO_SOT_SMD:SOT-23-3, F.Cu at (82.5, 66.8)
- added U202: TPS7B4254, Package_SO:Texas_R-PDSO-G8_EP2.95x4.9mm_Mask2.4x3.1mm, F.Cu at (76.5, 56.2)
- added U203: ISO1044BD, Package_SO:SOIC-8_5.3x5.3mm_P1.27mm, F.Cu at (66.9, 62.2)
- added U204: ISOM8600, zzLocalLibraries-Footprints:SOIC4_DFG_TEX-M, F.Cu at (67.0, 55.8)
- added U205: PUCC33420QRAQRQ1, zzLocalLibraries-Footprints:VSON-FCRLF12_RAQ_TEX, F.Cu at (76.4, 62.3)
- added U401: TL432DBZ, Package_TO_SOT_SMD:SOT-23-3, F.Cu at (78.8, 116.4)
- added U402: TPS7B4254, Package_SO:Texas_R-PDSO-G8_EP2.95x4.9mm_Mask2.4x3.1mm, F.Cu at (68.2, 122.4)
- added U403: ISO1044BD, Package_SO:SOIC-8_5.3x5.3mm_P1.27mm, F.Cu at (74.1, 132.0)
- added U404: ISOM8600, zzLocalLibraries-Footprints:SOIC4_DFG_TEX-M, F.Cu at (67.7, 131.9)
- added U405: PUCC33420QRAQRQ1, zzLocalLibraries-Footprints:VSON-FCRLF12_RAQ_TEX, F.Cu at (74.2, 122.5)
- C103, C105: value 22u -> 220n
- D102: value green -> blue
- J1: value Global LV and CAN -> glv; footprint zzLocalLibraries-Footprints:Molex_Micro-Fit_3.0_43045-0600_2x03_P3.00mm_Horizontal -> Connector_Molex:Molex_Micro-Fit_3.0_43650-0400_1x04_P3.00mm_Horizontal
- J101: value Global LV and CAN -> Conn_02x05_Odd_Even; footprint zzLocalLibraries-Footprints:Molex_Micro-Fit_3.0_43045-0600_2x03_P3.00mm_Horizontal -> Connector_PinHeader_1.27mm:PinHeader_2x05_P1.27mm_Vertical_SMD
- J2: value glv interface -> glv; footprint zzLocalLibraries-Footprints:Molex_Micro-Fit_3.0_43045-0600_2x03_P3.00mm_Horizontal -> Connector_Molex:Molex_Micro-Fit_3.0_43650-0400_1x04_P3.00mm_Horizontal
- R104, R315: moved to F.Cu
- R316, R317: footprint Resistor_SMD:R_1206_3216Metric_Pad1.30x1.75mm_HandSolder -> Resistor_SMD:R_0805_2012Metric_Pad1.20x1.40mm_HandSolder; moved to F.Cu
- U1: value ISO1044BD -> MX25L3233FM2; footprint Package_SO:SOIC-8_5.3x5.3mm_P1.27mm -> Package_SO:SOIC-8_3.9x4.9mm_P1.27mm
- U102: value TPS26625DRCR -> NCP114ASN180T2G; footprint zzLocalLibraries-Footprints:DRC0010J_NV -> Package_TO_SOT_SMD:SOT-23-5_HandSoldering; moved to F.Cu
- U2: value ISOM8110DFS -> XMSPM0G3519SPMR; footprint zzLocalLibraries-Footprints:ISOM811_SOIC-4_DFG -> zzLocalLibraries-Footprints:LQFP64_PM_TEX-M
- U3: value TPS7B4254 -> TMP110D; footprint Package_SO:Texas_R-PDSO-G8_EP2.95x4.9mm_Mask2.4x3.1mm -> Package_SON:Texas_X2SON-5_0.8x0.8mm_P0.48mm_RoutingVia
- moved J2 131.8 mm to (62.8, 137.6), turned to 90 degrees
- moved C104 107.3 mm to (80.4, 86.2)
- moved SW101 100.5 mm to (77.4, 103.0)
- moved U3 99.7 mm to (88.4, 108.2)
- moved U1 96.4 mm to (87.1, 97.2)
- moved U2 85.8 mm to (65.5, 89.4)
- moved R103 74.8 mm to (85.2, 89.0), turned to 0 degrees
- moved C105 74.0 mm to (80.4, 89.2), turned to 0 degrees
- moved J101 71.5 mm to (78.0, 98.0), turned to 0 degrees
- moved R104 68.6 mm to (85.2, 92.0), turned to 0 degrees
- moved J1 66.8 mm to (61.3, 50.9)
- moved D102 66.6 mm to (75.6, 92.3)
- moved R302 65.6 mm to (115.1, 47.3), turned to 0 degrees
- moved R301 65.2 mm to (115.1, 44.3)
- moved Y301 60.3 mm to (106.8, 57.5), turned to 0 degrees
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Connections:
- C103 pad 1: +5V -> Net-(U2-VCORE)
- C104 pad 1: +3.3V -> Net-(U2-VCORE)
- C105 pad 1: +3.3V -> Net-(D1-K)
- D102 pad 1: GND -> Net-(D102-K)
- D102 pad 2: Net-(D102-A) -> /led.sched
- J1 pad 1: /G_IL+ -> /CAN interface 1/IL-
- J1 pad 2: GND -> /CAN interface 1/IL+
- J1 pad 3: /G_CAN- -> /CAN interface 1/CAN+
- J1 pad 4: /G_IL+ -> /CAN interface 1/CAN-
- J101 pad 1: /G_IL+ -> +3.3V
- J101 pad 2: GND -> /prog.SWDIO
- J101 pad 3: /G_CAN- -> GND
- J101 pad 4: /G_IL+ -> /prog.SWCLK
- J101 pad 5: /GLV+ -> GND
- J101 pad 6: /G_CAN+ -> unconnected-(J101-Pin_6-Pad6)
- J2 pad 1: /CAN interface 1/IL+ -> /CAN interface 2/IL-
- J2 pad 2: /CAN interface 1/GLV- -> /CAN interface 2/IL+
- J2 pad 3: /CAN interface 1/CAN- -> /CAN interface 2/CAN+
- J2 pad 4: /CAN interface 1/IL+ -> /CAN interface 2/CAN-
- J301 pad L1: +5V -> +3.3V
- J301 pad L4: +5V -> +3.3V
- R103 pad 1: Net-(D105-K) -> Net-(D102-K)
- R104 pad 2: +3.3V -> /led.i1
- R316 pad 1: Net-(Q301-C) -> Net-(U301-LINKLED)
- R317 pad 1: Net-(Q302-C) -> Net-(U301-ACTLED)
- SW101 pad 1: GND -> Net-(U2-NRST)
- SW101 pad 2: /MCU_RESET -> GND
- U1 pad 1: /CAN interface 1/Vcc -> unconnected-(U1-~{CS}-Pad1)
- U1 pad 2: /CAN interface 1/TX -> unconnected-(U1-SO/SIO1-Pad2)
- U1 pad 3: /CAN interface 1/RX -> unconnected-(U1-~{WP}/SIO2-Pad3)
- U1 pad 4: /CAN interface 1/GND -> unconnected-(U1-GND-Pad4)
- U1 pad 5: Net-(U1-CANL) -> unconnected-(U1-SI/SIO0-Pad5)
- U1 pad 6: Net-(U1-CANH) -> unconnected-(U1-SCLK-Pad6)
- U1 pad 7: /CAN interface 1/GLV- -> unconnected-(U1-~{HOLD}/SIO3-Pad7)
- U102 pad 1: /GLV+ -> Net-(D1-K)
- U102 pad 2: Net-(U102-UVLO) -> GND
- U102 pad 3: Net-(U102-OVP) -> Net-(D1-K)
- U102 pad 5: GND -> +3.3V
- U2 pad 4: unconnected-(U2-C-Pad4) -> /can0.term
- U3 pad 3: /CAN interface 1/GLV- -> unconnected-(U3-ADD0-Pad3)
- U301 pad 38: unconnected-(U301-RSVD-Pad38) -> GND
- U301 pad 39: unconnected-(U301-RSVD-Pad39) -> GND
- U301 pad 40: unconnected-(U301-RSVD-Pad40) -> GND
- U301 pad 41: unconnected-(U301-RSVD-Pad41) -> GND
- U301 pad 42: unconnected-(U301-RSVD-Pad42) -> GND
Routing:
- net +5V: track 96.4 -> 0.00 mm, vias 1 -> 0
- net /Ethernet/+3.3VA: track 78.8 -> 0.00 mm, vias 3 -> 0
- net +3.3V: track 51.1 -> 0.00 mm, vias 2 -> 0
- net Net-(Q301-B): track 42.4 -> 0.00 mm, vias 1 -> 0
- net GND: track 41.6 -> 0.00 mm, vias 49 -> 0
- net Net-(Q302-B): track 39.9 -> 0.00 mm, vias 1 -> 0
- net /Ethernet/RD+: track 19.7 -> 0.00 mm
- net /Ethernet/RD-: track 19.6 -> 0.00 mm
- net /Ethernet/TD+: track 18.3 -> 0.00 mm, vias 2 -> 0
- net /GLV+: track 17.0 -> 0.00 mm, vias 1 -> 0
- net /Ethernet/TD-: track 16.7 -> 0.00 mm, vias 3 -> 0
- net /LV+: track 16.3 -> 0.00 mm, vias 1 -> 0
- net /led.sched: track 15.9 -> 0.00 mm
- net /G_CAN+: track 15.6 -> 0.00 mm, vias 2 -> 0
- net Net-(D102-A): track 15.0 -> 0.00 mm, vias 1 -> 0
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- removed copper zone on B.Cu, net GND
- removed copper zone on F.Cu, net GND
Other:
- board outline removed
- board text removed: "+ -"
- board text removed: "1.2"
- board text removed: "3/9/2026"
- board text removed: "A B"
- board text removed: "CAN"
- board text removed: "CAN-Eth bridge github.com/Gregification/BeeMS/"
- board text removed: "GLV"
- board text removed: "GND"
- board text removed: "IL"
- board text removed: "RX"
- board text removed: "SWCLK"
- board text removed: "SWDIO"
- board text removed: "TX"
- board text removed: "XDS110 debugger for scale"
- board text removed: "good luck unsoldering"
- board text removed: "tty 115200 8N1"
- board text removed: "±60Vmax, (17,31)V working"

Commit message: CANE put together and seemingly not exploding
meow meow meow
Parts:
- removed D101: green, LED_SMD:LED_0805_2012Metric_Pad1.15x1.40mm_HandSolder
- removed J101: Conn_02x05_Odd_Even, Connector_PinHeader_1.27mm:PinHeader_2x05_P1.27mm_Vertical_SMD
- removed R104: 2.4k, Resistor_SMD:R_0805_2012Metric_Pad1.20x1.40mm_HandSolder
- removed U3: TMP110D, Package_SON:Texas_X2SON-5_0.8x0.8mm_P0.48mm_RoutingVia
- added C108: 220n, Capacitor_SMD:C_0805_2012Metric_Pad1.18x1.45mm_HandSolder, F.Cu at (129.7, 75.2)
- added C109: 220n, Capacitor_SMD:C_0805_2012Metric_Pad1.18x1.45mm_HandSolder, F.Cu at (138.1, 108.4)
- added C315: 220n, Capacitor_SMD:C_0805_2012Metric_Pad1.18x1.45mm_HandSolder, F.Cu at (131.4, 54.1)
- added C825: 100n, Capacitor_SMD:C_0805_2012Metric_Pad1.18x1.45mm_HandSolder, B.Cu at (128.2, 83.0)
- added C826: 100n, Capacitor_SMD:C_0805_2012Metric_Pad1.18x1.45mm_HandSolder, B.Cu at (128.2, 86.9)
- added C827: 100n, Capacitor_SMD:C_0805_2012Metric_Pad1.18x1.45mm_HandSolder, B.Cu at (133.1, 87.8)
- added G***: LOGO, LOGO, B.Cu at (146.2, 97.0)
- added G***: LOGO, zzLocal Library:UTARacingSilkscreen, B.Cu at (141.8, 57.0)
- added H1: MountingHole, MountingHole:MountingHole_4.3mm_M4_ISO7380, F.Cu at (105.0, 55.0)
- added H2: MountingHole, MountingHole:MountingHole_4.3mm_M4_ISO7380, F.Cu at (155.0, 105.0)
- added H3: MountingHole, MountingHole:MountingHole_4.3mm_M4_ISO7380, F.Cu at (105.0, 105.0)
- added H4: MountingHole, MountingHole:MountingHole_4.3mm_M4_ISO7380, F.Cu at (155.0, 55.0)
- added J3: programming, Connector_PinHeader_2.54mm:PinHeader_1x03_P2.54mm_Vertical, F.Cu at (125.8, 97.2)
- added J4: UART, Connector_PinHeader_2.54mm:PinHeader_1x03_P2.54mm_Vertical, F.Cu at (138.8, 90.2)
- added R5: 40.2k, Resistor_SMD:R_0805_2012Metric_Pad1.20x1.40mm_HandSolder, B.Cu at (107.2, 71.1)
- added R7: 40.2k, Resistor_SMD:R_0805_2012Metric_Pad1.20x1.40mm_HandSolder, B.Cu at (104.7, 88.1)
- C103, C104, C311, C318, C319, IC1, R3, R310, R314, RN2, U401: moved to B.Cu
- J1, J2: footprint Connector_Molex:Molex_Micro-Fit_3.0_43650-0400_1x04_P3.00mm_Horizontal -> Connector_Molex:Molex_Micro-Fit_3.0_43045-0400_2x02_P3.00mm_Horizontal
- moved D102 82.5 mm to (157.8, 99.7), turned to 157.5 degrees
- moved SW101 79.0 mm to (155.9, 94.3), turned to 90 degrees
- moved U2 70.6 mm to (135.4, 99.3)
- moved R407 68.9 mm to (130.2, 107.6), turned to 0 degrees
- moved C405 67.5 mm to (111.9, 81.0), turned to -90 degrees
- moved C401 66.3 mm to (116.4, 96.2), turned to 180 degrees
- moved C107 64.9 mm to (144.8, 100.6), turned to 90 degrees
- moved R2 64.2 mm to (147.0, 100.6), turned to -90 degrees
- moved R103 62.5 mm to (145.8, 104.5)
- moved C103 62.3 mm to (139.1, 104.2), turned to 90 degrees
- moved J2 61.3 mm to (108.0, 96.2)
- moved C402 61.3 mm to (113.5, 97.1), turned to -90 degrees
- moved U1 60.6 mm to (147.7, 95.8), turned to 180 degrees
- moved C403 60.4 mm to (116.4, 98.3), turned to 180 degrees
- moved CR401 59.9 mm to (113.2, 105.6), turned to 180 degrees
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Connections:
- BZ1 pad 1: unconnected-(BZ1-+-Pad1) -> Net-(BZ1-+)
- BZ1 pad 2: unconnected-(BZ1---Pad2) -> Net-(BZ1--)
- C203 pad 1: /CAN interface 1/5v -> /CAN interface 1/GLV_5v
- C204 pad 1: /CAN interface 1/5v -> /CAN interface 1/GLV_5v
- C403 pad 1: /CAN interface 2/5v -> /CAN interface 2/GLV_5v
- C404 pad 1: /CAN interface 2/5v -> /CAN interface 2/GLV_5v
- CR201 pad 1: Net-(U203-CANH) -> Net-(U203-CANL)
- CR201 pad 2: Net-(U203-CANL) -> Net-(U203-CANH)
- D102 pad 1: Net-(D102-K) -> GND
- D102 pad 2: /led.sched -> Net-(D102-A)
- FL201 pad 1: /CAN interface 1/CAN+ -> /CAN interface 1/CAN-
- FL201 pad 2: Net-(U203-CANH) -> Net-(U203-CANL)
- FL201 pad 3: Net-(U203-CANL) -> Net-(U203-CANH)
- FL201 pad 4: /CAN interface 1/CAN- -> /CAN interface 1/CAN+
- IC1 pad 1: unconnected-(IC1-CPM1-Pad1) -> /buzzer.pm1
- IC1 pad 10: unconnected-(IC1-CN2-Pad10) -> Net-(IC1-CN2)
- IC1 pad 11: unconnected-(IC1-CP1-Pad11) -> Net-(IC1-CP1)
- IC1 pad 13: unconnected-(IC1-VOUT-Pad13) -> Net-(IC1-VOUT)
- IC1 pad 14: unconnected-(IC1-CP2-Pad14) -> Net-(IC1-CP2)
- IC1 pad 15: unconnected-(IC1-VIN-Pad15) -> +3.3V
- IC1 pad 2: unconnected-(IC1-CPM2-Pad2) -> /buzzer.pm2
- IC1 pad 3: unconnected-(IC1-DIN-Pad3) -> /buzzer.pwm
- IC1 pad 5: unconnected-(IC1-CN1-Pad5) -> Net-(IC1-CN1)
- IC1 pad 6: unconnected-(IC1-GND-Pad6) -> GND
- IC1 pad 7: unconnected-(IC1-VO2-Pad7) -> Net-(BZ1--)
- IC1 pad 9: unconnected-(IC1-VO1-Pad9) -> Net-(BZ1-+)
- J1 pad 1: /CAN interface 1/IL- -> /CAN interface 1/LV-
- J1 pad 2: /CAN interface 1/IL+ -> /CAN interface 1/LV+
- J2 pad 1: /CAN interface 2/IL- -> /CAN interface 2/LV-
- J2 pad 2: /CAN interface 2/IL+ -> /CAN interface 2/LV+
- R103 pad 1: Net-(D102-K) -> Net-(U2-PA0)
- R103 pad 2: GND -> Net-(D102-A)
- R405 pad 1: /CAN interface 2/CAN+ -> /CAN interface 2/CAN-
- RN1 pad 1: /CAN interface 1/LV- -> /CAN interface 1/5v_ldo_ref
- RN1 pad 3: Net-(RN1A-R1.2) -> /CAN interface 1/LV-
- RN1 pad 4: /CAN interface 1/5v_ldo_ref -> Net-(RN1A-R1.2)
- RN1 pad 5: Net-(D201-A) -> unconnected-(RN1C-R3.1-Pad5)
- RN1 pad 6: /CAN interface 1/LV+ -> unconnected-(RN1C-R3.2-Pad6)
- RN1 pad 7: Net-(RN1D-R4.1) -> Net-(D201-A)
- RN1 pad 8: /CAN interface 1/5v -> /CAN interface 1/LV+
- RN2 pad 1: /CAN interface 2/LV- -> /CAN interface 2/5v_ldo_ref
- RN2 pad 3: Net-(RN2A-R1.2) -> /CAN interface 2/LV-
- RN2 pad 4: /CAN interface 2/5v_ldo_ref -> Net-(RN2A-R1.2)
- RN2 pad 5: Net-(D401-A) -> unconnected-(RN2C-R3.1-Pad5)
- RN2 pad 6: /CAN interface 2/LV+ -> unconnected-(RN2C-R3.2-Pad6)
- RN2 pad 7: Net-(RN2D-R4.1) -> Net-(D401-A)
- RN2 pad 8: /CAN interface 2/5v -> /CAN interface 2/LV+
- U1 pad 1: unconnected-(U1-~{CS}-Pad1) -> /SECD.cs_fr
- U1 pad 2: unconnected-(U1-SO/SIO1-Pad2) -> /SECD.MISO/POCI
- U1 pad 3: unconnected-(U1-~{WP}/SIO2-Pad3) -> +3.3V
- U1 pad 4: unconnected-(U1-GND-Pad4) -> GND
- U1 pad 5: unconnected-(U1-SI/SIO0-Pad5) -> /SECD.MOSI/PICO
- U1 pad 6: unconnected-(U1-SCLK-Pad6) -> /SECD.SCLK
- U1 pad 7: unconnected-(U1-~{HOLD}/SIO3-Pad7) -> +3.3V
- U1 pad 8: unconnected-(U1-VCC-Pad8) -> +3.3V
- U2 pad 33: unconnected-(U2-PA0-Pad33) -> Net-(U2-PA0)
- U2 pad 4: /can0.term -> unconnected-(U2-PB16-Pad4)
- U2 pad 44: unconnected-(U2-PA4-Pad44) -> /SECD.MISO/POCI
- U2 pad 45: unconnected-(U2-PA5-Pad45) -> /SECD.MOSI/PICO
- U2 pad 46: unconnected-(U2-PA6-Pad46) -> /SECD.SCLK
- U2 pad 48: unconnected-(U2-PB1-Pad48) -> /SECD.cs_fr
- U2 pad 54: unconnected-(U2-PA8-Pad54) -> /uart1.TX
- U2 pad 55: unconnected-(U2-PA9-Pad55) -> /uart1.RX
- U2 pad 58: unconnected-(U2-PB6-Pad58) -> /eth.reset_N
- U2 pad 59: unconnected-(U2-PB7-Pad59) -> /eth.MISO/POCI
- U2 pad 60: unconnected-(U2-PB8-Pad60) -> /eth.MOSI/PICO
- U2 pad 61: unconnected-(U2-PB9-Pad61) -> /eth.SCLK
- U2 pad 62: unconnected-(U2-PB10-Pad62) -> /eth.cs_N
- U2 pad 63: unconnected-(U2-PB11-Pad63) -> GND
- U2 pad 64: unconnected-(U2-PB12-Pad64) -> /buzzer.pwm
- U2 pad 7: unconnected-(U2-PA14-Pad7) -> /can0.term
- U2 pad 8: unconnected-(U2-PA15-Pad8) -> /buzzer.pm1
- U2 pad 9: unconnected-(U2-PA16-Pad9) -> /buzzer.pm2
- U202 pad 1: /CAN interface 1/5v -> /CAN interface 1/GLV_5v
- U202 pad 4: /CAN interface 1/5v -> /CAN interface 1/GLV_5v
- U203 pad 8: /CAN interface 1/5v -> /CAN interface 1/GLV_5v
- U205 pad 1: Net-(RN1D-R4.1) -> Net-(U205-EN/FLT)
- U205 pad 2: /CAN interface 1/5v -> /CAN interface 1/GLV_5v
- U402 pad 1: /CAN interface 2/5v -> /CAN interface 2/GLV_5v
- U402 pad 4: /CAN interface 2/5v -> /CAN interface 2/GLV_5v
- U403 pad 8: /CAN interface 2/5v -> /CAN interface 2/GLV_5v
- U404 pad 3: /CAN interface 2/CAN- -> /CAN interface 2/CAN+
- U405 pad 1: Net-(RN2D-R4.1) -> Net-(U405-EN/FLT)
- U405 pad 2: /CAN interface 2/5v -> /CAN interface 2/GLV_5v
Routing:
- net +3.3V: track 0.00 -> 159.1 mm, vias 0 -> 7
- net /Ethernet/+3.3VA: track 0.00 -> 67.6 mm, vias 0 -> 3
- net /CAN interface 1/GLV_5v: track 0.00 -> 61.3 mm, vias 0 -> 2
- net Net-(J301-PadL3): track 0.00 -> 60.7 mm
- net Net-(J301-PadL2): track 0.00 -> 47.6 mm
- net /CAN interface 2/GLV_5v: track 0.00 -> 37.8 mm, vias 0 -> 1
- net /eth.cs_N: track 0.00 -> 35.5 mm
- net /eth.SCLK: track 0.00 -> 34.8 mm
- net /eth.MISO/POCI: track 0.00 -> 33.8 mm, vias 0 -> 2
- net /eth.MOSI/PICO: track 0.00 -> 33.1 mm
- net /eth.reset_N: track 0.00 -> 32.0 mm
- net /can0.term: track 0.00 -> 31.5 mm
- net /Ethernet/TD+: track 0.00 -> 31.3 mm, vias 0 -> 2
- net /Ethernet/TD-: track 0.00 -> 31.2 mm, vias 0 -> 2
- net /can0.RX: track 0.00 -> 30.3 mm
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- added copper zone on B.Cu, net /CAN interface 1/LV-
- added copper zone on F.Cu, net /CAN interface 1/LV-
- added copper zone on B.Cu, net /CAN interface 2/LV-
- added copper zone on F.Cu, net /CAN interface 2/LV-
- added copper zone on B.Cu, net GND
- added copper zone on F.Cu, net GND
Other:
- board outline added: 60 x 60 mm
- board text added: "(8,40)V +-45V max"
- board text added: "April 2026"
- board text added: "Board"
- board text added: "CAN L CAN H"
- board text added: "CAN#0"
- board text added: "CAN#1"
- board text added: "CAN0"
- board text added: "CAN1"
- board text added: "CANE v1.0"
- board text added: "Eth IP"
- board text added: "GND"
- board text added: "HV Isolation"
- board text added: "HW & SW info"
- board text added: "LV+ LV-"
- board text added: "Low Voltage"
- board text added: "R"
- board text added: "SWD CL IO"
- board text added: "T"
- board text added: "TTY 115200 8N1"
- board text added: "board powered from CAN interface"

Commit message: transcevier out of stock, swapped out
Parts:
- removed U203, U403: ISO1044BD, Package_SO:SOIC-8_5.3x5.3mm_P1.27mm
- added U3: ISO1042, Package_SO:SOIC-8_7.5x5.85mm_P1.27mm, F.Cu at (123.0, 67.5)
- added U4: ISO1042, Package_SO:SOIC-8_7.5x5.85mm_P1.27mm, F.Cu at (121.6, 106.8)
- CR401, R205, R407: moved to B.Cu
- moved R405 8.20 mm to (112.6, 100.3)
- moved R406 8.01 mm to (126.4, 76.7), turned to 0 degrees
- moved R407 7.16 mm to (127.0, 101.2), turned to -90 degrees
- moved R205 6.96 mm to (112.3, 73.9)
- moved U204 6.81 mm to (122.0, 73.3)
- moved U404 6.00 mm to (121.8, 101.3)
- moved FL201 3.93 mm to (114.5, 67.8)
- moved FL401 2.50 mm to (112.7, 104.3), turned to 0 degrees
- moved CR201 2.38 mm to (113.5, 72.8), turned to 180 degrees
- moved C108 2.09 mm to (129.1, 73.2)
- moved CR401 1.08 mm to (112.6, 106.5), turned to -90 degrees
- moved J3 0.55 mm to (125.9, 96.7)
- moved C403 0.10 mm to (116.4, 98.2)
Connections:
- R205 pad 1: /CAN interface 1/CAN+ -> /CAN interface 1/CAN-
- R405 pad 1: /CAN interface 2/CAN- -> /CAN interface 2/CAN+
- U2 pad 1: unconnected-(U2-PB13-Pad1) -> /can0.term
- U2 pad 15: unconnected-(U2-PB18-Pad15) -> /can1.term
- U2 pad 19: /can1.term -> unconnected-(U2-PB20-Pad19)
- U2 pad 7: /can0.term -> unconnected-(U2-PA14-Pad7)
- U204 pad 3: /CAN interface 1/CAN- -> Net-(R205-Pad2)
- U204 pad 4: Net-(R205-Pad2) -> /CAN interface 1/CAN+
- U404 pad 3: /CAN interface 2/CAN+ -> Net-(R405-Pad2)
- U404 pad 4: Net-(R405-Pad2) -> /CAN interface 2/CAN-
Routing:
- net +3.3V: track 159.1 -> 172.9 mm, vias 7 -> 6
- net /CAN interface 1/CAN+: track 6.22 -> 17.7 mm
- net /CAN interface 2/CAN+: track 18.0 -> 6.61 mm
- net /CAN interface 2/CAN-: track 26.4 -> 15.3 mm
- net /can0.term: track 31.5 -> 20.5 mm
- net /can0.TX: track 27.9 -> 34.2 mm
- net /CAN interface 1/GLV_5v: track 61.3 -> 56.2 mm
- net /can0.RX: track 30.3 -> 34.5 mm
- net /CAN interface 2/GLV_5v: track 37.8 -> 41.6 mm, vias 1 -> 3
- net /CAN interface 1/CAN-: track 16.9 -> 13.3 mm, vias 0 -> 1
- net Net-(R205-Pad2): track 2.74 -> 6.06 mm, vias 0 -> 1
- net Net-(U4-CANL): track 7.36 -> 4.07 mm, vias 0 -> 1
- net /CAN interface 2/LV-: track 10.00 -> 12.3 mm, vias 10 -> 9
- net Net-(U3-CANH): track 7.31 -> 5.21 mm
- net /can1.RX: track 10.8 -> 8.74 mm
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Other:
- board text added: "600Vdc isolation"
- board text removed: "HV Isolation"

Commit message: mmm
Parts:
- removed C103, C104, C401, C402, C403: 220n, Capacitor_SMD:C_0805_2012Metric_Pad1.18x1.45mm_HandSolder
- removed C404, C405: 22u, Capacitor_SMD:C_0805_2012Metric_Pad1.18x1.45mm_HandSolder
- removed CR401: ESD2CAN36DBZRQ1, Package_TO_SOT_SMD:TSOT-23_HandSoldering
- removed D401: TS4148, Diode_SMD:D_0805_2012Metric_Pad1.15x1.40mm_HandSolder
- removed FL401: Choke_CommonMode_FerriteCore_1243, zzLocalLibraries-Footprints:L_CommonModeChoke_Coilcraft_1812CAN
- removed J1, J2: glv, Connector_Molex:Molex_Micro-Fit_3.0_43045-0400_2x02_P3.00mm_Horizontal
- removed R2, R5, R7: 40.2k, Resistor_SMD:R_0805_2012Metric_Pad1.20x1.40mm_HandSolder
- removed R205, R405: 121, Resistor_SMD:R_0805_2012Metric_Pad1.20x1.40mm_HandSolder
- removed R406, R407: 750, Resistor_SMD:R_0805_2012Metric_Pad1.20x1.40mm_HandSolder
- removed RN1, RN2: 56K, zzLocalLibraries-Footprints:R_array_YCJ164_4
- removed U3, U4: ISO1042, Package_SO:SOIC-8_7.5x5.85mm_P1.27mm
- removed U401: TL432DBZ, Package_TO_SOT_SMD:SOT-23-3
- removed U402: TPS7B4254, Package_SO:Texas_R-PDSO-G8_EP2.95x4.9mm_Mask2.4x3.1mm
- removed U404: ISOM8600, zzLocalLibraries-Footprints:SOIC4_DFG_TEX-M
- removed U405: PUCC33420QRAQRQ1, zzLocalLibraries-Footprints:VSON-FCRLF12_RAQ_TEX
- added C1: 470n, Capacitor_SMD:C_0805_2012Metric_Pad1.18x1.45mm_HandSolder, F.Cu at (65.8, 91.8)
- added C101: 470n, Capacitor_SMD:C_0805_2012Metric_Pad1.18x1.45mm_HandSolder, F.Cu at (66.6, 36.1)
- added C106: 470n, Capacitor_SMD:C_0805_2012Metric_Pad1.18x1.45mm_HandSolder, F.Cu at (66.6, 39.2)
- added C110: 220n, Capacitor_SMD:C_0805_2012Metric_Pad1.18x1.45mm_HandSolder, F.Cu at (66.6, 42.2)
- added C111: 22u, Capacitor_SMD:C_0805_2012Metric_Pad1.18x1.45mm_HandSolder, F.Cu at (66.6, 45.2)
- added C112: 22u, Capacitor_SMD:C_0805_2012Metric_Pad1.18x1.45mm_HandSolder, F.Cu at (66.6, 48.2)
- added C113: 22u, Capacitor_SMD:C_0805_2012Metric_Pad1.18x1.45mm_HandSolder, F.Cu at (66.6, 51.2)
- added C206: 22u, Capacitor_SMD:C_0805_2012Metric_Pad1.18x1.45mm_HandSolder, F.Cu at (32.9, 77.2)
- added CR101: ESD2CAN36DBZRQ1, Package_TO_SOT_SMD:TSOT-23_HandSoldering, F.Cu at (91.1, 51.8)
- added D101: ES1D, Diode_SMD:D_SMA, F.Cu at (83.6, 51.6)
- added D103: ES1D, Diode_SMD:D_SMA, F.Cu at (83.6, 56.2)
- added D202: ES1D, Diode_SMD:D_SMA, F.Cu at (49.9, 82.1)
- added FL101: Choke_CommonMode_FerriteCore_1243, Inductor_SMD:L_CommonMode_Wurth_WE-CNSW-1206, F.Cu at (90.3, 59.8)
- added J101: glv, Connector_Molex:Molex_Micro-Fit_3.0_43045-0400_2x02_P3.00mm_Horizontal, F.Cu at (73.6, 44.6)
- added J201: glv, Connector_Molex:Molex_Micro-Fit_3.0_43045-0400_2x02_P3.00mm_Horizontal, F.Cu at (39.9, 70.5)
- added L101: 10u, Inductor_SMD:L_1210_3225Metric_Pad1.42x2.65mm_HandSolder, F.Cu at (90.6, 56.1)
- added L201: 10u, Inductor_SMD:L_1210_3225Metric_Pad1.42x2.65mm_HandSolder, F.Cu at (56.9, 82.1)
- added R1: 100k, Resistor_SMD:R_0805_2012Metric_Pad1.20x1.40mm_HandSolder, F.Cu at (65.7, 94.8)
- added R101: 121, Resistor_SMD:R_0805_2012Metric_Pad1.20x1.40mm_HandSolder, F.Cu at (92.0, 36.1)
- added R102: 750, Resistor_SMD:R_0805_2012Metric_Pad1.20x1.40mm_HandSolder, F.Cu at (92.0, 39.1)
- added R201: 121, Resistor_SMD:R_0805_2012Metric_Pad1.20x1.40mm_HandSolder, F.Cu at (58.3, 62.1)
- added R202: 750, Resistor_SMD:R_0805_2012Metric_Pad1.20x1.40mm_HandSolder, F.Cu at (58.3, 65.0)
- added RN101: 20k, zzLocalLibraries-Footprints:R_array_EXB2HV_8, F.Cu at (92.2, 43.2)
- added RN201: 20k, zzLocalLibraries-Footprints:R_array_EXB2HV_8, F.Cu at (58.5, 69.2)
- added TP1: TestPoint, TestPoint:TestPoint_Pad_D1.0mm, F.Cu at (80.5, 99.9)
- added TP101: TestPoint, TestPoint:TestPoint_Pad_D1.0mm, F.Cu at (80.5, 105.0)
- added TP201: TestPoint, TestPoint:TestPoint_Pad_D1.0mm, F.Cu at (85.6, 99.9)
- added U101: AP64060ZQ, Package_TO_SOT_SMD:TSOT-23-6, F.Cu at (82.1, 60.9)
- added U103: MCP2542FDxMF, Package_SO:SOIC-8_3.9x4.9mm_P1.27mm, F.Cu at (85.4, 38.0)
- added U104: ISO7721D, Package_SO:SOIC-8_3.9x4.9mm_P1.27mm, F.Cu at (85.4, 44.6)
- added U105: ISOM8600, zzLocalLibraries-Footprints:SOIC4_DFG_TEX-M, F.Cu at (74.3, 52.2)
- added U106: PUCC33420QRAQRQ1, zzLocalLibraries-Footprints:VSON-FCRLF12_RAQ_TEX, F.Cu at (73.1, 58.0)
- added U203: ISO7721D, Package_SO:SOIC-8_3.9x4.9mm_P1.27mm, F.Cu at (51.7, 70.5)
- C201, C202: value 220n -> 470n
- D201: value TS4148 -> ES1D; footprint Diode_SMD:D_0805_2012Metric_Pad1.15x1.40mm_HandSolder -> Diode_SMD:D_SMA
- FL201: footprint zzLocalLibraries-Footprints:L_CommonModeChoke_Coilcraft_1812CAN -> Inductor_SMD:L_CommonMode_Wurth_WE-CNSW-1206
- U201: value TL432DBZ -> AP64060ZQ; footprint Package_TO_SOT_SMD:SOT-23-3 -> Package_TO_SOT_SMD:TSOT-23-6
- U202: value TPS7B4254 -> MCP2542FDxMF; footprint Package_SO:Texas_R-PDSO-G8_EP2.95x4.9mm_Mask2.4x3.1mm -> Package_SO:SOIC-8_3.9x4.9mm_P1.27mm
- moved C203 83.8 mm to (32.9, 68.1)
- moved C201 83.4 mm to (32.9, 62.1)
- moved U204 81.6 mm to (40.6, 78.2), turned to 0 degrees
- moved C202 78.8 mm to (32.9, 65.1)
- moved U201 72.0 mm to (48.4, 86.8), turned to 0 degrees
- moved C205 70.8 mm to (32.9, 74.1), turned to 0 degrees
- moved C204 69.8 mm to (32.9, 71.1)
- moved U205 68.2 mm to (39.4, 84.0), turned to 0 degrees
- moved U202 65.5 mm to (51.7, 64.0), turned to 0 degrees
- moved D201 64.3 mm to (49.9, 77.6)
- moved FL201 60.6 mm to (56.6, 85.8)
- moved CR201 56.3 mm to (57.4, 77.8), turned to 0 degrees
Connections:
- C201 pad 1: /CAN interface 1/LV+ -> Net-(D201-K)
- C201 pad 2: /CAN interface 1/LV- -> /CAN interface 2/LV-
- C202 pad 1: /CAN interface 1/5v_ldo_ref -> Net-(D201-K)
- C202 pad 2: /CAN interface 1/LV- -> /CAN interface 2/LV-
- C203 pad 1: /CAN interface 1/GLV_5v -> Net-(U201-BST)
- C203 pad 2: /CAN interface 1/LV- -> Net-(D202-K)
- C204 pad 1: /CAN interface 1/GLV_5v -> /CAN interface 2/GLV_5v
- C204 pad 2: /CAN interface 1/LV- -> /CAN interface 2/LV-
- C205 pad 1: GND -> /CAN interface 2/GLV_5v
- C205 pad 2: /CAN interface 1/5v -> /CAN interface 2/LV-
- CR201 pad 1: Net-(U3-CANL) -> Net-(U202-CANL)
- CR201 pad 2: Net-(U3-CANH) -> Net-(U202-CANH)
- CR201 pad 3: /CAN interface 1/LV- -> /CAN interface 2/LV-
- D201 pad 1: /CAN interface 1/5v_ldo_ref -> Net-(D201-K)
- D201 pad 2: Net-(D201-A) -> /CAN interface 2/LV+
- FL201 pad 1: /CAN interface 1/CAN- -> /CAN interface 2/CAN-
- FL201 pad 2: Net-(U3-CANL) -> Net-(U202-CANL)
- FL201 pad 3: Net-(U3-CANH) -> Net-(U202-CANH)
- FL201 pad 4: /CAN interface 1/CAN+ -> /CAN interface 2/CAN+
- U201 pad 1: Net-(RN1A-R1.2) -> Net-(U201-BST)
- U201 pad 2: /CAN interface 1/5v_ldo_ref -> /CAN interface 2/LV-
- U201 pad 3: /CAN interface 1/LV- -> Net-(RN201D-R4.1)
- U202 pad 1: /CAN interface 1/GLV_5v -> Net-(U202-TXD)
- U202 pad 2: unconnected-(U202-NC-Pad2) -> /CAN interface 2/LV-
- U202 pad 3: /CAN interface 1/LV- -> /CAN interface 2/GLV_5v
- U202 pad 4: /CAN interface 1/GLV_5v -> Net-(U202-RXD)
- U202 pad 5: /CAN interface 1/5v_ldo_ref -> /CAN interface 2/GLV_5v
- U202 pad 6: /CAN interface 1/LV- -> Net-(U202-CANL)
- U202 pad 7: unconnected-(U202-NC-Pad7) -> Net-(U202-CANH)
- U202 pad 8: /CAN interface 1/LV+ -> /CAN interface 2/LV-
- U204 pad 4: /CAN interface 1/CAN+ -> /CAN interface 2/CAN+
- U205 pad 2: /CAN interface 1/GLV_5v -> /CAN interface 2/GLV_5v
- U205 pad 3: /CAN interface 1/LV- -> /CAN interface 2/LV-
- U205 pad 4: /CAN interface 1/LV- -> /CAN interface 2/LV-
- U205 pad 5: /CAN interface 1/LV- -> /CAN interface 2/LV-
- U205 pad 6: /CAN interface 1/LV- -> /CAN interface 2/LV-
- U205 pad 7: /CAN interface 1/5v -> /CAN interface 2/5v
- U205 pad 8: /CAN interface 1/5v -> /CAN interface 2/5v
Routing:
- net (no net): track 0.00 -> 57.8 mm, vias 0 -> 7
- net /CAN interface 1/5v_ldo_ref: track 18.9 -> 0.00 mm
- net /CAN interface 2/5v_ldo_ref: track 10.7 -> 0.00 mm, vias 2 -> 0
- net Net-(U3-CANL): track 9.95 -> 0.00 mm
- net Net-(U103-CANL): track 0.00 -> 9.95 mm
- net Net-(U4-CANH): track 6.40 -> 0.00 mm, vias 1 -> 0
- net Net-(R201-Pad2): track 6.06 -> 0.00 mm, vias 1 -> 0
- net Net-(R101-Pad2): track 0.00 -> 6.06 mm, vias 0 -> 1
- net Net-(U3-CANH): track 5.21 -> 0.00 mm
- net Net-(U103-CANH): track 0.00 -> 5.21 mm
- net Net-(R405-Pad2): track 5.00 -> 0.00 mm
- net Net-(U4-CANL): track 4.07 -> 0.00 mm, vias 1 -> 0
- net Net-(RN201H-R8.1): track 3.90 -> 0.00 mm, vias 1 -> 0
- net Net-(RN101H-R8.1): track 0.00 -> 3.90 mm, vias 0 -> 1
- net Net-(R407-Pad1): track 3.13 -> 0.00 mm, vias 1 -> 0
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