File: hardware/CANE Junction/CANE Junction.kicad_pcb (KiCad board)
At the start: 2 copper layers, 60 x 60 mm, 100 parts, among them IC1 PAM8904QJER, J101 glv, J201 glv, J3 programming, J301 RJ45_Amphenol_RJMG1BD3B8K1ANR, J4 UART, SW101 SW_Push, U1 MX25L3233FM2, U101 AP64060ZQ, U102 NCP114ASN180T2G, U103 MCP2542FDxMF, U104 ISO7721D, U105 ISOM8600, U106 PUCC33420QRAQRQ1, U2 XMSPM0G3519SPMR, U201 AP64060ZQ, U202 MCP2542FDxMF, U203 ISO7721D, U204 ISOM8600, U205 PUCC33420QRAQRQ1, U301 W5500, Y301 Crystal_GND24

Commit message: tmb pci technology
doner motherboard generator
Parts:
- removed the C105 at (116.2, 80.9)
- removed C108, C109: 220n, Capacitor_SMD:C_0805_2012Metric_Pad1.18x1.45mm_HandSolder
- removed C825, C826, C827: 100n, Capacitor_SMD:C_0805_2012Metric_Pad1.18x1.45mm_HandSolder
- removed D1, D2: SD0805S020S1R0, Diode_SMD:D_0805_2012Metric_Pad1.15x1.40mm_HandSolder
- removed TP1, TP101, TP201: TestPoint, TestPoint:TestPoint_Pad_D1.0mm
- removed U102: NCP114ASN180T2G, Package_TO_SOT_SMD:SOT-23-5_HandSoldering
- removed the U104 at (85.4, 44.6)
- added C10: 100n, Capacitor_SMD:C_0805_2012Metric_Pad1.18x1.45mm_HandSolder, F.Cu at (133.1, 81.9)
- added C11: 470n, Capacitor_SMD:C_0805_2012Metric_Pad1.18x1.45mm_HandSolder, F.Cu at (125.4, 97.8)
- added C110: 220n, Capacitor_SMD:C_0805_2012Metric_Pad1.18x1.45mm_HandSolder, F.Cu at (115.7, 76.1)
- added C2: 470n, Capacitor_SMD:C_0805_2012Metric_Pad1.18x1.45mm_HandSolder, B.Cu at (141.7, 105.0)
- added C3: 470n, Capacitor_SMD:C_0805_2012Metric_Pad1.18x1.45mm_HandSolder, F.Cu at (125.5, 61.9)
- added C5: 22u, Capacitor_SMD:C_0805_2012Metric_Pad1.18x1.45mm_HandSolder, F.Cu at (149.7, 98.9)
- added C7: 22u, Capacitor_SMD:C_0805_2012Metric_Pad1.18x1.45mm_HandSolder, F.Cu at (131.1, 90.2)
- added C8: 100n, Capacitor_SMD:C_0805_2012Metric_Pad1.18x1.45mm_HandSolder, F.Cu at (130.3, 84.7)
- added C9: 100n, Capacitor_SMD:C_0805_2012Metric_Pad1.18x1.45mm_HandSolder, F.Cu at (130.7, 81.4)
- added G***: LOGO, LOGO, B.Cu at (134.2, 95.7)
- added U106: NCP163ASN330T1G, Package_TO_SOT_SMD:SOT-23-5_HandSoldering, F.Cu at (125.5, 58.3)
- C1, C101, C201, C202, C313, R103, R303, R309, R313: moved to B.Cu
- C102: renamed from C106; moved to B.Cu
- D103, D202: value ES1D -> TS4148; footprint Diode_SMD:D_SMA -> Diode_SMD:D_0805_2012Metric_Pad1.15x1.40mm_HandSolder; moved to B.Cu
- IC1: moved to F.Cu
- U103, U202: value MCP2542FDxMF -> ISO1044BD; footprint Package_SO:SOIC-8_3.9x4.9mm_P1.27mm -> Package_SO:SOIC-8_5.3x6.2mm_P1.27mm
- U203: value ISO7721D -> ISOM8600; footprint Package_SO:SOIC-8_3.9x4.9mm_P1.27mm -> zzLocalLibraries-Footprints:SOIC4_DFG_TEX-M
- U204: value ISOM8600 -> PUCC33420QRAQRQ1; footprint zzLocalLibraries-Footprints:SOIC4_DFG_TEX-M -> zzLocalLibraries-Footprints:VSON-FCRLF12_RAQ_TEX
- U205: value PUCC33420QRAQRQ1 -> NCP163ASN330T1G; footprint zzLocalLibraries-Footprints:VSON-FCRLF12_RAQ_TEX -> Package_TO_SOT_SMD:SOT-23-5_HandSoldering
- moved C206 98.2 mm to (126.5, 106.9), turned to -90 degrees
- moved C205 89.8 mm to (116.4, 107.1), turned to -90 degrees
- moved C201 88.6 mm to (113.5, 98.9), turned to 90 degrees
- moved U205 88.0 mm to (125.8, 101.2), turned to 90 degrees
- moved R1 88.0 mm to (153.6, 98.6)
- moved C203 87.9 mm to (115.3, 98.9), turned to -90 degrees
- moved C204 86.8 mm to (112.8, 105.2), turned to 180 degrees
- moved U204 86.1 mm to (121.7, 107.1)
- moved C202 85.5 mm to (111.5, 98.9), turned to 90 degrees
- moved C1 79.1 mm to (143.7, 105.0), turned to 90 degrees
- moved R202 77.7 mm to (129.3, 96.7), turned to -45 degrees
- moved U202 75.3 mm to (121.6, 92.1), turned to 180 degrees
- moved J201 72.8 mm to (108.4, 95.2), turned to 90 degrees
- moved U203 71.0 mm to (121.5, 83.7), turned to 180 degrees
- moved D202 66.9 mm to (113.2, 103.9), turned to -135 degrees
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- renumbered C110 to C103, C111 to C104, C112 to C105, C113 to C106, U105 to U104, U106 to U105
Connections:
- net /CAN interface 1/5v renamed Net-(U105-SEL)
- net Net-(U103-CANL) renamed /CAN interface 1/C_P
- C206 pad 2: /CAN interface 2/5v -> Net-(U204-SEL)
- CR101 pad 2: Net-(U103-CANH) -> /CAN interface 1/C_N
- CR201 pad 1: Net-(U202-CANL) -> /CAN interface 2/C_N
- CR201 pad 2: Net-(U202-CANH) -> /CAN interface 2/C_P
- D102 pad 1: GND -> Net-(D102-K)
- FL101 pad 1: /CAN interface 1/CAN- -> /CAN interface 1/CAN+
- FL101 pad 3: Net-(U103-CANH) -> /CAN interface 1/C_N
- FL101 pad 4: /CAN interface 1/CAN+ -> /CAN interface 1/CAN-
- FL201 pad 1: /CAN interface 2/CAN- -> /CAN interface 2/CAN+
- FL201 pad 2: Net-(U202-CANL) -> /CAN interface 2/C_P
- FL201 pad 3: Net-(U202-CANH) -> /CAN interface 2/C_N
- FL201 pad 4: /CAN interface 2/CAN+ -> /CAN interface 2/CAN-
- R103 pad 1: Net-(U2-PA0) -> +3.3V
- R201 pad 1: /CAN interface 2/CAN- -> Net-(R201-Pad1)
- R201 pad 2: Net-(R201-Pad2) -> /CAN interface 2/CAN-
- RN101 pad 10: (no net) -> Net-(RN101G-R7.2)
- RN101 pad 11: (no net) -> Net-(RN101E-R5.2)
- RN101 pad 12: Net-(RN101D-R4.1) -> Net-(RN101E-R5.2)
- RN101 pad 13: Net-(RN101C-R3.1) -> /CAN interface 1/GLV_5v
- RN101 pad 14: Net-(RN101B-R2.1) -> unconnected-(RN101C-R3.2-Pad14)
- RN101 pad 15: Net-(RN101A-R1.1) -> unconnected-(RN101B-R2.2-Pad15)
- RN101 pad 2: Net-(RN101B-R2.1) -> unconnected-(RN101B-R2.1-Pad2)
- RN101 pad 3: Net-(RN101C-R3.1) -> unconnected-(RN101C-R3.1-Pad3)
- RN101 pad 5: /CAN interface 1/LV- -> Net-(RN101D-R4.1)
- RN101 pad 6: (no net) -> Net-(RN101F-R6.1)
- RN101 pad 7: (no net) -> Net-(RN101F-R6.1)
- RN101 pad 8: Net-(RN101H-R8.1) -> /CAN interface 1/LV-
- RN101 pad 9: /CAN interface 1/GLV_5v -> Net-(RN101G-R7.2)
- RN201 pad 1: Net-(RN201A-R1.1) -> /CAN interface 2/LV-
- RN201 pad 10: (no net) -> unconnected-(RN201G-R7.2-Pad10)
- RN201 pad 11: (no net) -> unconnected-(RN201F-R6.2-Pad11)
- RN201 pad 12: Net-(RN201D-R4.1) -> /CAN interface 2/GLV_5v
- RN201 pad 13: Net-(RN201C-R3.1) -> Net-(RN201C-R3.2)
- RN201 pad 14: Net-(RN201B-R2.1) -> Net-(RN201C-R3.2)
- RN201 pad 15: Net-(RN201A-R1.1) -> Net-(RN201A-R1.2)
- RN201 pad 16: /CAN interface 2/GLV_5v -> Net-(RN201A-R1.2)
- RN201 pad 3: Net-(RN201C-R3.1) -> Net-(RN201B-R2.1)
- RN201 pad 5: /CAN interface 2/LV- -> Net-(RN201D-R4.1)
- RN201 pad 6: (no net) -> unconnected-(RN201F-R6.1-Pad6)
- RN201 pad 7: (no net) -> unconnected-(RN201G-R7.1-Pad7)
- RN201 pad 8: Net-(RN201H-R8.1) -> /CAN interface 2/GLV_5v
- RN201 pad 9: /CAN interface 2/GLV_5v -> Net-(RN201H-R8.2)
- U101 pad 3: Net-(RN101D-R4.1) -> Net-(RN101G-R7.2)
- U103 pad 1: Net-(U103-TXD) -> +3.3V
- U103 pad 2: /CAN interface 1/LV- -> /can0.TX
- U103 pad 3: /CAN interface 1/GLV_5v -> /can0.RX
- U103 pad 4: Net-(U103-RXD) -> GND
- U103 pad 5: /CAN interface 1/GLV_5v -> /CAN interface 1/C_N
- U103 pad 7: Net-(U103-CANH) -> /CAN interface 1/LV-
- U103 pad 8: /CAN interface 1/LV- -> /CAN interface 1/GLV_5v
- U105 pad 1: Net-(RN101H-R8.1) -> Net-(RN101A-R1.1)
- U2 pad 11: unconnected-(U2-PA18-Pad11) -> /can1.term
- U2 pad 15: /can1.term -> unconnected-(U2-PB18-Pad15)
- U2 pad 33: Net-(U2-PA0) -> Net-(D102-K)
- U2 pad 43: unconnected-(U2-PA3-Pad43) -> /SECD.cs_fr
- U2 pad 48: /SECD.cs_fr -> unconnected-(U2-PB1-Pad48)
- U2 pad 56: unconnected-(U2-PA10-Pad56) -> GND
- U2 pad 57: unconnected-(U2-PA11-Pad57) -> /eth.reset_N
- U2 pad 58: /eth.reset_N -> /eth.irq_N
- U201 pad 3: Net-(RN201D-R4.1) -> Net-(RN201A-R1.2)
- U202 pad 1: Net-(U202-TXD) -> +3.3V
- U202 pad 2: /CAN interface 2/LV- -> /can1.TX
- U202 pad 3: /CAN interface 2/GLV_5v -> /can1.RX
- U202 pad 4: Net-(U202-RXD) -> GND
- U202 pad 5: /CAN interface 2/GLV_5v -> /CAN interface 2/C_N
- U202 pad 6: Net-(U202-CANL) -> /CAN interface 2/C_P
- U202 pad 7: Net-(U202-CANH) -> /CAN interface 2/LV-
- U202 pad 8: /CAN interface 2/LV- -> /CAN interface 2/GLV_5v
- U203 pad 1: /CAN interface 2/GLV_5v -> Net-(R202-Pad1)
- U203 pad 2: Net-(U202-TXD) -> GND
- U203 pad 3: Net-(U202-RXD) -> /CAN interface 2/CAN+
- U203 pad 4: /CAN interface 2/LV- -> Net-(R201-Pad1)
- U204 pad 1: Net-(R202-Pad1) -> Net-(RN201H-R8.2)
- U204 pad 2: GND -> /CAN interface 2/GLV_5v
- U204 pad 3: Net-(R201-Pad2) -> /CAN interface 2/LV-
- U204 pad 4: /CAN interface 2/CAN+ -> /CAN interface 2/LV-
- U205 pad 1: Net-(RN201H-R8.1) -> Net-(U204-SEL)
- U205 pad 2: /CAN interface 2/GLV_5v -> GND
- U205 pad 3: /CAN interface 2/LV- -> Net-(U204-SEL)
- U205 pad 4: /CAN interface 2/LV- -> unconnected-(U205-NC-Pad4)
- U205 pad 5: /CAN interface 2/LV- -> +3.3V
Routing:
- net (no net): track 57.8 -> 0.00 mm, vias 7 -> 0
- net /eth.irq_N: track 0.00 -> 31.7 mm
- net Net-(D1-K): track 24.9 -> 0.00 mm
- net /can1.RX: track 8.74 -> 31.5 mm
- net /can1.TX: track 7.76 -> 27.0 mm
- net /CAN interface 1/LV+: track 27.4 -> 9.87 mm
- net /CAN interface 2/C_P: track 0.00 -> 16.3 mm
- net Net-(RN101G-R7.2): track 0.00 -> 15.4 mm
- net Net-(U204-SEL): track 0.00 -> 14.0 mm
- net /CAN interface 2/CAN+: track 6.61 -> 20.5 mm
- net /CAN interface 2/GLV_5v: track 41.6 -> 27.8 mm, vias 3 -> 0
- net /CAN interface 1/GLV_5v: track 56.2 -> 42.5 mm, vias 2 -> 0
- net Net-(R202-Pad1): track 0.00 -> 13.1 mm
- net /CAN interface 1/C_N: track 0.00 -> 12.6 mm
- net Net-(D201-K): track 0.00 -> 12.5 mm, vias 0 -> 2
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- added copper zone on F.Cu, net Net-(D103-K)
- added copper zone on F.Cu, net Net-(D202-K)
Other:
- board text added: "(8,38)V +42V max"
- board text added: "CANE v1.1"
- board text added: "GND ^SWD"
- board text added: "IO CL"
- board text added: "antenna for 'them'"
- board text added: "tmb, LT is essential"
- board text removed: "(8,40)V +-45V max"
- board text removed: "Board"
- board text removed: "CAN L CAN H"
- board text removed: "CAN#0"
- board text removed: "CAN#1"
- board text removed: "CANE v1.0"
- board text removed: "Eth IP"
- board text removed: "LV+ LV-"
- board text removed: "SWD CL IO"
- board text removed: "board powered from CAN interface"
